File: hardware/tagbase-jlcpcb-v3/tagbase-jlcpcb-v3.kicad_pcb (KiCad board)
At the start: 2 copper layers, 50.8 x 69.9 mm, 41 parts, among them J1 Conn_01x04_Female, J101 Conn_02x03_Odd_Even, J102 Conn_02x05_Odd_Even, J104 USB_B_Mini, J2 Conn_01x02_Male, J3 Conn_01x02_Male, J5 Conn_01x02, SW1 SW_DIP_x04, U1 XC6206, U101 STM32F042K6Tx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

Commit message: update tagbase
Parts:
- removed J2, J3: Conn_01x02_Male, Connector_JST:JST_PH_B2B-PH-K_1x02_P2.00mm_Vertical
- U101: footprint tagbase:LQFP-32_7x7mm_P0.8mm -> Package_QFP:LQFP-32_7x7mm_P0.8mm
Connections:
- J101 pad 5: TAG_3V3 -> Net-(J101-Pad5)
- J102 pad 6: (no net) -> unconnected-(J102-Pad6)
- J102 pad 7: (no net) -> unconnected-(J102-Pad7)
- J102 pad 8: (no net) -> unconnected-(J102-Pad8)
- SW1 pad 8: TAG_3V3 -> Net-(J101-Pad5)
- U101 pad 11: (no net) -> unconnected-(U101-Pad11)
- U101 pad 12: (no net) -> unconnected-(U101-Pad12)
- U101 pad 13: (no net) -> unconnected-(U101-Pad13)
- U101 pad 15: (no net) -> unconnected-(U101-Pad15)
- U101 pad 2: (no net) -> unconnected-(U101-Pad2)
- U101 pad 25: (no net) -> unconnected-(U101-Pad25)
- U101 pad 27: (no net) -> unconnected-(U101-Pad27)
- U101 pad 3: (no net) -> unconnected-(U101-Pad3)
- U2 pad 3: (no net) -> unconnected-(U2-Pad3)
- U3 pad 3: (no net) -> unconnected-(U3-Pad3)
- U4 pad 1: (no net) -> TAG_3V3
- U5 pad 1: (no net) -> unconnected-(U5-Pad1)
Routing:
- net Net-(J101-Pad5): track 0.00 -> 27.7 mm, vias 0 -> 1
- net TAG_3V3: track 38.1 -> 12.0 mm
- net /VIN: vias 0 -> 2

Commit message: checkpoint
Parts:
- added J2: Conn_01x02, Connector_PinHeader_2.54mm:PinHeader_1x02_P2.54mm_Vertical, F.Cu at (147.2, 90.7)
Connections:
- SW1 pad 1: Net-(SW1-Pad1) -> unconnected-(SW1-Pad1)
- SW1 pad 8: Net-(J101-Pad5) -> unconnected-(SW1-Pad8)
- U4 pad 3: Net-(SW1-Pad1) -> +3V3
- U4 pad 4: +3V3 -> Net-(U4-Pad4)
Routing:
- net Net-(U4-Pad4): track 0.00 -> 30.9 mm, vias 0 -> 1
- net Net-(SW1-Pad1): track 8.81 -> 0.00 mm
- net Net-(J101-Pad5): track 27.7 -> 21.5 mm, vias 1 -> 0
- net +3V3: track 122.3 -> 125.3 mm, vias 9 -> 11
- net EXT_PWR: track 36.7 -> 38.1 mm
