File: hardware/tagbase-jlcpcb-v3/tagbase-jlcpcb-v3.kicad_sch (KiCad schematic)
At the start: 41 parts, among them J1 Conn_01x04_Female, J101 Conn_02x03_Odd_Even, J102 Conn_02x05_Odd_Even, J104 USB_B_Mini, J2 Conn_01x02_Male, J3 Conn_01x02_Male, J5 Conn_01x02, SW1 SW_DIP_x04, U1 XC6206, U101 STM32F042K6Tx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

Commit message: update tagbase
Parts:
- removed J2, J3: Conn_01x02_Male, Connector_JST:JST_PH_B2B-PH-K_1x02_P2.00mm_Vertical, symbol Connector_Generic:Conn_01x02
Connections:
- net TAG_3V3: now also U4.1; no longer J101.5 (Pin_5), SW1.8
- new net: J101.5 (Pin_5), SW1.8
- no-connect marks 15 -> 14
Other:
- note added: "Add jumper to enable resistor in v3.3"
- note added: "Moved TAG_3V3 to output of mux"
Changed lines of the file:
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@@
   (junction (at 93.98 177.8) (diameter 0) (color 0 0 0 0)
   )
-  (junction (at 119.38 31.75) (diameter 0) (color 0 0 0 0)
-  )
   (junction (at 184.15 40.64) (diameter 0) (color 0 0 0 0)
   )
@@
   (junction (at 227.33 143.51) (diameter 0) (color 0 0 0 0)
   )
-  (junction (at 228.6 40.64) (diameter 0) (color 0 0 0 0)
-  )
   (junction (at 44.45 29.21) (diameter 0) (color 0 0 0 0)
   )
@@
   )
   (junction (at 54.61 40.64) (diameter 0) (color 0 0 0 0)
-  )
-  (junction (at 119.38 34.29) (diameter 0) (color 0 0 0 0)
   )
   (junction (at 229.87 68.58) (diameter 0) (color 0 0 0 0)
@@
   (no_connect (at 85.09 80.01))
   (no_connect (at 85.09 82.55))
-  (no_connect (at 191.77 34.29))
   (no_connect (at 248.92 60.96))
   (wire (pts (xy 33.02 29.21) (xy 35.56 29.21))
@@
     (stroke (width 0) (type default) (color 0 0 0 0))
   )
-  (wire (pts (xy 119.38 29.21) (xy 119.38 31.75))
-    (stroke (width 0) (type default) (color 0 0 0 0))
-  )
   (wire (pts (xy 100.33 62.23) (xy 104.14 62.23))
     (stroke (width 0) (type default) (color 0 0 0 0))
@@
     (stroke (width 0) (type default) (color 0 0 0 0))
   )
+  (wire (pts (xy 191.77 34.29) (xy 199.39 34.29))
+    (stroke (width 0) (type default) (color 0 0 0 0))
+  )
   (wire (pts (xy 110.49 69.85) (xy 125.73 69.85))
     (stroke (width 0) (type default) (color 0 0 0 0))
@@
     (stroke (width 0) (type default) (color 0 0 0 0))
   )
-  (wire (pts (xy 119.38 34.29) (xy 121.92 34.29))
-    (stroke (width 0) (type default) (color 0 0 0 0))
-  )
-  (wire (pts (xy 116.84 34.29) (xy 119.38 34.29))
-    (stroke (width 0) (type default) (color 0 0 0 0))
-  )
   (wire (pts (xy 93.98 170.18) (xy 93.98 172.72))
     (stroke (width 0) (type default) (color 0 0 0 0))
@@
     (stroke (width 0) (type default) (color 0 0 0 0))
   )
-  (wire (pts (xy 228.6 40.64) (xy 220.98 40.64))
-    (stroke (width 0) (type default) (color 0 0 0 0))
-  )
   (wire (pts (xy 73.66 68.58) (xy 73.66 67.31))
     (stroke (width 0) (type default) (color 0 0 0 0))
@@
     (stroke (width 0) (type default) (color 0 0 0 0))
   )
-  (wire (pts (xy 119.38 31.75) (xy 121.92 31.75))
-    (stroke (width 0) (type default) (color 0 0 0 0))
-  )
   (wire (pts (xy 182.88 86.36) (xy 182.88 83.82))
     (stroke (width 0) (type default) (color 0 0 0 0))
@@
     (stroke (width 0) (type default) (color 0 0 0 0))
   )
-  (wire (pts (xy 119.38 34.29) (xy 119.38 36.83))
-    (stroke (width 0) (type default) (color 0 0 0 0))
-  )
   (wire (pts (xy 54.61 40.64) (xy 68.58 40.64))
     (stroke (width 0) (type default) (color 0 0 0 0))
@@
     (stroke (width 0) (type default) (color 0 0 0 0))
   )
-  (wire (pts (xy 116.84 31.75) (xy 119.38 31.75))
-    (stroke (width 0) (type default) (color 0 0 0 0))
-  )
   (wire (pts (xy 64.77 92.71) (xy 57.15 92.71))
     (stroke (width 0) (type default) (color 0 0 0 0))
@@
   (wire (pts (xy 256.54 35.56) (xy 256.54 41.91))
     (stroke (width 0) (type default) (color 0 0 0 0))
+  )
+  (text "Moved TAG_3V3 to output of \nmux" (at 199.39 30.48 0)
+    (effects (font (size 1.27 1.27)) (justify left bottom))
   )
   (text "Add protection for TagMirror and EXT_PWR" (at 130.81 101.6 0)
@@
     (effects (font (size 1.27 1.27)) (justify left bottom))
   )
+  (text "Add jumper to enable resistor in v3.3" (at 199.39 24.13 0)
+    (effects (font (size 1.27 1.27)) (justify left bottom))
+  )
   (label "USB_DP" (at 64.77 170.18 0)
     (effects (font (size 1.524 1.524)) (justify left bottom))
@@
     (effects (font (size 1.27 1.27)) (justify left bottom))
   )
-  (label "VIN" (at 119.38 29.21 180)
-    (effects (font (size 1.27 1.27)) (justify right bottom))
-  )
   (label "LED_RED" (at 121.92 134.62 180)
     (effects (font (size 1.524 1.524)) (justify right bottom))
@@
     )
   )
-  (global_label "TAG_3V3" (shape input) (at 220.98 40.64 180) (fields_autoplaced)
-    (effects (font (size 1.524 1.524)) (justify right))
-    (property "Intersheet References" "${INTERSHEET_REFS}" (id 0) (at 0 0 0)
+  (global_label "TAG_3V3" (shape input) (at 199.39 34.29 0) (fields_autoplaced)
+    (effects (font (size 1.524 1.524)) (justify left))
+    (property "Intersheet References" "${INTERSHEET_REFS}" (id 0) (at 420.37 74.93 0)
       (effects (font (size 1.27 1.27)) hide)
     )
@@
     )
     (property "Datasheet" "" (id 3) (at 172.72 64.77 0)
-      (effects (font (size 1.27 1.27)) hide)
-    )
-    (pin "1")
-  )
-  (symbol (lib_id "Connector_Generic:Conn_01x02") (at 111.76 31.75 0) (mirror y) (unit 1)
-    (in_bom yes) (on_board yes)
-    (property "Reference" "J2" (id 0) (at 109.0676 29.5402 0))
-    (property "Value" "Conn_01x02_Male" (id 1) (at 109.0676 29.5402 0)
-      (effects (font (size 1.27 1.27)) hide)
-    )
-    (property "Footprint" "Connector_JST:JST_PH_B2B-PH-K_1x02_P2.00mm_Vertical" (id 2) (at 111.76 31.75 0)
-      (effects (font (size 1.27 1.27)) hide)
-    )
-    (property "Datasheet" "~" (id 3) (at 111.76 31.75 0)
-      (effects (font (size 1.27 1.27)) hide)
-    )
-    (property "MPN" "B2B-PH-K-S(LF)(SN)" (id 4) (at 111.76 31.75 0)
-      (effects (font (size 1.27 1.27)) hide)
-    )
-    (pin "1")
-    (pin "2")
-  )
-  (symbol (lib_id "Connector_Generic:Conn_01x02") (at 127 31.75 0) (unit 1)
-    (in_bom yes) (on_board yes)
-    (property "Reference" "J3" (id 0) (at 126.2888 33.6042 0)
-      (effects (font (size 1.27 1.27)) (justify right))
-    )
-    (property "Value" "Conn_01x02_Male" (id 1) (at 129.6924 29.5402 0)
-      (effects (font (size 1.27 1.27)) hide)
-    )
-    (property "Footprint" "Connector_JST:JST_PH_B2B-PH-K_1x02_P2.00mm_Vertical" (id 2) (at 127 31.75 0)
-      (effects (font (size 1.27 1.27)) hide)
-    )
-    (property "Datasheet" "~" (id 3) (at 127 31.75 0)
-      (effects (font (size 1.27 1.27)) hide)
-    )
-    (property "MPN" "B2B-PH-K-S(LF)(SN)" (id 4) (at 127 31.75 0)
-      (effects (font (size 1.27 1.27)) hide)
-    )
-    (pin "1")
-    (pin "2")
-  )
-  (symbol (lib_id "power:GND") (at 119.38 36.83 0) (unit 1)
-    (in_bom yes) (on_board yes)
-    (property "Reference" "#PWR0111" (id 0) (at 119.38 43.18 0)
-      (effects (font (size 1.27 1.27)) hide)
-    )
-    (property "Value" "GND" (id 1) (at 119.507 41.2242 0))
-    (property "Footprint" "" (id 2) (at 119.38 36.83 0)
-      (effects (font (size 1.27 1.27)) hide)
-    )
-    (property "Datasheet" "" (id 3) (at 119.38 36.83 0)
       (effects (font (size 1.27 1.27)) hide)
     )
@@
       (reference "#PWR0110") (unit 1) (value "+3.3V") (footprint "")
     )
-    (path "/00000000-0000-0000-0000-00005ed89e67"
-      (reference "#PWR0111") (unit 1) (value "GND") (footprint "")
-    )
     (path "/00000000-0000-0000-0000-00005bf237f8"
       (reference "#PWR0112") (unit 1) (value "GND") (footprint "")
@@
       (reference "J1") (unit 1) (value "Conn_01x04_Female") (footprint "Connector_JST:JST_XH_B04B-XH-AM_1x04_P2.50mm_Vertical")
     )
-    (path "/00000000-0000-0000-0000-00005ed89b49"
-      (reference "J2") (unit 1) (value "Conn_01x02_Male") (footprint "Connector_JST:JST_PH_B2B-PH-K_1x02_P2.00mm_Vertical")
-    )
-    (path "/00000000-0000-0000-0000-00005ed89cd6"
-      (reference "J3") (unit 1) (value "Conn_01x02_Male") (footprint "Connector_JST:JST_PH_B2B-PH-K_1x02_P2.00mm_Vertical")
-    )
     (path "/00000000-0000-0000-0000-00005fce7579"

Commit message: checkpoint
Parts:
- added J2: Conn_01x02, Connector_PinHeader_2.54mm:PinHeader_1x02_P2.54mm_Vertical, symbol Connector_Generic:Conn_01x02
Connections:
- net +3V3: now also U4.3; no longer U4.4
- net at J101.5 (Pin_5): now also J2.2 (Pin_2); no longer SW1.8
- net at SW1.1: no longer U4.3
- new net: J2.1 (Pin_1), U4.4
- no-connect marks 14 -> 17
Other:
- note removed: "Add jumper to enable resistor in v3.3"
- note removed: "Moved TAG_3V3 to output of mux"
- moved on the sheet: J101
