File: hardware/PresTag/PresTag-v3.kicad_sch (KiCad schematic)
At the start: 20 parts, among them J201 CONN_02X04, J301 Conn_01x01, J302 Conn_01x01, J303 Conn_01x01, J304 Conn_01x01, J401 CONN_01X02, Q501 Q_NPN_BEC, U1 at25ex321D-UUN, U2 LPS27HHWTR, U302 stm32l431kc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

Commit message: update lps27 part number
Parts:
- U2: DISTPN 497-LPS27HHWCT-ND -> 497-LPS27HHTWCT-ND; MPN LPS27HHWTR -> LPS27HHTWTR
Changed lines of the file:
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@@
       (effects (font (size 1.524 1.524)))
     )
-    (property "DISTPN" "497-LPS27HHWCT-ND" (id 4) (at 58.42 135.89 0)
+    (property "DISTPN" "497-LPS27HHTWCT-ND" (id 4) (at 58.42 135.89 0)
       (effects (font (size 1.27 1.27)) hide)
     )
@@
       (effects (font (size 1.27 1.27)) hide)
     )
-    (property "MPN" "LPS27HHWTR" (id 6) (at 58.42 138.43 0)
+    (property "MPN" "LPS27HHTWTR" (id 6) (at 58.42 138.43 0)
       (effects (font (size 1.27 1.27)) hide)
     )
