File: hardware/tagbase-jlcpcb-v7/tagbase-jlcpcb-v3.kicad_sch (KiCad schematic)
At the start: 40 parts, among them J1 Conn_01x04_Female, J101 Conn_02x03_Odd_Even, J102 Conn_02x05_Odd_Even, J104 USB_B_Mini, J2 Conn_01x06, J5 Conn_01x02, SW1 SW_DIP_x04, U1 XC6206, U105 Tactile Switch, U2 TS5A3159ADBVR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

Commit message: update tagbase v7
Parts:
- removed H101, H102, H103, H104: MountingHole, tagbase:MountingHole_3.2mm_M3, symbol Mechanical:MountingHole
- added H1, H2, H3, H4: MountingHole, MountingHole:MountingHole_2.5mm, symbol Mechanical:MountingHole
- J104: DISTPN 151-1206-ND -> (none); LCSC (none) -> C2681563; MFN EDAC -> SHOU HAN; MPN 690-005-299-043 -> MINI 5PTP
- R5: LCSC (none) -> C23140; MFN (none) -> Uniroyal; MPN (none) -> 0603WAF330JT5E
- R6: LCSC (none) -> C23255; MFN (none) -> Uniroyal; MPN (none) -> 0603WAF820JT5E
- SW1: footprint Button_Switch_SMD:SW_DIP_SPSTx06_Slide_Copal_CHS-06B_W7.62mm_P1.27mm -> Button_Switch_SMD:SW_DIP_SPSTx06_Slide_KingTek_DSHP06TS_W7.62mm_P1.27mm; DISTPN CT3110CT-ND -> (none); LCSC (none) -> C3293146; MFN CTS Electrocomponents -> kangshen; MPN 218-4LPSTR -> DSHP06TSGER
- U6: LCSC (none) -> C961597; MFN (none) -> STMicroelectronics; MPN (none) -> STM32F042G6U6
Connections:
- net +3.3V is gone; now on net +3V3: D101.2 (A), D102.2 (A), U4.3, U5.4
- net EXT_PWR: now also U6.11 (PA5); no longer U6.14 (PB0)
- net TAG_3V3: now also J2.6 (Pin_6); no longer J2.3 (Pin_3)
- net TAG_RESET: now also J2.3 (Pin_3); no longer J2.4 (Pin_4)
- net TAG_SCK: now also J2.4 (Pin_4); no longer J2.6 (Pin_6)
