File: hardware/tagbase-jlcpcb-v7/tagbase-jlcpcb-v3.kicad_pcb (KiCad board)
At the start: 2 copper layers, 50.8 x 69.9 mm, 40 parts, among them J1 Conn_01x04_Female, J101 Conn_02x03_Odd_Even, J102 Conn_02x05_Odd_Even, J104 USB_B_Mini, J2 Conn_01x06, J5 Conn_01x02, SW1 SW_DIP_x04, U1 XC6206, U105 Tactile Switch, U2 TS5A3159ADBVR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

Commit message: update tagbase v7
Parts:
- removed H101, H102, H103, H104: MountingHole, tagbase:MountingHole_3.2mm_M3
- added H1: MountingHole, MountingHole:MountingHole_2.5mm, F.Cu at (106.0, 92.0)
- added H2: MountingHole, MountingHole:MountingHole_2.5mm, F.Cu at (106.0, 111.0)
- added H3: MountingHole, MountingHole:MountingHole_2.5mm, F.Cu at (148.0, 92.0)
- added H4: MountingHole, MountingHole:MountingHole_2.5mm, F.Cu at (148.0, 111.0)
- SW1: footprint Button_Switch_SMD:SW_DIP_SPSTx06_Slide_Copal_CHS-06B_W7.62mm_P1.27mm -> Button_Switch_SMD:SW_DIP_SPSTx06_Slide_KingTek_DSHP06TS_W7.62mm_P1.27mm
- moved C104 39.9 mm to (148.6, 53.1)
- moved C1 39.7 mm to (142.6, 53.1)
- moved U1 39.7 mm to (145.6, 53.1)
- moved D1 35.8 mm to (142.1, 57.6)
- moved J2 23.4 mm to (126.8, 78.2), turned to 180 degrees
- moved D105 21.7 mm to (109.5, 56.8)
- moved R107 21.7 mm to (107.6, 56.8)
- moved U2 6.22 mm to (118.0, 74.2), turned to 90 degrees
- moved R104 3.66 mm to (127.6, 74.6), turned to 0 degrees
- moved C2 2.21 mm to (127.9, 71.5)
- moved C101 1.45 mm to (119.7, 65.9), turned to -90 degrees
- moved C3 1.45 mm to (128.9, 62.6), turned to 90 degrees
- moved R102 0.60 mm to (138.2, 53.0)
- moved R105 0.54 mm to (117.2, 70.8)
- turned D3 to -90 degrees
Connections:
- D101 pad 2: +3.3V -> +3V3
- D102 pad 2: +3.3V -> +3V3
- J2 pad 3: TAG_3V3 -> TAG_RESET
- J2 pad 4: TAG_RESET -> TAG_SCK
- J2 pad 6: TAG_SCK -> TAG_3V3
- U4 pad 3: +3.3V -> +3V3
- U5 pad 4: +3.3V -> +3V3
- U6 pad 11: unconnected-(U6-Pad11) -> EXT_PWR
- U6 pad 14: EXT_PWR -> unconnected-(U6-Pad14)
Routing:
- net +3V3: track 56.8 -> 126.0 mm, vias 4 -> 5
- net /VIN: track 83.2 -> 14.7 mm, vias 1 -> 0
- net TAG_3V3: track 9.24 -> 39.5 mm, vias 0 -> 3
- net +3.3V: track 29.5 -> 0.00 mm, vias 5 -> 0
- net TAG_MIRROR: track 0.00 -> 20.6 mm
- net TAG_3V3_EN: track 0.00 -> 17.4 mm
- net TAG_SCK: track 10.9 -> 26.3 mm
- net TAG_SWDIO: track 26.2 -> 38.4 mm
- net ~{TAG_VBAT_EN}: track 0.00 -> 10.9 mm
- net TAG_VBAT: track 22.3 -> 30.9 mm
- net Net-(R108-Pad1): track 0.00 -> 8.30 mm
- net /LED_GREEN: track 8.54 -> 15.8 mm
- net VUSB: track 47.1 -> 39.9 mm
- net /NRST: track 8.29 -> 15.4 mm, vias 1 -> 2
- net Net-(R104-Pad2): track 0.00 -> 6.19 mm
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Other:
- board text added: "MS412/414 2K MS518 1.5K MS621/920 620 ------------ Charger Resistor"
- board text added: "SCK"
