File: hardware/Multicharger-jlcpcb/Multicharger-jlcpcb.kicad_pcb (KiCad board)
At the start: 2 copper layers, 48.3 x 43.2 mm, 26 parts, among them J101 Conn_01x02, J102 Conn_01x02, J103 Tagbase, J104 USB_B_Mini, SW101 SW_DIP_x04, U101 TPS3700, U106 XC6206-3.3V

Commit message: complete JLCPCB multicharger
Parts:
- added R2: spare, Resistor_SMD:R_0603_1608Metric_Pad0.98x0.95mm_HandSolder, F.Cu at (136.2, 67.0)
Connections:
- SW101 pad 4: unconnected-(SW101-Pad4) -> Net-(SW101-Pad4)
- SW101 pad 5: unconnected-(SW101-Pad5) -> TAG_VBAT
Routing:
- net TAG_VBAT: track 32.0 -> 51.2 mm
- net +3V3: track 23.6 -> 34.4 mm
- net /VIN: track 105.8 -> 112.8 mm
- net Net-(SW101-Pad4): track 0.00 -> 3.85 mm
- net GND: track 32.0 -> 35.0 mm, vias 7 -> 9
- net Net-(R106-Pad1): track 1.80 -> 3.99 mm
- net Net-(R107-Pad1): track 1.80 -> 3.99 mm
- net Net-(R1-Pad1): track 1.80 -> 3.99 mm
Other:
- board text added: "NC"
