File: hardware/Multicharger-jlcpcb/Multicharger-jlcpcb.kicad_pcb (KiCad board)
At the start: 2 copper layers, 48.3 x 43.2 mm, 27 parts, among them J101 Conn_01x02, J102 Conn_01x02, J103 Tagbase, J104 USB_B_Mini, SW101 SW_DIP_x04, U101 TPS3700, U106 XC6206-3.3V

Commit message: updated jlcpcb multicharger
Parts:
- added D105: D_Schottky, Diode_SMD:D_SOD-323, F.Cu at (132.2, 70.5)
- D101: value No Go -> No Go Red
- D102: value LED -> BLUE
- D103: value Go -> Go Green
- D104: value D -> D_Schottky; footprint Diode_SMD:D_0402_1005Metric -> Diode_SMD:D_SOD-323
- R1: value 620 -> 680
- R101: value 1.2K -> 220
- R102, R105: value 1.2K -> 120
- R103: value 910K -> 91K; footprint Resistor_SMD:R_0402_1005Metric -> Resistor_SMD:R_0603_1608Metric
- R104: value 130K -> 13K; footprint Resistor_SMD:R_0402_1005Metric -> Resistor_SMD:R_0603_1608Metric
- R106: footprint Resistor_SMD:R_0402_1005Metric -> Resistor_SMD:R_0603_1608Metric
- R107: value 2000 -> 2.2K; footprint Resistor_SMD:R_0402_1005Metric -> Resistor_SMD:R_0603_1608Metric
- moved D104 3.98 mm to (132.2, 72.8), turned to 180 degrees
- moved U106 3.71 mm to (136.1, 72.2)
- moved R101 3.22 mm to (123.2, 82.8)
- moved C106 2.69 mm to (134.9, 74.5)
- moved C107 2.20 mm to (136.8, 69.8), turned to 180 degrees
- moved R104 1.98 mm to (135.4, 81.2)
- moved D101 1.60 mm to (123.2, 81.0), turned to 0 degrees
- moved R103 0.66 mm to (135.6, 77.7)
- moved R106 0.31 mm to (131.8, 66.7)
- moved R1 0.15 mm to (129.5, 66.7)
Connections:
- C106 pad 1: /VIN -> Net-(C106-Pad1)
- U106 pad 3: /VIN -> Net-(C106-Pad1)
Routing:
- net Net-(C106-Pad1): track 0.00 -> 5.00 mm
- net +3V3: track 34.0 -> 30.5 mm
- net Net-(R101-Pad1): track 6.19 -> 9.15 mm
- net /Vsense: track 4.41 -> 6.70 mm
- net GND: track 35.0 -> 36.7 mm
- net /VIN: track 112.8 -> 111.2 mm
- net Net-(J104-Pad1): track 4.48 -> 5.93 mm
Other:
- board text added: "2.2K"
- board text added: "680"
- board text added: "BitTag Charger V5.1"
- board text added: "Geoffrey Brown 7/9/2023"
- board text added: "MS920 = 680 MS621 = 680 MS518 = 1.5K MS414 = 2.2K"
- board text removed: "2K"
- board text removed: "620"
- board text removed: "BitTag Charger V5"
- board text removed: "Geoffrey Brown 6/3/2023"
- board text removed: "MS920 = 620 MS621 = 620 MS518 = 1.5K MS414 = 2K"

Commit message: update multicharger
Parts:
- removed D105: D_Schottky, Diode_SMD:D_SOD-323
- U106: value XC6206-3.3V -> AP7370
- moved D104 0.82 mm to (132.3, 72.0), turned to 90 degrees
Connections:
- C106 pad 1: Net-(C106-Pad1) -> /VIN
- U106 pad 3: Net-(C106-Pad1) -> /VIN
Routing:
- net /VIN: track 111.2 -> 117.2 mm
- net Net-(C106-Pad1): track 5.00 -> 0.00 mm
- net Net-(D104-Pad2): track 5.93 -> 6.88 mm

Commit message: update multicharger resistors
Parts:
- R101: value 220 -> 330
- R102, R105: value 120 -> 220
Changed lines of the file:
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@@
     (descr "Resistor SMD 0603 (1608 Metric), square (rectangular) end terminal, IPC_7351 nominal, (Body size source: IPC-SM-782 page 72, https://www.pcb-3d.com/wordpress/wp-content/uploads/ipc-sm-782a_amendment_1_and_2.pdf), generated with kicad-footprint-generator")
     (tags "resistor")
-    (property "Description" "100mW Thick Film Resistors ±100ppm/℃ ±1% 120Ω 0603 ")
-    (property "LCSC" "C22787")
+    (property "Description" "100mW Thick Film Resistors ±100ppm/℃ ±1% 220Ω 0603 ")
+    (property "LCSC" "C22962")
     (property "MFN" "Uniroyal")
-    (property "MPN" "0603WAF1200T5E")
+    (property "MPN" "0603WAF2200T5E")
     (property "Sheetfile" "Multicharger-jlcpcb.kicad_sch")
     (property "Sheetname" "")
@@
       (effects (font (size 1 1) (thickness 0.15)))
     )
-    (fp_text value "120" (at 0 1.43 -90) (layer "F.Fab")
+    (fp_text value "220" (at 0 1.43 -90) (layer "F.Fab")
       (effects (font (size 1 1) (thickness 0.15)))
     )
@@
     (descr "Resistor SMD 0603 (1608 Metric), square (rectangular) end terminal, IPC_7351 nominal, (Body size source: IPC-SM-782 page 72, https://www.pcb-3d.com/wordpress/wp-content/uploads/ipc-sm-782a_amendment_1_and_2.pdf), generated with kicad-footprint-generator")
     (tags "resistor")
-    (property "Description" "100mW Thick Film Resistors ±100ppm/℃ ±1% 129Ω 0603 ")
-    (property "LCSC" "C22787")
+    (property "Description" "100mW Thick Film Resistors ±100ppm/℃ ±1% 220Ω 0603 ")
+    (property "LCSC" "C22962")
     (property "LCSCC" "")
     (property "MFN" "Uniroyal")
-    (property "MPN" "0603WAF1200T5E")
+    (property "MPN" "0603WAF2200T5E")
     (property "Sheetfile" "Multicharger-jlcpcb.kicad_sch")
     (property "Sheetname" "")
@@
       (effects (font (size 1 1) (thickness 0.15)))
     )
-    (fp_text value "120" (at 0 1.43 180) (layer "F.Fab")
+    (fp_text value "220" (at 0 1.43 180) (layer "F.Fab")
       (effects (font (size 1 1) (thickness 0.15)))
     )
@@
     (descr "Resistor SMD 0603 (1608 Metric), square (rectangular) end terminal, IPC_7351 nominal, (Body size source: IPC-SM-782 page 72, https://www.pcb-3d.com/wordpress/wp-content/uploads/ipc-sm-782a_amendment_1_and_2.pdf), generated with kicad-footprint-generator")
     (tags "resistor")
-    (property "Description" "100mW Thick Film Resistors ±100ppm/℃ ±1% 220Ω 0603 ")
-    (property "LCSC" "C22962")
+    (property "Description" "100mW Thick Film Resistors ±100ppm/℃ ±1% 330Ω 0603 Chip")
+    (property "LCSC" "C23138")
     (property "MFN" "Uniroyal")
-    (property "MPN" "0603WAF2200T5E")
+    (property "MPN" "0603WAF3300T5E")
     (property "Sheetfile" "Multicharger-jlcpcb.kicad_sch")
     (property "Sheetname" "")
@@
       (effects (font (size 1 1) (thickness 0.15)))
     )
-    (fp_text value "220" (at 0 1.43 180) (layer "F.Fab")
-      (effects (font (size 1 1) (thickness 0.15)))
-    )
+    (fp_text value "330" (at 0 1.43 180) (layer "F.Fab")
+      (effects (font (size 1 1) (thickness 0.15)))
+    )
