File: hardware/Multicharger-jlcpcb/Multicharger-jlcpcb.kicad_sch (KiCad schematic)
At the start: 26 parts, among them J101 Conn_01x02, J102 Conn_01x02, J103 Tagbase, J104 USB_B_Mini, SW101 SW_DIP_x04, U101 TPS3700, U106 XC6206-3.3V

Commit message: complete JLCPCB multicharger
Parts:
- added R2: spare, Resistor_SMD:R_0603_1608Metric_Pad0.98x0.95mm_HandSolder, symbol Device:R
- J101, J102, J103, MK101, MK102, MK103, MK104: now left out of the parts list
- J104: LCSC (none) -> C2681563; MFN (none) -> SHOU HAN; MPN (none) -> MINI 5PTP
Connections:
- net +3V3: now also R2.1
- net TAG_VBAT: now also SW101.5
- net at SW101.4: now also R2.2
- no-connect marks 7 -> 5
Changed lines of the file:
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@@
   (junction (at 114.3 146.05) (diameter 0) (color 0 0 0 0)
   )
+  (junction (at 76.2 99.06) (diameter 0) (color 0 0 0 0)
+  )
   (junction (at 111.76 96.52) (diameter 0) (color 0 0 0 0)
   )
   (junction (at 147.32 41.91) (diameter 0) (color 0 0 0 0)
+  )
+  (junction (at 111.76 99.06) (diameter 0) (color 0 0 0 0)
   )
   (junction (at 76.2 96.52) (diameter 0) (color 0 0 0 0)
@@
   (no_connect (at 86.36 55.88))
   (no_connect (at 167.64 148.59))
-  (no_connect (at 91.44 101.6))
   (no_connect (at 86.36 53.34))
   (no_connect (at 180.34 148.59))
-  (no_connect (at 106.045 101.6))
   (wire (pts (xy 147.32 36.83) (xy 147.32 41.91))
     (stroke (width 0) (type default) (color 0 0 0 0))
@@
     (stroke (width 0) (type default) (color 0 0 0 0))
   )
+  (wire (pts (xy 106.68 101.6) (xy 111.76 101.6))
+    (stroke (width 0) (type default) (color 0 0 0 0))
+  )
   (wire (pts (xy 114.3 148.59) (xy 118.11 148.59))
     (stroke (width 0) (type default) (color 0 0 0 0))
@@
     (stroke (width 0) (type default) (color 0 0 0 0))
   )
+  (wire (pts (xy 111.76 101.6) (xy 111.76 99.06))
+    (stroke (width 0) (type default) (color 0 0 0 0))
+  )
   (wire (pts (xy 140.97 41.91) (xy 147.32 41.91))
     (stroke (width 0) (type default) (color 0 0 0 0))
   )
+  (wire (pts (xy 87.63 101.6) (xy 91.44 101.6))
+    (stroke (width 0) (type default) (color 0 0 0 0))
+  )
   (wire (pts (xy 88.9 48.26) (xy 86.36 48.26))
     (stroke (width 0) (type default) (color 0 0 0 0))
@@
     (stroke (width 0) (type default) (color 0 0 0 0))
   )
+  (wire (pts (xy 76.2 99.06) (xy 76.2 101.6))
+    (stroke (width 0) (type default) (color 0 0 0 0))
+  )
   (wire (pts (xy 87.63 99.06) (xy 91.44 99.06))
     (stroke (width 0) (type default) (color 0 0 0 0))
@@
   )
   (wire (pts (xy 218.44 73.66) (xy 218.44 76.2))
+    (stroke (width 0) (type default) (color 0 0 0 0))
+  )
+  (wire (pts (xy 76.2 101.6) (xy 80.01 101.6))
     (stroke (width 0) (type default) (color 0 0 0 0))
   )
@@
       (effects (font (size 1.27 1.27)) hide)
     )
-    (property "MFN" "" (id 4) (at 78.74 53.34 0)
-      (effects (font (size 1.524 1.524)) hide)
-    )
-    (property "MPN" "" (id 5) (at 78.74 53.34 0)
-      (effects (font (size 1.524 1.524)) hide)
-    )
-    (property "Digikey" "" (id 6) (at 78.74 53.34 0)
+    (property "MFN" "SHOU HAN" (id 4) (at 78.74 53.34 0)
+      (effects (font (size 1.524 1.524)) hide)
+    )
+    (property "MPN" "MINI 5PTP" (id 5) (at 78.74 53.34 0)
+      (effects (font (size 1.524 1.524)) hide)
+    )
+    (property "LCSC" "C2681563" (id 6) (at 78.74 53.34 0)
       (effects (font (size 1.524 1.524)) hide)
     )
@@
   )
   (symbol (lib_id "Connector_Generic:Conn_02x03_Odd_Even") (at 172.72 148.59 0) (mirror x) (unit 1)
-    (in_bom yes) (on_board yes)
+    (in_bom no) (on_board yes)
     (property "Reference" "J103" (id 0) (at 173.99 153.67 0))
     (property "Value" "Tagbase" (id 1) (at 173.99 143.51 0))
@@
     )
     (property "Value" "GND" (id 1) (at 133.35 58.42 0))
-    (property "Footprint" "" (id 2) (at 133.35 54.61 0))
-    (property "Datasheet" "" (id 3) (at 133.35 54.61 0))
+    (property "Footprint" "" (id 2) (at 133.35 54.61 0)
+      (effects (font (size 1.27 1.27)) hide)
+    )
+    (property "Datasheet" "" (id 3) (at 133.35 54.61 0)
+      (effects (font (size 1.27 1.27)) hide)
+    )
     (pin "1")
   )
@@
     )
     (property "Value" "+3V3" (id 1) (at 147.32 33.274 0))
-    (property "Footprint" "" (id 2) (at 147.32 36.83 0))
-    (property "Datasheet" "" (id 3) (at 147.32 36.83 0))
+    (property "Footprint" "" (id 2) (at 147.32 36.83 0)
+      (effects (font (size 1.27 1.27)) hide)
+    )
+    (property "Datasheet" "" (id 3) (at 147.32 36.83 0)
+      (effects (font (size 1.27 1.27)) hide)
+    )
     (pin "1")
   )
   (symbol (lib_id "Mechanical:MountingHole") (at 36.83 191.77 0) (unit 1)
-    (in_bom yes) (on_board yes)
+    (in_bom no) (on_board yes)
     (property "Reference" "MK101" (id 0) (at 36.83 186.69 0))
     (property "Value" "Mounting_Hole" (id 1) (at 36.83 188.595 0))
@@
   )
   (symbol (lib_id "Mechanical:MountingHole") (at 53.34 191.77 0) (unit 1)
-    (in_bom yes) (on_board yes)
+    (in_bom no) (on_board yes)
     (property "Reference" "MK102" (id 0) (at 53.34 186.69 0))
     (property "Value" "Mounting_Hole" (id 1) (at 53.34 188.595 0))
@@
   )
   (symbol (lib_id "Mechanical:MountingHole") (at 68.58 191.77 0) (unit 1)
-    (in_bom yes) (on_board yes)
+    (in_bom no) (on_board yes)
     (property "Reference" "MK103" (id 0) (at 68.58 186.69 0))
     (property "Value" "Mounting_Hole" (id 1) (at 68.58 188.595 0))
@@
   )
   (symbol (lib_id "Mechanical:MountingHole") (at 82.55 191.77 0) (unit 1)
-    (in_bom yes) (on_board yes)
+    (in_bom no) (on_board yes)
     (property "Reference" "MK104" (id 0) (at 82.55 186.69 0))
     (property "Value" "Mounting_Hole" (id 1) (at 82.55 188.595 0))
@@
     )
     (property "Value" "+3V3" (id 1) (at 160.02 141.224 0))
-    (property "Footprint" "" (id 2) (at 160.02 144.78 0))
-    (property "Datasheet" "" (id 3) (at 160.02 144.78 0))
+    (property "Footprint" "" (id 2) (at 160.02 144.78 0)
+      (effects (font (size 1.27 1.27)) hide)
+    )
+    (property "Datasheet" "" (id 3) (at 160.02 144.78 0)
+      (effects (font (size 1.27 1.27)) hide)
+    )
     (pin "1")
   )
@@
     )
     (property "Value" "GND" (id 1) (at 116.84 120.65 0))
-    (property "Footprint" "" (id 2) (at 116.84 116.84 0))
-    (property "Datasheet" "" (id 3) (at 116.84 116.84 0))
+    (property "Footprint" "" (id 2) (at 116.84 116.84 0)
+      (effects (font (size 1.27 1.27)) hide)
+    )
+    (property "Datasheet" "" (id 3) (at 116.84 116.84 0)
+      (effects (font (size 1.27 1.27)) hide)
+    )
     (pin "1")
   )
@@
   )
   (symbol (lib_id "Connector_Generic:Conn_01x02") (at 123.19 146.05 0) (unit 1)
-    (in_bom yes) (on_board yes)
+    (in_bom no) (on_board yes)
     (property "Reference" "J102" (id 0) (at 123.19 143.51 0)
       (effects (font (size 1.27 1.27)) (justify left))
@@
   )
   (symbol (lib_id "Connector_Generic:Conn_01x02") (at 104.14 146.05 0) (mirror y) (unit 1)
-    (in_bom yes) (on_board yes)
+    (in_bom no) (on_board yes)
     (property "Reference" "J101" (id 0) (at 104.14 143.51 0))
     (property "Value" "Conn_01x02" (id 1) (at 106.172 142.8496 0)
@@
     )
     (property "Value" "GND" (id 1) (at 114.3 154.94 0))
-    (property "Footprint" "" (id 2) (at 114.3 151.13 0))
-    (property "Datasheet" "" (id 3) (at 114.3 151.13 0))
+    (property "Footprint" "" (id 2) (at 114.3 151.13 0)
+      (effects (font (size 1.27 1.27)) hide)
+    )
+    (property "Datasheet" "" (id 3) (at 114.3 151.13 0)
+      (effects (font (size 1.27 1.27)) hide)
+    )
     (pin "1")
   )
@@
       (effects (font (size 1.27 1.27)) hide)
     )
-    (property "LCSC" "C2837790" (id 6) (at 96.52 41.91 0)
+    (property "LCSC" "C2837790" (id 7) (at 96.52 41.91 0)
       (effects (font (size 1.524 1.524)) hide)
     )
@@
     )
     (property "Value" "+3V3" (id 1) (at 76.2 89.154 0))
-    (property "Footprint" "" (id 2) (at 76.2 92.71 0))
-    (property "Datasheet" "" (id 3) (at 76.2 92.71 0))
+    (property "Footprint" "" (id 2) (at 76.2 92.71 0)
+      (effects (font (size 1.27 1.27)) hide)
+    )
+    (property "Datasheet" "" (id 3) (at 76.2 92.71 0)
+      (effects (font (size 1.27 1.27)) hide)
+    )
     (pin "1")
   )
@@
       (effects (font (size 1.27 1.27)) hide)
     )
-    (property "LSCS" "" (id 7) (at 99.06 99.06 0)
+    (property "LSCS" "" (id 8) (at 99.06 99.06 0)
       (effects (font (size 1.524 1.524)) hide)
     )
@@
     (pin "8")
   )
+  (symbol (lib_id "Device:R") (at 83.82 101.6 90) (unit 1)
+    (in_bom no) (on_board yes)
+    (property "Reference" "R2" (id 0) (at 88.265 100.33 90))
+    (property "Value" "spare" (id 1) (at 83.82 101.6 90))
+    (property "Footprint" "Resistor_SMD:R_0603_1608Metric_Pad0.98x0.95mm_HandSolder" (id 2) (at 83.82 103.378 90)
+      (effects (font (size 1.27 1.27)) hide)
+    )
+    (property "Datasheet" "~" (id 3) (at 83.82 101.6 0)
+      (effects (font (size 1.27 1.27)) hide)
+    )
+    (pin "1")
+    (pin "2")
+  )
   (sheet_instances
     (path "/" (page "1"))
@@
       (reference "R1") (unit 1) (value "620") (footprint "Resistor_SMD:R_0402_1005Metric")
     )
+    (path "/baf4555a-bd5b-4a25-8eda-5a3973cc2df0"
+      (reference "R2") (unit 1) (value "spare") (footprint "Resistor_SMD:R_0603_1608Metric_Pad0.98x0.95mm_HandSolder")
+    )
     (path "/00000000-0000-0000-0000-00005b72d71f"

Commit message: convert multicharger for jlcpcb
Parts:
- D104: LCSC C2837790 -> C191023; MFN Rohm -> Guangdong Hottech; MPN RB161QS-40T18R -> 1N5819WS
- R1: footprint Resistor_SMD:R_0402_1005Metric -> Resistor_SMD:R_0603_1608Metric; LCSC C445593 -> C191023; MFN Panasonic Electronic -> Uniroyal; MPN ERA2AEB621X -> 0603WAF6200T5E
- R101, R102, R105: value 1K -> 1.2K; footprint Resistor_SMD:R_0402_1005Metric -> Resistor_SMD:R_0603_1608Metric; LCSC C279981 -> C21189; MFN Viking Tech -> Uniroyal; MPN CR-02FL6----1K -> 0603WAF0000T5E
- R103: Digikey YAG3257CT-ND -> (none); MPN RC0402FR-07910KL -> FRC0603J914TS
- R104: Digikey YAG2969CT-ND -> (none); MPN RC0402FR-07130KL -> RC0402FR-07910KL
- U106: JlcRotOffset (none) -> 180
Changed lines of the file:
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@@
     (in_bom yes) (on_board yes)
     (property "Reference" "R102" (id 0) (at 96.52 50.292 90))
-    (property "Value" "1K" (id 1) (at 96.52 48.26 90))
-    (property "Footprint" "Resistor_SMD:R_0402_1005Metric" (id 2) (at 96.52 46.482 90)
+    (property "Value" "1.2K" (id 1) (at 96.52 48.26 90))
+    (property "Footprint" "Resistor_SMD:R_0603_1608Metric" (id 2) (at 96.52 46.482 90)
       (effects (font (size 1.27 1.27)) hide)
     )
@@
       (effects (font (size 1.27 1.27)) hide)
     )
-    (property "MPN" "CR-02FL6----1K" (id 4) (at 96.52 48.26 90)
-      (effects (font (size 1.27 1.27)) hide)
-    )
-    (property "MFN" "Viking Tech" (id 6) (at 96.52 48.26 0)
-      (effects (font (size 1.27 1.27)) hide)
-    )
-    (property "Description" "RES SMD 1K OHM 5% 1/16W 0402" (id 7) (at 96.52 48.26 0)
-      (effects (font (size 1.27 1.27)) hide)
-    )
-    (property "LCSC" "C279981" (id 8) (at 96.52 48.26 90)
+    (property "MPN" "0603WAF0000T5E" (id 4) (at 96.52 48.26 90)
+      (effects (font (size 1.27 1.27)) hide)
+    )
+    (property "MFN" "Uniroyal" (id 6) (at 96.52 48.26 0)
+      (effects (font (size 1.27 1.27)) hide)
+    )
+    (property "Description" "RES SMD 1.2K OHM 5% 1/16W " (id 7) (at 96.52 48.26 0)
+      (effects (font (size 1.27 1.27)) hide)
+    )
+    (property "LCSC" "C21189" (id 8) (at 96.52 48.26 90)
       (effects (font (size 1.524 1.524)) hide)
     )
@@
     (property "LCSC" "C2891841" (id 8) (at 133.35 41.91 0)
       (effects (font (size 1.27 1.27)) hide)
+    )
+    (property "JlcRotOffset" "180" (id 8) (at 133.35 41.91 0)
+      (effects (font (size 1.524 1.524)) hide)
     )
     (pin "1")
@@
     (property "Reference" "R1" (id 0) (at 88.9 92.71 90))
     (property "Value" "620" (id 1) (at 83.82 93.98 90))
-    (property "Footprint" "Resistor_SMD:R_0402_1005Metric" (id 2) (at 83.82 93.98 0)
+    (property "Footprint" "Resistor_SMD:R_0603_1608Metric" (id 2) (at 83.82 93.98 0)
       (effects (font (size 1.27 1.27)) hide)
     )
@@
       (effects (font (size 1.27 1.27)) hide)
     )
-    (property "MPN" "ERA2AEB621X" (id 4) (at 83.82 93.98 90)
+    (property "MPN" "0603WAF6200T5E" (id 4) (at 83.82 93.98 90)
       (effects (font (size 1.27 1.27)) hide)
     )
@@
       (effects (font (size 1.27 1.27)) hide)
     )
-    (property "MFN" "Panasonic Electronic" (id 6) (at 83.82 93.98 0)
-      (effects (font (size 1.27 1.27)) hide)
-    )
-    (property "Description" "RES SMD 620 OHM 5% 1/10W 0402" (id 7) (at 83.82 93.98 0)
-      (effects (font (size 1.27 1.27)) hide)
-    )
-    (property "LCSC" "C445593" (id 8) (at 83.82 93.98 0)
+    (property "MFN" "Uniroyal" (id 6) (at 83.82 93.98 0)
+      (effects (font (size 1.27 1.27)) hide)
+    )
+    (property "LCSC" "C191023" (id 8) (at 83.82 93.98 0)
       (effects (font (size 1.27 1.27)) hide)
     )
@@
       (effects (font (size 1.27 1.27)) hide)
     )
-    (property "MPN" "RC0402FR-07910KL" (id 4) (at 116.84 100.33 90)
-      (effects (font (size 1.524 1.524)) hide)
-    )
-    (property "Digikey" "YAG3257CT-ND" (id 5) (at 116.84 100.33 0)
+    (property "MPN" "FRC0603J914TS" (id 4) (at 116.84 100.33 90)
+      (effects (font (size 1.524 1.524)) hide)
+    )
+    (property "Digikey" "" (id 5) (at 116.84 100.33 0)
       (effects (font (size 1.27 1.27)) hide)
     )
@@
       (effects (font (size 1.27 1.27)) hide)
     )
-    (property "Description" "RES SMD 910K OHM 1% 1/16W 0402" (id 7) (at 116.84 100.33 0)
+    (property "Description" "RES SMD 910K OHM 1% 1/16W " (id 7) (at 116.84 100.33 0)
       (effects (font (size 1.27 1.27)) hide)
     )
@@
       (effects (font (size 1.27 1.27)) hide)
     )
-    (property "MPN" "RC0402FR-07130KL" (id 4) (at 116.84 110.49 90)
-      (effects (font (size 1.524 1.524)) hide)
-    )
-    (property "Digikey" "YAG2969CT-ND" (id 5) (at 116.84 110.49 0)
+    (property "MPN" "RC0402FR-07910KL" (id 4) (at 116.84 110.49 90)
+      (effects (font (size 1.524 1.524)) hide)
+    )
+    (property "Digikey" "" (id 5) (at 116.84 110.49 0)
       (effects (font (size 1.27 1.27)) hide)
     )
@@
       (effects (font (size 1.27 1.27)) hide)
     )
-    (property "Description" "RES SMD 130K OHM 1% 1/16W 0402" (id 7) (at 116.84 110.49 0)
+    (property "Description" "RES SMD 130K OHM 1% 1/16W " (id 7) (at 116.84 110.49 0)
       (effects (font (size 1.27 1.27)) hide)
     )
@@
     (in_bom yes) (on_board yes)
     (property "Reference" "R105" (id 0) (at 226.568 92.71 90))
-    (property "Value" "1K" (id 1) (at 228.6 92.71 90))
-    (property "Footprint" "Resistor_SMD:R_0402_1005Metric" (id 2) (at 230.378 92.71 90)
+    (property "Value" "1.2K" (id 1) (at 228.6 92.71 90))
+    (property "Footprint" "Resistor_SMD:R_0603_1608Metric" (id 2) (at 230.378 92.71 90)
       (effects (font (size 1.27 1.27)) hide)
     )
@@
       (effects (font (size 1.27 1.27)) hide)
     )
-    (property "MPN" "CR-02FL6----1K" (id 4) (at 228.6 92.71 90)
-      (effects (font (size 1.27 1.27)) hide)
-    )
-    (property "MFN" "Viking Tech" (id 6) (at 228.6 92.71 0)
-      (effects (font (size 1.27 1.27)) hide)
-    )
-    (property "Description" "RES SMD 1K OHM 5% 1/16W 0402" (id 7) (at 228.6 92.71 0)
+    (property "MPN" "0603WAF0000T5E" (id 4) (at 228.6 92.71 90)
+      (effects (font (size 1.27 1.27)) hide)
+    )
+    (property "MFN" "Uniroyal" (id 6) (at 228.6 92.71 0)
+      (effects (font (size 1.27 1.27)) hide)
+    )
+    (property "Description" "RES SMD 1.2K OHM 5% 1/16W " (id 7) (at 228.6 92.71 0)
       (effects (font (size 1.27 1.27)) hide)
     )
@@
       (effects (font (size 1.524 1.524)) hide)
     )
-    (property "LCSC" "C279981" (id 9) (at 228.6 92.71 0)
+    (property "LCSC" "C21189" (id 9) (at 228.6 92.71 0)
       (effects (font (size 1.27 1.27)) hide)
     )
@@
     (in_bom yes) (on_board yes)
     (property "Reference" "R101" (id 0) (at 216.408 92.71 90))
-    (property "Value" "1K" (id 1) (at 218.44 92.71 90))
-    (property "Footprint" "Resistor_SMD:R_0402_1005Metric" (id 2) (at 220.218 92.71 90)
+    (property "Value" "1.2K" (id 1) (at 218.44 92.71 90))
+    (property "Footprint" "Resistor_SMD:R_0603_1608Metric" (id 2) (at 220.218 92.71 90)
       (effects (font (size 1.27 1.27)) hide)
     )
@@
       (effects (font (size 1.27 1.27)) hide)
     )
-    (property "MPN" "CR-02FL6----1K" (id 4) (at 218.44 92.71 90)
-      (effects (font (size 1.27 1.27)) hide)
-    )
-    (property "MFN" "Viking Tech" (id 6) (at 218.44 92.71 0)
-      (effects (font (size 1.27 1.27)) hide)
-    )
-    (property "Description" "RES SMD 1K OHM 5% 1/16W 0402" (id 7) (at 218.44 92.71 0)
-      (effects (font (size 1.27 1.27)) hide)
-    )
-    (property "LCSC" "C279981" (id 8) (at 218.44 92.71 90)
+    (property "MPN" "0603WAF0000T5E" (id 4) (at 218.44 92.71 90)
+      (effects (font (size 1.27 1.27)) hide)
+    )
+    (property "MFN" "Uniroyal" (id 6) (at 218.44 92.71 0)
+      (effects (font (size 1.27 1.27)) hide)
+    )
+    (property "Description" "RES SMD 1.2K OHM 5% 1/16W " (id 7) (at 218.44 92.71 0)
+      (effects (font (size 1.27 1.27)) hide)
+    )
+    (property "LCSC" "C21189" (id 8) (at 218.44 92.71 90)
       (effects (font (size 1.524 1.524)) hide)
     )
@@
       (effects (font (size 1.27 1.27)) hide)
     )
-    (property "MPN" "RB161QS-40T18R" (id 4) (at 96.52 41.91 90)
-      (effects (font (size 1.27 1.27)) hide)
-    )
-    (property "MFN" "Rohm" (id 6) (at 96.52 41.91 0)
-      (effects (font (size 1.27 1.27)) hide)
-    )
-    (property "LCSC" "C2837790" (id 7) (at 96.52 41.91 0)
+    (property "MPN" "1N5819WS" (id 4) (at 96.52 41.91 90)
+      (effects (font (size 1.27 1.27)) hide)
+    )
+    (property "MFN" "Guangdong Hottech" (id 6) (at 96.52 41.91 0)
+      (effects (font (size 1.27 1.27)) hide)
+    )
+    (property "LCSC" "C191023" (id 7) (at 96.52 41.91 0)
       (effects (font (size 1.524 1.524)) hide)
     )
@@
       (effects (font (size 1.524 1.524)) hide)
     )
-    (property "LCSC" "C3034155" (id 8) (at 99.06 99.06 0)
+    (property "LCSC" "C3034155" (id 9) (at 99.06 99.06 0)
       (effects (font (size 1.27 1.27)) hide)
     )
@@
     )
     (path "/00000000-0000-0000-0000-00005b721820"
-      (reference "R1") (unit 1) (value "620") (footprint "Resistor_SMD:R_0402_1005Metric")
+      (reference "R1") (unit 1) (value "620") (footprint "Resistor_SMD:R_0603_1608Metric")
     )
     (path "/baf4555a-bd5b-4a25-8eda-5a3973cc2df0"
@@
     )
     (path "/00000000-0000-0000-0000-00005b72d71f"
-      (reference "R101") (unit 1) (value "1K") (footprint "Resistor_SMD:R_0402_1005Metric")
+      (reference "R101") (unit 1) (value "1.2K") (footprint "Resistor_SMD:R_0603_1608Metric")
     )
     (path "/00000000-0000-0000-0000-00005b06b8b2"
-      (reference "R102") (unit 1) (value "1K") (footprint "Resistor_SMD:R_0402_1005Metric")
+      (reference "R102") (unit 1) (value "1.2K") (footprint "Resistor_SMD:R_0603_1608Metric")
     )
     (path "/00000000-0000-0000-0000-00005b72cf14"
@@
     )
     (path "/00000000-0000-0000-0000-00005b72d633"
-      (reference "R105") (unit 1) (value "1K") (footprint "Resistor_SMD:R_0402_1005Metric")
+      (reference "R105") (unit 1) (value "1.2K") (footprint "Resistor_SMD:R_0603_1608Metric")
     )
     (path "/00000000-0000-0000-0000-00006111918b"

Commit message: remove voltage shutdown from BitTag
Parts:
- D104: LCSC C191023 -> C2837790; MFN Guangdong Hottech -> Rohm; MPN 1N5819WS -> RB161QS-40T18R JLCPCB Part #
- R1: LCSC C191023 -> C23220
Changed lines of the file:
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@@
       (effects (font (size 1.27 1.27)) hide)
     )
-    (property "JlcRotOffset" "180" (id 8) (at 133.35 41.91 0)
+    (property "JlcRotOffset" "180" (id 9) (at 133.35 41.91 0)
       (effects (font (size 1.524 1.524)) hide)
     )
@@
       (effects (font (size 1.27 1.27)) hide)
     )
-    (property "LCSC" "C191023" (id 8) (at 83.82 93.98 0)
+    (property "LCSC" "C23220" (id 8) (at 83.82 93.98 0)
       (effects (font (size 1.27 1.27)) hide)
     )
@@
       (effects (font (size 1.27 1.27)) hide)
     )
-    (property "MPN" "1N5819WS" (id 4) (at 96.52 41.91 90)
-      (effects (font (size 1.27 1.27)) hide)
-    )
-    (property "MFN" "Guangdong Hottech" (id 6) (at 96.52 41.91 0)
-      (effects (font (size 1.27 1.27)) hide)
-    )
-    (property "LCSC" "C191023" (id 7) (at 96.52 41.91 0)
-      (effects (font (size 1.524 1.524)) hide)
-    )
+    (property "MPN" "RB161QS-40T18R JLCPCB Part # " (id 4) (at 96.52 41.91 90)
+      (effects (font (size 1.27 1.27)) hide)
+    )
+    (property "MFN" "Rohm" (id 6) (at 96.52 41.91 0)
+      (effects (font (size 1.27 1.27)) hide)
+    )
+    (property "LCSC" "C2837790" (id 7) (at 96.52 41.91 0)
+      (effects (font (size 1.524 1.524)) hide)
+    )

Commit message: correct multicharger load resistor part numbers
Parts:
- R101, R102, R105: LCSC C21189 -> C114605; MFN Uniroyal -> Yaego; MPN 0603WAF0000T5E -> RC0603FR-071K2L
Changed lines of the file:
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@@
       (effects (font (size 1.27 1.27)) hide)
     )
-    (property "MPN" "0603WAF0000T5E" (id 4) (at 96.52 48.26 90)
-      (effects (font (size 1.27 1.27)) hide)
-    )
-    (property "MFN" "Uniroyal" (id 6) (at 96.52 48.26 0)
+    (property "MPN" "RC0603FR-071K2L" (id 4) (at 96.52 48.26 90)
+      (effects (font (size 1.27 1.27)) hide)
+    )
+    (property "MFN" "Yaego" (id 6) (at 96.52 48.26 0)
       (effects (font (size 1.27 1.27)) hide)
     )
@@
       (effects (font (size 1.27 1.27)) hide)
     )
-    (property "LCSC" "C21189" (id 8) (at 96.52 48.26 90)
+    (property "LCSC" "C114605" (id 8) (at 96.52 48.26 90)
       (effects (font (size 1.524 1.524)) hide)
     )
@@
       (effects (font (size 1.27 1.27)) hide)
     )
-    (property "MPN" "0603WAF0000T5E" (id 4) (at 228.6 92.71 90)
-      (effects (font (size 1.27 1.27)) hide)
-    )
-    (property "MFN" "Uniroyal" (id 6) (at 228.6 92.71 0)
+    (property "MPN" "RC0603FR-071K2L" (id 4) (at 228.6 92.71 90)
+      (effects (font (size 1.27 1.27)) hide)
+    )
+    (property "MFN" "Yaego" (id 6) (at 228.6 92.71 0)
       (effects (font (size 1.27 1.27)) hide)
     )
@@
       (effects (font (size 1.524 1.524)) hide)
     )
-    (property "LCSC" "C21189" (id 9) (at 228.6 92.71 0)
+    (property "LCSC" "C114605" (id 9) (at 228.6 92.71 0)
       (effects (font (size 1.27 1.27)) hide)
     )
@@
       (effects (font (size 1.27 1.27)) hide)
     )
-    (property "MPN" "0603WAF0000T5E" (id 4) (at 218.44 92.71 90)
-      (effects (font (size 1.27 1.27)) hide)
-    )
-    (property "MFN" "Uniroyal" (id 6) (at 218.44 92.71 0)
+    (property "MPN" "RC0603FR-071K2L" (id 4) (at 218.44 92.71 90)
+      (effects (font (size 1.27 1.27)) hide)
+    )
+    (property "MFN" "Yaego" (id 6) (at 218.44 92.71 0)
       (effects (font (size 1.27 1.27)) hide)
     )
@@
       (effects (font (size 1.27 1.27)) hide)
     )
-    (property "LCSC" "C21189" (id 8) (at 218.44 92.71 90)
-      (effects (font (size 1.524 1.524)) hide)
-    )
+    (property "LCSC" "C114605" (id 8) (at 218.44 92.71 90)
+      (effects (font (size 1.524 1.524)) hide)
+    )
