File: hardware/Multicharger-jlcpcb/Multicharger-jlcpcb.kicad_sch (KiCad schematic)
At the start: 28 parts, among them J101 Conn_01x02, J102 Conn_01x02, J103 Tagbase, J104 USB_B_Mini, SW101 SW_DIP_x04, U101 TPS3700, U106 XC6206-3.3V

Commit message: update multicharger
Parts:
- removed D105: D_Schottky, Diode_SMD:D_SOD-323, symbol Device:D_Schottky
- D102: C72041 C72041 -> (none); LCSC (none) -> C72041
- R107: LCSC 0603WAF2201T5E -> C4190
- U106: value XC6206-3.3V -> AP7370; LCSC C2891841 -> C3745233; MFN Yongyutai -> diodes; MPN XC6206-3.3V -> AP7370-33SA-7
Connections:
- net VIN: now also C106.1, U106.3 (VI)
Changed lines of the file:
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@@
-    (stroke (width 0) (type default) (color 0 0 0 0))
-  )
-  (wire (pts (xy 115.57 41.91) (xy 116.84 41.91))
     (stroke (width 0) (type default) (color 0 0 0 0))
   )
@@
     (stroke (width 0) (type default) (color 0 0 0 0))
   )
-  (wire (pts (xy 104.14 41.91) (xy 107.95 41.91))
+  (wire (pts (xy 104.14 41.91) (xy 116.84 41.91))
     (stroke (width 0) (type default) (color 0 0 0 0))
   )
@@
       (effects (font (size 1.27 1.27)) hide)
     )
-    (property "C72041" "C72041" (id 9) (at 104.14 53.34 0)
+    (property "LCSC" "C72041" (id 9) (at 104.14 53.34 0)
       (effects (font (size 0 0)) hide)
     )
@@
     (in_bom yes) (on_board yes)
     (property "Reference" "U106" (id 0) (at 133.35 38.1 0))
-    (property "Value" "XC6206-3.3V" (id 1) (at 127 33.02 0)
+    (property "Value" "AP7370" (id 1) (at 127 33.02 0)
       (effects (font (size 1.27 1.27)) (justify left))
     )
@@
       (effects (font (size 1.27 1.27) italic) hide)
     )
-    (property "Datasheet" "https://www.torexsemi.com/file/xc6206/XC6206.pdf" (id 3) (at 133.35 41.91 0)
-      (effects (font (size 1.27 1.27)) hide)
-    )
-    (property "MFN" "Yongyutai" (id 4) (at 133.35 41.91 0)
-      (effects (font (size 1.524 1.524)) hide)
-    )
-    (property "MPN" "XC6206-3.3V" (id 5) (at 133.35 41.91 0)
+    (property "Datasheet" "https://www.diodes.com/assets/Datasheets/AP7370.pdf" (id 3) (at 133.35 41.91 0)
+      (effects (font (size 1.27 1.27)) hide)
+    )
+    (property "MFN" "diodes" (id 4) (at 133.35 41.91 0)
+      (effects (font (size 1.524 1.524)) hide)
+    )
+    (property "MPN" "AP7370-33SA-7" (id 5) (at 133.35 41.91 0)
       (effects (font (size 1.524 1.524)) hide)
     )
@@
       (effects (font (size 1.27 1.27)) hide)
     )
-    (property "LCSC" "C2891841" (id 8) (at 133.35 41.91 0)
+    (property "LCSC" "C3745233" (id 8) (at 133.35 41.91 0)
       (effects (font (size 1.27 1.27)) hide)
     )
@@
       (effects (font (size 1.27 1.27)) hide)
     )
-    (property "LCSC" "0603WAF2201T5E" (id 8) (at 83.82 99.06 0)
+    (property "LCSC" "C4190" (id 8) (at 83.82 99.06 0)
       (effects (font (size 1.27 1.27)) hide)
     )
@@
     (pin "8")
   )
-  (symbol (lib_id "Device:D_Schottky") (at 111.76 41.91 180) (unit 1)
-    (in_bom yes) (on_board yes)
-    (property "Reference" "D105" (id 0) (at 111.76 38.1 0))
-    (property "Value" "D_Schottky" (id 1) (at 112.0775 38.1 0)
-      (effects (font (size 1.27 1.27)) hide)
-    )
-    (property "Footprint" "Diode_SMD:D_SOD-323" (id 2) (at 111.76 41.91 0)
-      (effects (font (size 1.27 1.27)) hide)
-    )
-    (property "Datasheet" "~" (id 3) (at 111.76 41.91 0)
-      (effects (font (size 1.27 1.27)) hide)
-    )
-    (property "MFN" "Guangdong Hottech" (id 4) (at 111.76 41.91 0)
-      (effects (font (size 1.524 1.524)) hide)
-    )
-    (property "MPN" "1N5819WS" (id 5) (at 111.76 41.91 0)
-      (effects (font (size 1.524 1.524)) hide)
-    )
-    (property "LCSC" "C191023" (id 6) (at 111.76 41.91 0)
-      (effects (font (size 1.524 1.524)) hide)
-    )
-    (pin "1")
-    (pin "2")
-  )
   (symbol (lib_id "Device:R") (at 83.82 101.6 90) (unit 1)
     (in_bom no) (on_board yes)
@@
       (reference "D104") (unit 1) (value "D_Schottky") (footprint "Diode_SMD:D_SOD-323")
     )
-    (path "/3d3d8aed-3320-4e60-870a-6f704c6611ac"
-      (reference "D105") (unit 1) (value "D_Schottky") (footprint "Diode_SMD:D_SOD-323")
-    )
     (path "/00000000-0000-0000-0000-00005bef58a9"
       (reference "J101") (unit 1) (value "Conn_01x02") (footprint "Connector_JST:JST_PH_B2B-PH-K_1x02_P2.00mm_Vertical")
@@
     )
     (path "/00000000-0000-0000-0000-00005b67840c"
-      (reference "U106") (unit 1) (value "XC6206-3.3V") (footprint "Package_TO_SOT_SMD:SOT-23-3")
-    )
-  )
+      (reference "U106") (unit 1) (value "AP7370") (footprint "Package_TO_SOT_SMD:SOT-23-3")
+    )
+  )

Commit message: update multicharger resistors
Parts:
- R101: value 220 -> 330; LCSC C22962 -> C23138; MPN 0603WAF2200T5E -> 0603WAF3300T5E
- R102, R105: value 120 -> 220; LCSC C22787 -> C22962; MPN 0603WAF1200T5E -> 0603WAF2200T5E
Changed lines of the file:
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@@
     (in_bom yes) (on_board yes)
     (property "Reference" "R102" (id 0) (at 96.52 50.292 90))
-    (property "Value" "120" (id 1) (at 96.52 48.26 90))
+    (property "Value" "220" (id 1) (at 96.52 48.26 90))
     (property "Footprint" "Resistor_SMD:R_0603_1608Metric" (id 2) (at 96.52 46.482 90)
       (effects (font (size 1.27 1.27)) hide)
@@
       (effects (font (size 1.27 1.27)) hide)
     )
-    (property "MPN" "0603WAF1200T5E" (id 4) (at 96.52 48.26 90)
+    (property "MPN" "0603WAF2200T5E" (id 4) (at 96.52 48.26 90)
       (effects (font (size 1.27 1.27)) hide)
     )
@@
       (effects (font (size 1.27 1.27)) hide)
     )
-    (property "Description" "100mW Thick Film Resistors ±100ppm/℃ ±1% 120Ω 0603 " (id 7) (at 96.52 48.26 0)
-      (effects (font (size 1.27 1.27)) hide)
-    )
-    (property "LCSC" "C22787" (id 8) (at 96.52 48.26 90)
+    (property "Description" "100mW Thick Film Resistors ±100ppm/℃ ±1% 220Ω 0603 " (id 7) (at 96.52 48.26 0)
+      (effects (font (size 1.27 1.27)) hide)
+    )
+    (property "LCSC" "C22962" (id 8) (at 96.52 48.26 90)
       (effects (font (size 1.524 1.524)) hide)
     )
@@
     (in_bom yes) (on_board yes)
     (property "Reference" "R105" (id 0) (at 226.568 92.71 90))
-    (property "Value" "120" (id 1) (at 228.6 92.71 90))
+    (property "Value" "220" (id 1) (at 228.6 92.71 90))
     (property "Footprint" "Resistor_SMD:R_0603_1608Metric" (id 2) (at 230.378 92.71 90)
       (effects (font (size 1.27 1.27)) hide)
@@
       (effects (font (size 1.27 1.27)) hide)
     )
-    (property "MPN" "0603WAF1200T5E" (id 4) (at 228.6 92.71 90)
+    (property "MPN" "0603WAF2200T5E" (id 4) (at 228.6 92.71 90)
       (effects (font (size 1.27 1.27)) hide)
     )
@@
       (effects (font (size 1.27 1.27)) hide)
     )
-    (property "Description" "100mW Thick Film Resistors ±100ppm/℃ ±1% 129Ω 0603 " (id 7) (at 228.6 92.71 0)
+    (property "Description" "100mW Thick Film Resistors ±100ppm/℃ ±1% 220Ω 0603 " (id 7) (at 228.6 92.71 0)
       (effects (font (size 1.27 1.27)) hide)
     )
@@
       (effects (font (size 1.524 1.524)) hide)
     )
-    (property "LCSC" "C22787" (id 9) (at 228.6 92.71 0)
+    (property "LCSC" "C22962" (id 9) (at 228.6 92.71 0)
       (effects (font (size 1.27 1.27)) hide)
     )
@@
     (in_bom yes) (on_board yes)
     (property "Reference" "R101" (id 0) (at 216.408 92.71 90))
-    (property "Value" "220" (id 1) (at 218.44 92.71 90))
+    (property "Value" "330" (id 1) (at 218.44 92.71 90))
     (property "Footprint" "Resistor_SMD:R_0603_1608Metric" (id 2) (at 220.218 92.71 90)
       (effects (font (size 1.27 1.27)) hide)
@@
       (effects (font (size 1.27 1.27)) hide)
     )
-    (property "MPN" "0603WAF2200T5E" (id 4) (at 218.44 92.71 90)
+    (property "MPN" "0603WAF3300T5E" (id 4) (at 218.44 92.71 90)
       (effects (font (size 1.27 1.27)) hide)
     )
@@
       (effects (font (size 1.27 1.27)) hide)
     )
-    (property "Description" "100mW Thick Film Resistors ±100ppm/℃ ±1% 220Ω 0603 " (id 7) (at 218.44 92.71 0)
-      (effects (font (size 1.27 1.27)) hide)
-    )
-    (property "LCSC" "C22962" (id 8) (at 218.44 92.71 90)
+    (property "Description" "100mW Thick Film Resistors ±100ppm/℃ ±1% 330Ω 0603 Chip" (id 7) (at 218.44 92.71 0)
+      (effects (font (size 1.27 1.27)) hide)
+    )
+    (property "LCSC" "C23138" (id 8) (at 218.44 92.71 90)
       (effects (font (size 1.524 1.524)) hide)
     )
@@
     )
     (path "/00000000-0000-0000-0000-00005b72d71f"
-      (reference "R101") (unit 1) (value "220") (footprint "Resistor_SMD:R_0603_1608Metric")
+      (reference "R101") (unit 1) (value "330") (footprint "Resistor_SMD:R_0603_1608Metric")
     )
     (path "/00000000-0000-0000-0000-00005b06b8b2"
-      (reference "R102") (unit 1) (value "120") (footprint "Resistor_SMD:R_0603_1608Metric")
+      (reference "R102") (unit 1) (value "220") (footprint "Resistor_SMD:R_0603_1608Metric")
     )
     (path "/00000000-0000-0000-0000-00005b72cf14"
@@
     )
     (path "/00000000-0000-0000-0000-00005b72d633"
-      (reference "R105") (unit 1) (value "120") (footprint "Resistor_SMD:R_0603_1608Metric")
+      (reference "R105") (unit 1) (value "220") (footprint "Resistor_SMD:R_0603_1608Metric")
     )
     (path "/00000000-0000-0000-0000-00006111918b"
