File: hardware/Templates/TagProto/TagProto.kicad_sch (KiCad schematic)
At the start: 20 parts, among them J201 CONN_02X04, J401 CONN_01X02, Q501 Q_NPN_BEC, U1 at25ff321D-UUN, U302 stm32l431kc, U501 RV-3028-C7

Commit message: checkpoint
Parts:
- removed J201: CONN_02X04, bittag:tagpoints6, symbol Connector_Generic:Conn_02x03_Odd_Even
- added J1: Conn_01x06, library:CONN_B6B-ZR_JST, symbol Connector_Generic:Conn_01x06
- added J2: Conn_01x04, Connector_PinHeader_2.54mm:PinHeader_1x05_P2.54mm_Vertical, symbol Connector_Generic:Conn_01x05
- J401: footprint bittag:MS621 -> library:MS621
Connections:
- net +2V5: now also J1.6 (Pin_6)
- net AT25_MISO: now also U302.27 (PB4), J2.3 (Pin_3); no longer U302.12 (PA6)
- net AT25_MOSI: now also U302.28 (PB5), J2.2 (Pin_2); no longer U302.13 (PA7)
- net AT25_SCK: now also U302.26 (PB3), J2.5 (Pin_5); no longer U302.11 (PA5)
- net AT25_nCS: now also U302.25 (PA15), J2.4 (Pin_4); no longer U302.10 (PA4)
- net GND: now also J1.1 (Pin_1), J2.1 (Pin_1)
- net RST: now also J1.3 (Pin_3)
- net SWCLK: now also J1.4 (Pin_4)
- net SWDIO: now also J1.2 (Pin_2)
- net VBAT: now also J1.5 (Pin_5)
- net PB0: now reaches U302.14 (PB0)
- net PB1: now reaches U302.15 (PB1)
- net PA8: now reaches U302.18 (PA8)
- net PA9: now reaches U302.19 (PA9)
- net PA10: now reaches U302.20 (PA10)
- net PA11_MISO: now reaches U302.21 (PA11)
- net PA12_MOSI: now reaches U302.22 (PA12)
- net PA0: now reaches U302.6 (PA0)
- net PA1_SCK: now reaches U302.7 (PA1)
- net PA2: now reaches U302.8 (PA2)
- net PA3: now reaches U302.9 (PA3)
- net SCL renamed RTC_SCL
- net SDA renamed RTC_SDA
- new net PA4: U302.10 (PA4)
- new net PA5_SCK: U302.11 (PA5)
- new net PA6_MISO: U302.12 (PA6)
- new net PA7_MOSI: U302.13 (PA7)
- no-connect marks 2 -> 4
Other:
- note removed: "Test Points"
- moved on the sheet: C101, C2, C3, C4, C404, C501, C502, C503, D401, H1, H2, H3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
