File: hardware/BitTagNG-LIS2DU12/BitTagNG-LIS2DU12.kicad_sch (KiCad schematic)
At the start: 22 parts, among them J201 CONN_02X04, J301 Conn_01x01, J302 Conn_01x01, J303 Conn_01x01, J304 Conn_01x01, J401 CONN_01X02, Q501 Q_NPN_BEC, U1 at25ex321D-UUN, U3 LIS2DW12TR, U302 stm32l431kc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

Commit message: update design
Connections:
- net AT25_MISO: now also U302.27 (PB4); no longer U302.21 (PA11)
- net AT25_MOSI: now also U302.28 (PB5); no longer U302.22 (PA12)
- net AT25_nCS: now also U302.25 (PA15); no longer U302.20 (PA10)
- net GND: no longer U302.9 (PA3)
- net ACCEL_SCK: now reaches U302.11 (PA5)
- net ACCEL_SCK: now also U3.1 (SCL/SPC)
- net ACCEL_MOSI: now reaches U302.13 (PA7)
- net ACCEL_MOSI: now also U3.4 (SDA/SDI/SDO)
- net ACCEL_CS: now reaches U3.2 (CS)
- net ACCEL_CS: now also U302.10 (PA4)
- net ACCEL_MISO: now reaches U3.3 (SDO/SA0)
- net ACCEL_MISO: now also U302.12 (PA6)
- removed net ACCEL_SCL: U3.1 (SCL/SPC), U302.12 (PA6)
- removed net ACCEL_SDA: U3.4 (SDA/SDI/SDO), U302.10 (PA4)
- no-connect marks 17 -> 10
Other:
- title: BitTag with External Memory -> BitTag with External Memory and LI2DW12
Changed lines of the file:
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@@
 	(paper "USLetter")
 	(title_block
-		(title "BitTag with External Memory")
-		(date "2021-09-26")
+		(title "BitTag with External Memory and LI2DW12")
+		(date "2025-02-19")
 		(company "IUCS")
 		(comment 1 "Geoffrey Brown")
@@
 	)
 	(no_connect
-		(at 123.19 53.34)
-	)
-	(no_connect
-		(at 63.5 160.02)
-	)
-	(no_connect
 		(at 153.67 91.44)
 	)
 	(no_connect
-		(at 87.63 91.44)
-	)
-	(no_connect
-		(at 87.63 88.9)
-	)
-	(no_connect
-		(at 115.57 119.38)
+		(at 110.49 119.38)
 	)
 	(no_connect
-		(at 63.5 157.48)
+		(at 125.73 100.33)
 	)
 	(no_connect
@@
 	)
 	(no_connect
-		(at 120.65 119.38)
-	)
-	(no_connect
 		(at 123.19 119.38)
 	)
 	(no_connect
-		(at 130.81 53.34)
-	)
-	(no_connect
 		(at 153.67 93.98)
 	)
@@
 	)
 	(no_connect
-		(at 125.73 53.34)
-	)
-	(no_connect
 		(at 213.36 125.73)
 	)
@@
 	(text "Note: PA15 and PB4 pulled up on reset !"
 		(exclude_from_sim no)
-		(at 130.81 49.53 0)
+		(at 96.012 34.544 0)
 		(effects
 			(font
@@
 		)
 	)
+	(label "WKUP4"
+		(at 63.5 165.1 180)
+		(effects
+			(font
+				(size 1.524 1.524)
+			)
+			(justify right bottom)
+		)
+	)
 	(label "SDA"
 		(at 120.65 53.34 90)
@@
 		)
 	)
-	(label "WKUP4"
-		(at 63.5 165.1 180)
-		(effects
-			(font
-				(size 1.524 1.524)
-			)
-			(justify right bottom)
-		)
-	)
 	(label "clkout"
 		(at 213.36 123.19 180)
@@
 		)
 	)
-	(label "ACCEL_SDA"
+	(label "ACCEL_MOSI"
 		(at 63.5 162.56 180)
 		(effects
@@
 		)
 	)
+	(label "ACCEL_CS"
+		(at 113.03 119.38 270)
+		(effects
+			(font
+				(size 1.524 1.524)
+			)
+			(justify right bottom)
+		)
+	)
 	(label "WKUP4"
 		(at 119.38 154.94 0)
@@
 	)
 	(label "AT25_MOSI"
-		(at 153.67 83.82 0)
+		(at 123.19 53.34 90)
 		(effects
 			(font
@@
 	)
 	(label "AT25_nCS"
-		(at 153.67 88.9 0)
+		(at 130.81 53.34 90)
 		(effects
 			(font
@@
 		)
 	)
-	(label "ACCEL_SCL"
+	(label "ACCEL_SCK"
 		(at 63.5 154.94 180)
 		(effects
@@
 		)
 	)
+	(label "ACCEL_MISO"
+		(at 118.11 119.38 270)
+		(effects
+			(font
+				(size 1.524 1.524)
+			)
+			(justify right bottom)
+		)
+	)
 	(label "AT25_MISO"
-		(at 153.67 86.36 0)
+		(at 125.73 53.34 90)
 		(effects
 			(font
@@
 		)
 	)
+	(label "ACCEL_CS"
+		(at 63.5 157.48 180)
+		(effects
+			(font
+				(size 1.524 1.524)
+			)
+			(justify right bottom)
+		)
+	)
 	(label "SCL"
 		(at 118.11 53.34 90)
@@
 		)
 	)
-	(label "ACCEL_SCL"
-		(at 118.11 119.38 270)
+	(label "ACCEL_MISO"
+		(at 63.5 160.02 180)
+		(effects
+			(font
+				(size 1.524 1.524)
+			)
+			(justify right bottom)
+		)
+	)
+	(label "ACCEL_SCK"
+		(at 115.57 119.38 270)
 		(effects
 			(font
@@
 		)
 	)
-	(label "ACCEL_SDA"
-		(at 113.03 119.38 270)
+	(label "ACCEL_MOSI"
+		(at 120.65 119.38 270)
 		(effects
 			(font
@@
 					(unit 1)
 				)
-			)
-		)
-	)
-	(symbol
-		(lib_id "power:GND")
-		(at 110.49 119.38 0)
-		(unit 1)
-		(exclude_from_sim no)
-		(in_bom yes)
-		(on_board yes)
-		(dnp no)
-		(property "Reference" "#PWR0117"
-			(at 110.49 125.73 0)
-			(effects
-				(font
-					(size 1.27 1.27)
-				)
-				(hide yes)
-			)
-		)
-		(property "Value" "GND"
-			(at 110.49 123.19 0)
-			(effects
-				(font
-					(size 1.27 1.27)
-				)
-			)
-		)
-		(property "Footprint" ""
-			(at 110.49 119.38 0)
-			(effects
-				(font
-					(size 1.27 1.27)
-				)
-				(hide yes)
-			)
-		)
-		(property "Datasheet" ""
-			(at 110.49 119.38 0)
-			(effects
-				(font
-					(size 1.27 1.27)
-				)
-				(hide yes)
-			)
-		)
-		(property "Description" ""
-			(at 110.49 119.38 0)
-			(effects
-				(font
-					(size 1.27 1.27)
-				)
-				(hide yes)
-			)
-		)
-		(pin "1"
-		)
-		(instances
-			(project ""
-				(path "/e44ca67a-43be-444b-8652-f54825a2eb6f"
-					(reference "#PWR0117")
-					(unit 1)
-				)

Commit message: updated latest board design
Parts:
- C2: DISTPN 490-10403-1-ND -> 490-7229-2-ND; LCSC C181047 -> C76929; MFN Murata -> murata; MPN C181047 -> GRM033R60J105MEA2D
Connections:
- net ACCEL_CS: now also U302.7 (PA1); no longer U302.10 (PA4)
- net ACCEL_SCK: now also U302.9 (PA3); no longer U302.11 (PA5)
- net GND: now also U3.5 (NC)
- net WKUP4: no longer U3.5 (NC)
- net ACCEL_SDI_SDO: now reaches U302.6 (PA0)
- net ACCEL_SDI_SDO: now also U3.4 (SDA/SDI/SDO)
- net ACCEL_MISO: no longer names the net of U302.12 (PA6)
- net ACCEL_MISO: no longer U3.3 (SDO/SA0)
- net ACCEL_MOSI: no longer names the net of U302.13 (PA7)
- net ACCEL_MOSI: no longer U3.4 (SDA/SDI/SDO)
- no-connect marks 10 -> 17
Other:
- note added: "PA4 -- LPTIM2_OUT PA8 -- LPTIM2_OUT parts with LPTIM2 active in STOP2 STM32L422KBU6 STM32L412KBU6"
Changed lines of the file:
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@@
 	)
 	(junction
+		(at 59.69 167.64)
+		(diameter 0)
+		(color 0 0 0 0)
+	)
+	(junction
 		(at 245.11 33.02)
 		(diameter 0)
@@
 	)
 	(no_connect
+		(at 153.67 83.82)
+	)
+	(no_connect
+		(at 113.03 119.38)
+	)
+	(no_connect
+		(at 118.11 119.38)
+	)
+	(no_connect
+		(at 120.65 119.38)
+	)
+	(no_connect
 		(at 153.67 91.44)
 	)
 	(no_connect
-		(at 110.49 119.38)
+		(at 153.67 86.36)
 	)
 	(no_connect
@@
 	)
 	(no_connect
+		(at 63.5 160.02)
+	)
+	(no_connect
 		(at 119.38 157.48)
 	)
@@
 	)
 	(no_connect
+		(at 153.67 88.9)
+	)
+	(no_connect
+		(at 115.57 119.38)
+	)
+	(no_connect
 		(at 125.73 119.38)
 	)
@@
 	(wire
 		(pts
+			(xy 63.5 165.1) (xy 59.69 165.1)
+		)
+		(stroke
+			(width 0)
+			(type default)
+		)
+	)
+	(wire
+		(pts
 			(xy 104.14 49.53) (xy 110.49 49.53)
 		)
@@
 	(wire
 		(pts
+			(xy 59.69 165.1) (xy 59.69 167.64)
+		)
+		(stroke
+			(width 0)
+			(type default)
+		)
+	)
+	(wire
+		(pts
 			(xy 41.91 41.91) (xy 41.91 44.45)
 		)
@@
 		)
 	)
-	(label "WKUP4"
-		(at 63.5 165.1 180)
+	(text "\nPA4 -- LPTIM2_OUT\nPA8 -- LPTIM2_OUT\n\nparts with LPTIM2 active in STOP2\n\nSTM32L422KBU6\nSTM32L412KBU6"
+		(exclude_from_sim no)
+		(at 166.624 135.89 0)
 		(effects
 			(font
 				(size 1.524 1.524)
 			)
-			(justify right bottom)
 		)
 	)
@@
 		)
 	)
-	(label "ACCEL_MOSI"
+	(label "ACCEL_SDI_SDO"
 		(at 63.5 162.56 180)
 		(effects
@@
 	)
 	(label "ACCEL_CS"
-		(at 113.03 119.38 270)
+		(at 87.63 91.44 180)
 		(effects
 			(font
@@
 		)
 	)
-	(label "ACCEL_MISO"
-		(at 118.11 119.38 270)
+	(label "ACCEL_SDI_SDO"
+		(at 87.63 88.9 180)
 		(effects
 			(font
@@
 		)
 	)
-	(label "ACCEL_MISO"
-		(at 63.5 160.02 180)
-		(effects
-			(font
-				(size 1.524 1.524)
-			)
-			(justify right bottom)
-		)
-	)
 	(label "ACCEL_SCK"
-		(at 115.57 119.38 270)
+		(at 110.49 119.38 270)
 		(effects
 			(font
@@
 		)
 	)
-	(label "ACCEL_MOSI"
-		(at 120.65 119.38 270)
-		(effects
-			(font
-				(size 1.524 1.524)
-			)
-			(justify right bottom)
-		)
-	)
 	(global_label "SWCLK"
 		(shape input)
@@
 			)
 		)
-		(property "MFN" "Murata"
+		(property "MFN" "murata"
 			(at 179.07 100.33 0)
 			(effects
@@
 			)
 		)
-		(property "MPN" "C181047"
+		(property "MPN" "GRM033R60J105MEA2D"
 			(at 179.07 100.33 0)
 			(effects
@@
 			)
 		)
-		(property "DISTPN" "490-10403-1-ND"
+		(property "DISTPN" "490-7229-2-ND"
 			(at 110.49 198.12 0)
 			(effects
@@
 			)
 		)
-		(property "LCSC" "C181047"
+		(property "LCSC" "C76929"
 			(at 179.07 100.33 0)
 			(effects

Commit message: working on compass board
Parts:
- U3: value LIS2DW12TR -> LIS2DU12TR; footprint AccelTag:LIS2DW12TR -> AccelTag:LGA-12L_LIS2DU12_STM; symbol lis2dw12:LIS2DW12TR -> lis2du12:LIS2DU12TR
Connections:
- net GND: no longer U3.5 (NC)
Other:
- note added: "PA3 is not SCK PA0 is not SDO This wiring is for bit-banged SPI"
Changed lines of the file:
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@@
 	)
 	(junction
-		(at 59.69 167.64)
-		(diameter 0)
-		(color 0 0 0 0)
-	)
-	(junction
 		(at 245.11 33.02)
 		(diameter 0)
@@
 	)
 	(no_connect
-		(at 63.5 160.02)
+		(at 58.42 160.02)
 	)
 	(no_connect
@@
 	(wire
 		(pts
-			(xy 63.5 167.64) (xy 59.69 167.64)
+			(xy 58.42 167.64) (xy 54.61 167.64)
 		)
 		(stroke
@@
 	(wire
 		(pts
-			(xy 63.5 165.1) (xy 59.69 165.1)
-		)
-		(stroke
-			(width 0)
-			(type default)
-		)
-	)
-	(wire
-		(pts
 			(xy 104.14 49.53) (xy 110.49 49.53)
 		)
@@
 	(wire
 		(pts
-			(xy 59.69 165.1) (xy 59.69 167.64)
-		)
-		(stroke
-			(width 0)
-			(type default)
-		)
-	)
-	(wire
-		(pts
 			(xy 41.91 41.91) (xy 41.91 44.45)
 		)
@@
 	(wire
 		(pts
-			(xy 59.69 167.64) (xy 59.69 171.45)
+			(xy 54.61 167.64) (xy 54.61 171.45)
 		)
 		(stroke
@@
 		)
 	)
+	(text "PA3 is not SCK\nPA0 is not SDO\nThis wiring is for bit-banged SPI"
+		(exclude_from_sim no)
+		(at 45.212 141.732 0)
+		(effects
+			(font
+				(size 1.524 1.524)
+			)
+		)
+	)
 	(text "Note: PA15 and PB4 pulled up on reset !"
 		(exclude_from_sim no)
@@
 	)
 	(label "ACCEL_SDI_SDO"
-		(at 63.5 162.56 180)
+		(at 58.42 162.56 180)
 		(effects
 			(font
@@
 	)
 	(label "ACCEL_SCK"
-		(at 63.5 154.94 180)
+		(at 58.42 154.94 180)
 		(effects
 			(font
@@
 	)
 	(label "ACCEL_CS"
-		(at 63.5 157.48 180)
+		(at 58.42 157.48 180)
 		(effects
 			(font
@@
 	)
 	(symbol
-		(lib_id "lis2dw12:LIS2DW12TR")
-		(at 63.5 154.94 0)
+		(lib_id "lis2du12:LIS2DU12TR")
+		(at 58.42 154.94 0)
 		(unit 1)
 		(exclude_from_sim no)
@@
 		(on_board yes)
 		(dnp no)
-		(fields_autoplaced yes)
 		(property "Reference" "U3"
-			(at 91.44 144.78 0)
+			(at 88.9 144.78 0)
 			(effects
 				(font
@@
 			)
 		)
-		(property "Value" "LIS2DW12TR"
-			(at 91.44 147.32 0)
+		(property "Value" "LIS2DU12TR"
+			(at 88.9 147.32 0)
 			(effects
 				(font
@@
 			)
 		)
-		(property "Footprint" "AccelTag:LIS2DW12TR"
-			(at 63.5 154.94 0)
+		(property "Footprint" "AccelTag:LGA-12L_LIS2DU12_STM"
+			(at 58.42 154.94 0)
 			(effects
 				(font
@@
 			)
 		)
-		(property "Datasheet" "LIS2DW12TR"
-			(at 63.5 154.94 0)
+		(property "Datasheet" "LIS2DU12TR"
+			(at 58.42 154.94 0)
 			(effects
 				(font
@@
 		)
 		(property "Description" ""
-			(at 63.5 154.94 0)
+			(at 58.42 154.94 0)
 			(effects
 				(font
@@
 	(symbol
 		(lib_id "power:GND")
-		(at 59.69 171.45 0)
+		(at 54.61 171.45 0)
 		(unit 1)
 		(exclude_from_sim no)
@@
 		(dnp no)
 		(property "Reference" "#PWR02"
-			(at 59.69 177.8 0)
+			(at 54.61 177.8 0)
 			(effects
 				(font
@@
 		)
 		(property "Value" "GND"
-			(at 59.69 175.26 0)
+			(at 54.61 175.26 0)
 			(effects
 				(font
@@
 		)
 		(property "Footprint" ""
-			(at 59.69 171.45 0)
+			(at 54.61 171.45 0)
 			(effects
 				(font
@@
 		)
 		(property "Datasheet" ""
-			(at 59.69 171.45 0)
+			(at 54.61 171.45 0)
 			(effects
 				(font
@@
 		)
 		(property "Description" ""
-			(at 59.69 171.45 0)
+			(at 54.61 171.45 0)
 			(effects
 				(font

Commit message: designed compass tag
Parts:
- U3: footprint AccelTag:LGA-12L_LIS2DU12_STM -> LGA-12L_LIS2DU12_STM
Connections:
- net USART2_CK: now reaches U302.10 (PA4)
- net USART2_CK: now also U3.1 (SCL/SPC)
- net USART2_RX: now reaches U3.3 (SDO/SA0)
- net USART2_RX: now also U302.9 (PA3)
- net WKUP1: now reaches U3.5 (NC)
- net WKUP1: now also U3.12 (INT1), U302.6 (PA0)
- removed net ACCEL_SCK: U3.1 (SCL/SPC), U302.9 (PA3)
- net ACCEL_SDI_SDO renamed USART2_TX
- net USART2_TX: now also U302.8 (PA2); no longer U302.6 (PA0)
- removed net WKUP4: U3.12 (INT1), U302.8 (PA2)
- no-connect marks 17 -> 14
Other:
- note removed: "Connect wkup1, wkup4 to enable wakeup on both edges"
- note removed: "PA3 is not SCK PA0 is not SDO This wiring is for bit-banged SPI"
Changed lines of the file:
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@@
 	)
 	(no_connect
-		(at 113.03 119.38)
-	)
-	(no_connect
 		(at 118.11 119.38)
 	)
@@
 	)
 	(no_connect
-		(at 125.73 100.33)
-	)
-	(no_connect
-		(at 58.42 160.02)
-	)
-	(no_connect
 		(at 119.38 157.48)
 	)
@@
 		)
 	)
-	(text "PA3 is not SCK\nPA0 is not SDO\nThis wiring is for bit-banged SPI"
-		(exclude_from_sim no)
-		(at 45.212 141.732 0)
-		(effects
-			(font
-				(size 1.524 1.524)
-			)
-		)
-	)
 	(text "Note: PA15 and PB4 pulled up on reset !"
 		(exclude_from_sim no)
@@
 		)
 	)
-	(text "Connect wkup1, wkup4 to enable wakeup on both edges"
+	(text "\nPA4 -- LPTIM2_OUT\nPA8 -- LPTIM2_OUT\n\nparts with LPTIM2 active in STOP2\n\nSTM32L422KBU6\nSTM32L412KBU6"
 		(exclude_from_sim no)
-		(at 35.56 120.65 0)
+		(at 166.624 135.89 0)
 		(effects
 			(font
 				(size 1.524 1.524)
 			)
-			(justify left bottom)
 		)
 	)
-	(text "\nPA4 -- LPTIM2_OUT\nPA8 -- LPTIM2_OUT\n\nparts with LPTIM2 active in STOP2\n\nSTM32L422KBU6\nSTM32L412KBU6"
-		(exclude_from_sim no)
-		(at 166.624 135.89 0)
+	(label "USART2_CK"
+		(at 113.03 119.38 270)
 		(effects
 			(font
 				(size 1.524 1.524)
 			)
+			(justify right bottom)
 		)
 	)
@@
 		)
 	)
-	(label "WKUP4"
-		(at 83.82 93.98 180)
+	(label "WKUP1"
+		(at 87.63 88.9 180)
 		(effects
 			(font
@@
 		)
 	)
-	(label "ACCEL_SDI_SDO"
-		(at 58.42 162.56 180)
+	(label "USART2_RX"
+		(at 58.42 160.02 180)
 		(effects
 			(font
@@
 		)
 	)
-	(label "WKUP4"
+	(label "WKUP1"
 		(at 119.38 154.94 0)
 		(effects
@@
 		)
 	)
+	(label "WKUP1"
+		(at 58.42 165.1 180)
+		(effects
+			(font
+				(size 1.524 1.524)
+			)
+			(justify right bottom)
+		)
+	)
 	(label "AT25_MOSI"
 		(at 123.19 53.34 90)
@@
 		)
 	)
-	(label "ACCEL_SCK"
+	(label "USART2_CK"
 		(at 58.42 154.94 180)
 		(effects
@@
 		)
 	)
-	(label "ACCEL_SDI_SDO"
-		(at 87.63 88.9 180)
+	(label "USART2_TX"
+		(at 83.82 93.98 180)
 		(effects
 			(font
@@
 		)
 	)
-	(label "ACCEL_SCK"
-		(at 110.49 119.38 270)
-		(effects
-			(font
-				(size 1.524 1.524)
-			)
-			(justify right bottom)
-		)
-	)
 	(label "AT25_SCK"
 		(at 128.27 53.34 90)
@@
 		)
 	)
+	(label "USART2_RX"
+		(at 110.49 119.38 270)
+		(effects
+			(font
+				(size 1.524 1.524)
+			)
+			(justify right bottom)
+		)
+	)
+	(label "USART2_TX"
+		(at 58.42 162.56 180)
+		(effects
+			(font
+				(size 1.524 1.524)
+			)
+			(justify right bottom)
+		)
+	)
 	(global_label "SWCLK"
 		(shape input)
@@
 			)
 		)
-		(property "Description" ""
+		(property "Description" "Power symbol creates a global label with name \"GND\" , ground"
 			(at 41.91 44.45 0)
 			(effects
@@
 			)
 		)
-		(property "Description" ""
+		(property "Description" "Power symbol creates a global label with name \"GND\" , ground"
 			(at 68.58 104.14 0)
 			(effects
@@
 			)
 		)
-		(property "Description" ""
+		(property "Description" "Power symbol creates a global label with name \"GND\" , ground"
 			(at 128.27 121.92 0)
 			(effects
@@
 			)
 		)
-		(property "Description" ""
+		(property "Description" "Power symbol creates a global label with name \"+2V5\""
 			(at 82.55 73.66 0)
 			(effects
@@
 			)
 		)
-		(property "Description" ""
+		(property "Description" "Power symbol creates a global label with name \"+2V5\""
 			(at 179.07 95.25 0)
 			(effects
@@
 			)
 		)
-		(property "Description" ""
+		(property "Description" "Power symbol creates a global label with name \"GND\" , ground"
 			(at 104.14 52.07 0)
 			(effects
@@
 			)
 		)
-		(property "Description" ""
+		(property "Description" "Power symbol creates a global label with name \"GND\" , ground"
 			(at 205.74 34.29 0)
 			(effects
@@
 			)
 		)
-		(property "Description" ""
+		(property "Description" "Power symbol creates a global label with name \"GND\" , ground"
 			(at 256.54 140.97 0)
 			(effects
@@
 			)
 		)
-		(property "Description" ""
+		(property "Description" "Power symbol creates a global label with name \"+2V5\""
 			(at 256.54 123.19 0)
 			(effects
@@
 			)
 		)
-		(property "Description" ""
+		(property "Description" "Power symbol creates a global label with name \"+2V5\""
 			(at 245.11 22.86 0)
 			(effects
@@
 			)
 		)
-		(property "Datasheet" ""
+		(property "Datasheet" "~"
 			(at 232.41 22.86 0)
 			(effects
@@
 			)
 		)
-		(property "Description" ""
+		(property "Description" "Special symbol for telling ERC where power comes from"
 			(at 232.41 22.86 0)
 			(effects
@@
 			)
 		)
-		(property "Description" ""
+		(property "Description" "Power symbol creates a global label with name \"GND\" , ground"
 			(at 245.11 45.72 0)
 			(effects
@@
 			)
 		)
-		(property "Description" ""
+		(property "Description" "Power symbol creates a global label with name \"+2V5\""
 			(at 74.93 29.21 0)
 			(effects
@@
 			)
 		)
-		(property "Description" ""
+		(property "Description" "Power symbol creates a global label with name \"GND\" , ground"
 			(at 179.07 104.14 0)
 			(effects
@@
 			)
 		)
-		(property "Description" ""
+		(property "Description" "Power symbol creates a global label with name \"GND\" , ground"
 			(at 138.43 185.42 0)
 			(effects
@@
 			)
 		)
-		(property "Description" ""
+		(property "Description" "Power symbol creates a global label with name \"GND\" , ground"
 			(at 123.19 171.45 0)
 			(effects
@@
 			)
 		)
-		(property "Description" ""
+		(property "Description" "Power symbol creates a global label with name \"+2V5\""
 			(at 135.89 153.67 0)
 			(effects
@@
 			)
 		)
-		(property "Footprint" "AccelTag:LGA-12L_LIS2DU12_STM"
+		(property "Footprint" "LGA-12L_LIS2DU12_STM"
 			(at 58.42 154.94 0)
 			(effects
@@
 			)
 		)
-		(property "Description" ""
+		(property "Description" "Power symbol creates a global label with name \"GND\" , ground"
 			(at 54.61 171.45 0)
 			(effects
@@
 			)
 		)
-		(property "Description" ""
+		(property "Description" "Power symbol creates a global label with name \"GND\" , ground"
 			(at 243.84 140.97 0)
 			(effects
