File: hardware/TagMagAccelPresBreakout/TagMagAccelPresBreakout.kicad_pcb (KiCad board)
At the start: 2 copper layers, 50 x 35 mm, 28 parts, among them J1 Conn_01x06, J2 Conn_01x04, J3 Conn_01x04, J4 Conn_01x06, J401 CONN_01X02, J5 Conn_01x06, Q501 Q_NPN_BEC, U1 at25ff321D-UUN, U2 LIS2DU12TR, U3 LPS27HHWTR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

Commit message: finish breakout board with mag, accel, pres
Parts:
- removed C3: 22uf, Capacitor_SMD:C_0402_1005Metric
- added C5: 0.1uf, Capacitor_SMD:C_0201_0603Metric, F.Cu at (131.2, 106.9)
- added C7: 0.1uf, Capacitor_SMD:C_0201_0603Metric, F.Cu at (132.7, 108.5)
- added C8: 1uf, Capacitor_SMD:C_0201_0603Metric, F.Cu at (129.8, 104.8)
- added C9: 1uf, Capacitor_SMD:C_0201_0603Metric, F.Cu at (131.2, 106.1)
- added J6: Conn_02x04_Counter_Clockwise, Connector_PinHeader_2.54mm:PinHeader_2x04_P2.54mm_Vertical, F.Cu at (141.5, 105.3)
- added U4: AK09940A, library:AK09940a, F.Cu at (130.8, 108.6)
- added U5: TPS7A2018PDQN, Package_SON:Texas_X2SON-4_1x1mm_P0.65mm, F.Cu at (131.2, 104.6)
- U1: value at25ff321D-UUN -> at25xe321D-UUN
- moved C6 6.33 mm to (119.6, 108.0), turned to 180 degrees
- moved U3 3.18 mm to (119.4, 105.9), turned to 180 degrees
- moved J401 2.09 mm to (138.6, 118.1)
Connections:
- J5 pad 2: /LPS_TX -> /LPS_SCK
- J5 pad 3: /LPS_SCK -> /LPS_PWR
- J5 pad 4: /LPS_PWR -> /LPS_CS
- J5 pad 6: /LPS_CS -> /LPS_TX
- U302 pad 15: /AK_PWR -> /AK_CS
- U302 pad 21: /AK_CS -> /AK_RSTN
- U302 pad 22: /AK_EN -> /AK_PWR
Routing:
- net /AK_PWR: track 0.00 -> 25.8 mm
- net /AK_USART1_TX: track 0.00 -> 25.1 mm, vias 0 -> 2
- net /AK_RSTN: track 0.00 -> 23.8 mm, vias 0 -> 2
- net /AK_USART1_CK: track 0.00 -> 22.6 mm, vias 0 -> 2
- net /AK_USART1_RX: track 0.00 -> 22.1 mm, vias 0 -> 2
- net /AK_CS: track 0.00 -> 21.1 mm
- net +1V8: track 0.00 -> 17.6 mm, vias 0 -> 2
- net GND: track 44.9 -> 53.9 mm, vias 17 -> 19
- net VIN: track 74.9 -> 80.5 mm, vias 3 -> 4
- net /LPS_SCK: track 16.2 -> 19.4 mm
- net /LPS_PWR: track 17.5 -> 20.7 mm
- net /LPS_CS: track 19.4 -> 16.9 mm
- net /LIS_INT1: track 17.8 -> 17.1 mm, vias 4 -> 2
- net /LPS_TX: vias 2 -> 0
Other:
- board text added: "+1V8"
- board text added: "CLK"
- board text added: "CS"
- board text added: "MAG"
- board text added: "PWR"
- board text added: "RSTN"
- board text added: "RX"
- board text added: "TX"
- board text removed: "LPS_CS"
- board text removed: "LPS_PWR"
- board text removed: "LPS_RX"
- board text removed: "LPS_SCK"
- board text removed: "LPS_TX"

Commit message: checkpoint
Connections:
- net RST renamed /RST
- net VBAT renamed /VBAT
- net VIN renamed +2V5
Other:
- board text added: "Tag Breakout with AK09940a, LIS2DU12, LPS27 Geoffrey Brown 3/16/2025"
