File: hardware/BitPresTag/BitPresTag.kicad_pcb (KiCad board)
At the start: 2 copper layers, 17 x 10 mm, 23 parts, among them J201 CONN_02X04, J301 Conn_01x01, J302 Conn_01x01, J303 Conn_01x01, J304 Conn_01x01, J401 CONN_01X02, Q501 Q_NPN_BEC, U1 at25ex321D-UUN, U2 adxl362, U3 LPS27HHWTR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

Commit message: checkpoint hardware designs
Connections:
- C1 pad 1: Net-(U2-VDDI/O) -> VIN
- U2 pad 1: Net-(U2-VDDI/O) -> VIN
- U302 pad 10: /LPS_CS -> /LPS_SCK
- U302 pad 7: /LPS_SCK -> /LPS_CS
Routing:
- net VIN: track 34.1 -> 42.5 mm
- net /LPS_SCK: track 8.76 -> 3.37 mm
- net /LPS_CS: track 4.93 -> 2.60 mm
- net Net-(U2-VDDI/O): track 1.34 -> 0.00 mm
- net /LPS_MOSI: track 5.48 -> 4.85 mm
