File: hardware/BitPresTag/BitPresTag.kicad_sch (KiCad schematic)
At the start: 23 parts, among them J201 CONN_02X04, J301 Conn_01x01, J302 Conn_01x01, J303 Conn_01x01, J304 Conn_01x01, J401 CONN_01X02, Q501 Q_NPN_BEC, U1 at25ex321D-UUN, U2 adxl362, U3 LPS27HHWTR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

Commit message: checkpoint hardware designs
Connections:
- net +2V5: now also C1.1, U2.1 (VDDI/O)
- net LPS_CS: now also U302.7 (PA1); no longer U302.10 (PA4)
- net LPS_SCK: now also U302.10 (PA4); no longer U302.7 (PA1)
Other:
- title: BitTag with External Memory and LI2DW12 -> BitTag with External Memory and LPS27
Changed lines of the file:
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@@
 	(paper "USLetter")
 	(title_block
-		(title "BitTag with External Memory and LI2DW12")
-		(date "2025-02-19")
+		(title "BitTag with External Memory and LPS27")
+		(date "2025-04-25")
 		(company "IUCS")
 		(comment 1 "Geoffrey Brown")
+		(comment 3 "checked pinouts 4/25/25")
 	)
 	(junction
@@
 	)
 	(junction
+		(at 26.67 148.59)
+		(diameter 0)
+		(color 0 0 0 0)
+	)
+	(junction
 		(at 245.11 24.13)
 		(diameter 0)
@@
 		)
 	)
-	(label "LPS_SCK"
+	(label "LPS_CS"
 		(at 87.63 91.44 180)
 		(effects
@@
 		)
 	)
-	(label "LPS_CS"
+	(label "LPS_SCK"
 		(at 113.03 119.38 270)
 		(effects
@@
 					(unit 1)
 				)
+			)
+		)
+	)
+	(symbol
+		(lib_id "power:+2V5")
+		(at 26.67 148.59 0)
+		(unit 1)
+		(exclude_from_sim no)
+		(in_bom yes)
+		(on_board yes)
+		(dnp no)
+		(property "Reference" "#PWR8"
+			(at 26.67 152.4 0)
+			(effects
+				(font
+					(size 1.27 1.27)
+				)
+				(hide yes)
+			)
+		)
+		(property "Value" "+2V5"
+			(at 27.051 144.1958 0)
+			(effects
+				(font
+					(size 1.27 1.27)
+				)
+			)
+		)
+		(property "Footprint" ""
+			(at 26.67 148.59 0)
+			(effects
+				(font
+					(size 1.27 1.27)
+				)
+				(hide yes)
+			)
+		)
+		(property "Datasheet" ""
+			(at 26.67 148.59 0)
+			(effects
+				(font
+					(size 1.27 1.27)
+				)
+				(hide yes)
+			)
+		)
+		(property "Description" ""
+			(at 26.67 148.59 0)
+			(effects
+				(font
+					(size 1.27 1.27)
+				)
+				(hide yes)
+			)
+		)
+		(pin "1"
+		)
+		(instances
+			(project "BitPresTag"
+				(path "/e44ca67a-43be-444b-8652-f54825a2eb6f"
+					(reference "#PWR8")
+					(unit 1)
+				)
