File: hardware/CompassTagBreakout/CompassTagBreakout.kicad_pcb (KiCad board)
At the start: 2 copper layers, 48.3 x 48.3 mm, 15 parts, among them J3 Conn_01x17, J4 Conn_01x17, U1 TPS7A2018PDQN, U2 AT25XE321, U3 AK09940A, U4 LIS2DU12TR

Commit message: checkpoint
Connections:
- U3 pad A4: /AK_MISO -> /AK_MOSI
- U3 pad B4: /AK_MOSI -> /AK_MISO
Routing:
- net /AK_MOSI: track 24.6 -> 21.6 mm
Changed lines of the file:
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@@
 			(size 0.2286 0.2286)
 			(layers "F.Cu" "F.Paste" "F.Mask")
-			(net 27 "/AK_MISO")
+			(net 28 "/AK_MOSI")
 			(pinfunction "SDA/SI")
 			(pintype "bidirectional")
@@
 			(size 0.2286 0.2286)
 			(layers "F.Cu" "F.Paste" "F.Mask")
-			(net 28 "/AK_MOSI")
+			(net 27 "/AK_MISO")
 			(pinfunction "SO")
 			(pintype "output")
@@
 			)
 		)
+		(property "LCSC" "C2878130"
+			(at 0 0 0)
+			(unlocked yes)
+			(layer "F.Fab")
+			(hide yes)
+			(effects
+				(font
+					(size 1 1)
+					(thickness 0.15)
+				)
+			)
+		)
 		(property ki_fp_filters "*X2SON*1x1mm*P0.65mm*")
 		(sheetname "Root")
@@
 	)
 	(segment
-		(start 126.5684 107.2316)
-		(end 126.5684 107.0284)
+		(start 126.5684 107.0284)
+		(end 126.5684 107.2316)
 		(width 0.1524)
 		(layer "F.Cu")
@@
 	)
 	(segment
-		(start 122.5 108.2)
-		(end 125.6 108.2)
+		(start 126.5684 107.2316)
+		(end 125.238315 108.561685)
 		(width 0.1524)
 		(layer "F.Cu")
@@
 	)
 	(segment
-		(start 125.6 108.2)
-		(end 126.5684 107.2316)
+		(start 125.238315 108.561685)
+		(end 122.630685 108.561685)
 		(width 0.1524)
 		(layer "F.Cu")
@@
 	)
 	(via
-		(at 122.5 108.2)
+		(at 122.630685 108.561685)
 		(size 0.6096)
 		(drill 0.3)
@@
 	)
 	(segment
-		(start 122.4 106.68)
-		(end 122.4 108.1)
+		(start 122.4 108.331)
+		(end 122.630685 108.561685)
 		(width 0.1524)
 		(layer "B.Cu")
@@
 	)
 	(segment
-		(start 122.4 108.1)
-		(end 122.5 108.2)
+		(start 122.4 106.68)
+		(end 122.4 108.331)
 		(width 0.1524)
 		(layer "B.Cu")
@@
 	)
 	(segment
-		(start 126.1684 107.0284)
-		(end 125.7428 107.454)
-		(width 0.1524)
-		(layer "F.Cu")
-		(net 27)
-	)
-	(segment
 		(start 108.573 107.454)
-		(end 106.807 109.22)
+		(end 122.78679 107.454)
 		(width 0.1524)
 		(layer "F.Cu")
@@
 	)
 	(segment
-		(start 125.7428 107.454)
+		(start 106.807 109.22)
 		(end 108.573 107.454)
 		(width 0.1524)
@@
 	)
 	(segment
-		(start 126.1684 106.6284)
-		(end 123.79081 106.6284)
+		(start 122.78679 107.454)
+		(end 123.61239 106.6284)
 		(width 0.1524)
 		(layer "F.Cu")
-		(net 28)
+		(net 27)
 	)
 	(segment
-		(start 123.21921 107.2)
-		(end 107.5922 107.2)
+		(start 123.61239 106.6284)
+		(end 126.1684 106.6284)
 		(width 0.1524)
 		(layer "F.Cu")
-		(net 28)
+		(net 27)
 	)
 	(segment
-		(start 107.5922 107.2)
-		(end 106.6 108.1922)
+		(start 123.5716 107.0284)
+		(end 122.8 107.8)
 		(width 0.1524)
 		(layer "F.Cu")
@@
 	)
 	(segment
-		(start 106.6 108.1922)
-		(end 106.381271 108.1922)
+		(start 126.1684 107.0284)
+		(end 123.5716 107.0284)
 		(width 0.1524)
 		(layer "F.Cu")
@@
 	)
 	(segment
-		(start 123.79081 106.6284)
-		(end 123.21921 107.2)
+		(start 122.5 107.8)
+		(end 122.1 108.2)
 		(width 0.1524)
 		(layer "F.Cu")
@@
 	)
 	(segment
-		(start 105.7 110.907)
+		(start 110.113 108.2)
 		(end 106.553 111.76)
 		(width 0.1524)
@@
 	)
 	(segment
-		(start 105.7 108.873471)
-		(end 105.7 110.907)
+		(start 122.8 107.8)
+		(end 122.5 107.8)
 		(width 0.1524)
 		(layer "F.Cu")
@@
 	)
 	(segment
-		(start 106.381271 108.1922)
-		(end 105.7 108.873471)
+		(start 122.1 108.2)
+		(end 110.113 108.2)
 		(width 0.1524)
 		(layer "F.Cu")

Commit message: checkpoint
Parts:
- moved C9 0.90 mm to (122.3, 81.3)
Routing:
- net /TAG_3V3: track 91.4 -> 92.3 mm
Changed lines of the file:
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@@
 	(footprint "Capacitor_SMD:C_0201_0603Metric"
 		(layer "F.Cu")
-		(at 123.205 81.325 -90)
+		(at 122.305 81.325 -90)
 		(descr "Capacitor SMD 0201 (0603 Metric), square (rectangular) end terminal, IPC_7351 nominal, (Body size source: https://www.vishay.com/docs/20052/crcw0201e3.pdf), generated with kicad-footprint-generator")
 		(tags "capacitor")
@@
 	)
 	(segment
-		(start 123.2 82.3)
-		(end 123.205 82.295)
+		(start 122.3 82.3)
+		(end 122.305 82.295)
 		(width 0.1524)
 		(layer "F.Cu")
@@
 	)
 	(segment
-		(start 123.205 81.645)
-		(end 123.205 82.295)
+		(start 122.305 81.645)
+		(end 122.305 82.295)
 		(width 0.1524)
 		(layer "F.Cu")
@@
 	)
 	(via
-		(at 123.205 82.295)
+		(at 122.305 82.295)
 		(size 0.6096)
 		(drill 0.3)
@@
 	)
 	(segment
+		(start 125.03 81.005)
+		(end 122.305 81.005)
+		(width 0.1524)
+		(layer "F.Cu")
+		(net 2)
+	)
+	(segment
 		(start 151.0656 81.5344)
 		(end 150 82.6)
@@
 	)
 	(segment
+		(start 125.05 80.985)
+		(end 125.03 81.005)
+		(width 0.1524)
+		(layer "F.Cu")
+		(net 2)
+	)
+	(segment
 		(start 128.854299 100.334299)
 		(end 129.025 100.505)
@@
 	)
 	(segment
-		(start 125.03 81.005)
-		(end 125.05 80.985)
-		(width 0.1524)
-		(layer "F.Cu")
-		(net 2)
-	)
-	(segment
 		(start 127.35 84.75)
 		(end 118.85 84.75)
@@
 		(width 0.1524)
 		(layer "F.Cu")
-		(net 2)
-	)
-	(segment
-		(start 123.205 81.005)
-		(end 125.03 81.005)
-		(width 0.1524)
-		(layer "F.Cu")

Commit message: checkpoint -- order compass proto board
Other:
- board text added: "Geoffrey Brown 6/3/2025"
- board text removed: "Geoffrey Brown 4/17/2025"
Changed lines of the file:
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@@
 		(layer "Edge.Cuts")
 	)
-	(gr_text "Geoffrey Brown\n4/17/2025"
+	(gr_text "Geoffrey Brown\n6/3/2025"
 		(at 130.59 112.98 0)
 		(layer "B.SilkS")

Commit message: update proto boards
Parts:
- moved C9 1.80 mm to (120.5, 81.2)
Routing:
- net /TAG_3V3: track 92.3 -> 94.1 mm
Changed lines of the file:
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@@
 		(sheetname "Root")
 		(sheetfile "CompassTagBreakout.kicad_sch")
-		(attr smd)
+		(attr smd dnp)
 		(fp_line
 			(start 2.76 3.21)
@@
 	(footprint "Capacitor_SMD:C_0201_0603Metric"
 		(layer "F.Cu")
-		(at 122.305 81.325 -90)
+		(at 120.505 81.225 -90)
 		(descr "Capacitor SMD 0201 (0603 Metric), square (rectangular) end terminal, IPC_7351 nominal, (Body size source: https://www.vishay.com/docs/20052/crcw0201e3.pdf), generated with kicad-footprint-generator")
 		(tags "capacitor")
@@
 	)
 	(segment
-		(start 122.3 82.3)
-		(end 122.305 82.295)
-		(width 0.1524)
-		(layer "F.Cu")
-		(net 1)
-	)
-	(segment
 		(start 130.685357 107.1)
 		(end 130.360357 107.425)
@@
 	)
 	(segment
+		(start 120.505 81.545)
+		(end 120.505 82.595)
+		(width 0.1524)
+		(layer "F.Cu")
+		(net 1)
+	)
+	(segment
 		(start 127.934301 101.8844)
 		(end 127.9844 101.834301)
@@
 		(net 1)
 	)
-	(segment
-		(start 122.305 81.645)
-		(end 122.305 82.295)
-		(width 0.1524)
-		(layer "F.Cu")
-		(net 1)
-	)
 	(via
 		(at 129.3 86.6)
@@
 	)
 	(via
-		(at 122.305 82.295)
+		(at 120.505 82.595)
 		(size 0.6096)
 		(drill 0.3)
@@
 	)
 	(segment
-		(start 125.03 81.005)
-		(end 122.305 81.005)
-		(width 0.1524)
-		(layer "F.Cu")
-		(net 2)
-	)
-	(segment
 		(start 151.0656 81.5344)
 		(end 150 82.6)
@@
 	)
 	(segment
+		(start 124.97 80.905)
+		(end 125.05 80.985)
+		(width 0.1524)
+		(layer "F.Cu")
+		(net 2)
+	)
+	(segment
 		(start 127.35 84.75)
 		(end 118.85 84.75)
@@
 		(width 0.1524)
 		(layer "F.Cu")
+		(net 2)
+	)
+	(segment
+		(start 120.505 80.905)
+		(end 124.97 80.905)
+		(width 0.1524)
+		(layer "F.Cu")
