File: hardware/tag-breakout-l432v1/tag-breakout-l432v1.kicad_sch (KiCad schematic)
At the start: 29 parts, among them J1 Conn_01x04_Female, J102 Conn_02x05_Odd_Even, J104 USB_B_Mini, J2 Conn_01x02_Male, SW1 SW_DIP_x04, U1 XC6206, U101 STM32F042K6Tx, U105 Tactile Switch, U2 TS5A3159ADBVR, U4 TS5A3159ADBVR

Commit message: checkpoint
Other:
- note added: "Check the use of pwr_in_mirror -- may need different pin for adc"
- note added: "control of swd is wrong. MISO/MOSI not connected correctly. Enable pin is wrong"
Changed lines of the file:
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@@
+		)
+	)
+	(text "Check the use of pwr_in_mirror -- may need different pin for adc"
+		(exclude_from_sim no)
+		(at 207.264 127.508 0)
+		(effects
+			(font
+				(size 1.27 1.27)
+			)
+		)
+	)
+	(text "control of swd is wrong.   MISO/MOSI not connected correctly.  Enable pin is wrong"
+		(exclude_from_sim no)
+		(at 230.378 85.344 0)
+		(effects
+			(font
+				(size 1.27 1.27)
+			)
 		)
 	)
