File: hardware/tag-breakout-l432v1/tag-breakout-l432v1.kicad_sch (KiCad schematic)
At the start: 29 parts, among them J1 Conn_01x04_Female, J102 Conn_02x05_Odd_Even, J104 USB_B_Mini, J2 Conn_01x02_Male, SW1 SW_DIP_x04, U1 XC6206, U101 STM32F042K6Tx, U105 Tactile Switch, U2 TS5A3159ADBVR, U4 TS5A3159ADBVR

Commit message: update prototype boards
Parts:
- removed U2: TS5A3159ADBVR, Package_TO_SOT_SMD:SOT-23-6, symbol Analog_Switch:TS5A3159ADBVR
Connections:
- net EXT_PWR: no longer U101.20 (PA10)
- net PWR_IN_MIRROR: now also U101.15 (PB1); no longer U101.19 (PA9)
- net TAG_SWDIO: now also R106.2, U101.12 (PA6)
Other:
- note removed: "Check the use of pwr_in_mirror -- may need different pin for adc"
- note removed: "control of swd is wrong. MISO/MOSI not connected correctly. Enable pin is wrong"
- moved on the sheet: U4B

Commit message: checkpoint
Parts:
- added TP1: SWDIO, TestPoint:TestPoint_Pad_D2.0mm, symbol Connector:TestPoint
- added TP2: SCK, TestPoint:TestPoint_Pad_D2.0mm, symbol Connector:TestPoint
Connections:
- net TAG_SCK: now also TP2.1
- net TAG_SWDIO: now also TP1.1
Other:
- title: Tag Breakout Board with stlink -> Tag Breakout Board with stm32l432k
- moved on the sheet: C1, C104, C107, C11, C2, D2, D3, U1

Commit message: Working board file for tag-breakout-base-l432-v1
Parts:
- D1: LCSC C72043 -> C5123548; MFN Everlight Elec -> Silverlight; MPN 19-217/GHC-YR1S2/3T -> P0603P1N46G12
Changed lines of the file:
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@@
 			)
 		)
-		(property "MPN" "19-217/GHC-YR1S2/3T"
+		(property "MPN" "P0603P1N46G12 "
 			(at 114.3 129.54 0)
 			(effects
@@
 			)
 		)
-		(property "LCSC" " C72043"
+		(property "LCSC" "C5123548"
 			(at 283.21 170.18 0)
 			(effects
@@
 			)
 		)
-		(property "MFN" "Everlight Elec"
+		(property "MFN" "Silverlight"
 			(at 283.21 170.18 0)
 			(effects
