File: hardware/tag-breakout-l432v1/tag-breakout-l432v1.kicad_pcb (KiCad board)
At the start: 2 copper layers, 53.3 x 73.7 mm, 43 parts, among them J1 Conn_01x04_Female, J102 Conn_02x05_Odd_Even, J104 USB_B_Mini, J2 Conn_01x02_Male, J3 Conn_01x17, J4 Conn_01x17, J5 Conn_01x02_Male, Q1 Q_NPN_BEC, SW1 SW_DIP_x04, U1 XC6206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

Commit message: checkpoint -- order compass proto board
Parts:
- R106: value 100 -> 200
- R2: value 36 -> 35.7
- U1: footprint Package_TO_SOT_SMD:SOT-23 -> Package_TO_SOT_SMD:SOT-23-3
- moved U1 0.22 mm to (142.4, 59.3)
Connections:
- R106 pad 1: Net-(U101-PA4) -> Net-(U101-PA7)
- U101 pad 10: Net-(U101-PA4) -> unconnected-(U101-PA4-Pad10)
- U101 pad 12: PWR_IN_MIRROR -> Net-(U101-PA6)
- U101 pad 13: unconnected-(U101-PA7-Pad13) -> Net-(U101-PA7)
- U101 pad 19: unconnected-(U101-PA9-Pad19) -> PWR_IN_MIRROR
- U101 pad 9: Net-(U101-PA3) -> unconnected-(U101-PA3-Pad9)
- U2 pad 6: Net-(U101-PA3) -> Net-(U101-PA6)
Routing:
- net Net-(U101-PA6): track 0.00 -> 9.62 mm
- net Net-(U101-PA7): track 0.00 -> 8.60 mm
- net Net-(U101-PA3): track 5.90 -> 0.00 mm
- net Net-(U101-PA4): track 5.27 -> 0.00 mm
- net PWR_IN_MIRROR: track 21.3 -> 24.2 mm, vias 0 -> 2
- net TAG_SCK: track 24.8 -> 24.7 mm, vias 2 -> 4

Commit message: update proto boards
Parts:
- J3, J4: footprint Connector_PinSocket_2.54mm:PinSocket_1x17_P2.54mm_Vertical -> library:PinHeader_1x17_P2.54mm_Vertical_Staggered
Other:
- board text added: "3V3 src"
- board text added: "Geoffrey Brown 6/6/25"
- board text added: "TAG_3v3"
- board text removed: "Geoffrey Brown 4/28/25"

Commit message: update prototype boards
Parts:
- removed U2: TS5A3159ADBVR, Package_TO_SOT_SMD:SOT-23-6
- moved R106 2.17 mm to (136.1, 80.5), turned to 180 degrees
Connections:
- R106 pad 2: Net-(R106-Pad2) -> TAG_SWDIO
- U101 pad 12: Net-(U101-PA6) -> TAG_SWDIO
- U101 pad 15: unconnected-(U101-PB1-Pad15) -> PWR_IN_MIRROR
- U101 pad 19: PWR_IN_MIRROR -> unconnected-(U101-PA9-Pad19)
- U101 pad 20: EXT_PWR -> unconnected-(U101-PA10-Pad20)
Routing:
- net TAG_SWDIO: track 12.7 -> 23.6 mm
- net Net-(U101-PA6): track 9.62 -> 0.00 mm
- net +3V3: track 94.1 -> 85.4 mm
- net EXT_PWR: track 39.7 -> 31.6 mm
- net PWR_IN_MIRROR: track 24.2 -> 20.3 mm, vias 2 -> 0
- net TAG_SCK: track 24.7 -> 21.5 mm, vias 4 -> 2
- net Net-(R106-Pad2): track 2.01 -> 0.00 mm
- net GND: track 65.2 -> 64.2 mm, vias 29 -> 28

Commit message: checkpoint
Parts:
- removed J5: Conn_01x02_Male, Connector_PinHeader_2.54mm:PinHeader_1x02_P2.54mm_Vertical
- added TP1: SWDIO, TestPoint:TestPoint_Pad_D2.0mm, B.Cu at (137.9, 88.8)
- added TP2: SCK, TestPoint:TestPoint_Pad_D2.0mm, B.Cu at (132.2, 91.4)
- moved C9 2.87 mm to (126.2, 100.1), turned to -90 degrees
- moved R106 2.84 mm to (135.6, 77.7), turned to -90 degrees
Connections:
- C10 pad 1: /stm32/TAG_PWR -> TAG_3V3
- C3 pad 1: /stm32/TAG_PWR -> TAG_3V3
- C4 pad 1: /stm32/TAG_PWR -> TAG_3V3
- C6 pad 1: /stm32/TAG_PWR -> TAG_3V3
- C7 pad 1: /stm32/TAG_PWR -> TAG_3V3
- C9 pad 1: /stm32/TAG_PWR -> TAG_3V3
- J3 pad 7: /stm32/TAG_PWR -> TAG_3V3
- J4 pad 1: /stm32/TAG_PWR -> TAG_3V3
- U3 pad 1: /stm32/TAG_PWR -> TAG_3V3
- U3 pad 17: /stm32/TAG_PWR -> TAG_3V3
- U3 pad 5: /stm32/TAG_PWR -> TAG_3V3
- U6 pad 7: /stm32/TAG_PWR -> TAG_3V3
Routing:
- net /stm32/TAG_PWR: track 102.4 -> 0.00 mm, vias 4 -> 0
- net TAG_3V3: track 9.38 -> 105.1 mm, vias 0 -> 4
- net Net-(U101-PA7): track 8.30 -> 3.63 mm
- net TAG_SCK: track 21.5 -> 24.4 mm
- net +3V3: track 85.4 -> 83.0 mm, vias 2 -> 1
- net /stm32/rtc_sda: track 37.2 -> 35.7 mm
Other:
- board text added: "SCK"
- board text added: "SWDIO"
- board text removed: "3V3 src"
- board text removed: "TAG_3v3"
