File: hardware/BitPresTagBreakout/BitPresTagBreakout.kicad_pcb (KiCad board)
At the start: 2 copper layers, 48.3 x 48.3 mm, 10 parts, among them J3 Conn_01x17, J4 Conn_01x17, U2 AT25XE321, U3 LPS27HHWTR, U4 adxl362

Commit message: checkpoint
Parts:
- moved C9 2.00 mm to (121.2, 81.3)
Routing:
- net /TAG_3V3: track 114.0 -> 116.0 mm
Changed lines of the file:
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@@
 	(footprint "Capacitor_SMD:C_0201_0603Metric"
 		(layer "F.Cu")
-		(at 123.205 81.325 -90)
+		(at 121.205 81.325 -90)
 		(descr "Capacitor SMD 0201 (0603 Metric), square (rectangular) end terminal, IPC_7351 nominal, (Body size source: https://www.vishay.com/docs/20052/crcw0201e3.pdf), generated with kicad-footprint-generator")
 		(tags "capacitor")
@@
 	)
 	(segment
-		(start 123.2 82.3)
-		(end 123.205 82.295)
+		(start 121.2 82.3)
+		(end 121.205 82.295)
 		(width 0.1524)
 		(layer "F.Cu")
@@
 	)
 	(segment
-		(start 123.205 81.645)
-		(end 123.205 82.295)
+		(start 121.205 81.645)
+		(end 121.205 82.295)
 		(width 0.1524)
 		(layer "F.Cu")
@@
 	)
 	(via
-		(at 123.205 82.295)
+		(at 121.205 82.295)
 		(size 0.6096)
 		(drill 0.3)
@@
 	)
 	(segment
-		(start 125.03 81.005)
-		(end 125.05 80.985)
-		(width 0.1524)
-		(layer "F.Cu")
-		(net 2)
-	)
-	(segment
 		(start 127.35 84.75)
 		(end 118.85 84.75)
@@
 	)
 	(segment
-		(start 105.703 92.29)
-		(end 106.553 91.44)
+		(start 125.03 81.005)
+		(end 125.05 80.985)
 		(width 0.1524)
 		(layer "F.Cu")
@@
 	)
 	(segment
-		(start 123.205 81.005)
+		(start 121.205 81.005)
 		(end 125.03 81.005)
 		(width 0.1524)
 		(layer "F.Cu")
+		(net 2)
+	)
+	(segment
+		(start 105.703 92.29)
+		(end 106.553 91.44)
+		(width 0.1524)
+		(layer "F.Cu")

Commit message: checkpoint -- order compass proto board
Other:
- board text added: "Geoffrey Brown 6/3/2025"
- board text removed: "Geoffrey Brown 4/17/2025"
Changed lines of the file:
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@@
 		(sheetname "Root")
 		(sheetfile "BitPresTagBreakout.kicad_sch")
-		(attr smd)
+		(attr smd dnp)
 		(fp_line
 			(start 2.76 3.21)
@@
 			)
 		)
+		(property "LCSC" "C3253631"
+			(at 0 0 -90)
+			(unlocked yes)
+			(layer "F.Fab")
+			(hide yes)
+			(effects
+				(font
+					(size 1 1)
+					(thickness 0.15)
+				)
+			)
+		)
 		(property ki_fp_filters "QFN_HHWTR_STM QFN_HHWTR_STM-M QFN_HHWTR_STM-L")
 		(sheetname "Root")
@@
 			)
 		)
+		(property "LCSC" "C181047"
+			(at 0 0 0)
+			(unlocked yes)
+			(layer "F.Fab")
+			(hide yes)
+			(effects
+				(font
+					(size 1 1)
+					(thickness 0.15)
+				)
+			)
+		)
 		(property ki_fp_filters "C_*")
 		(sheetname "Root")
@@
 			)
 		)
-		(property "MFN" ""
+		(property "MFN" "Murata"
 			(at 0 0 -90)
 			(unlocked yes)
@@
 			)
 		)
-		(property "MPN" "CL05F104ZO5NNNC"
+		(property "MPN" "GRM033C81E104KE14D"
+			(at 0 0 -90)
+			(unlocked yes)
+			(layer "F.Fab")
+			(hide yes)
+			(effects
+				(font
+					(size 1 1)
+					(thickness 0.15)
+				)
+			)
+		)
+		(property "LCSC" "C181047"
 			(at 0 0 -90)
 			(unlocked yes)
@@
 			)
 		)
+		(property "LCSC" "C192252"
+			(at 0 0 0)
+			(unlocked yes)
+			(layer "F.Fab")
+			(hide yes)
+			(effects
+				(font
+					(size 1 1)
+					(thickness 0.15)
+				)
+			)
+		)
 		(sheetname "Root")
 		(sheetfile "BitPresTagBreakout.kicad_sch")
@@
 		(layer "Edge.Cuts")
 	)
-	(gr_text "Geoffrey Brown\n4/17/2025"
+	(gr_text "Geoffrey Brown\n6/3/2025"
 		(at 130.59 112.98 0)
 		(layer "B.SilkS")
