File: hardware/CompassTag/CompassTag.kicad_pcb (KiCad board)
At the start: 2 copper layers, 18 x 9 mm, 28 parts, among them J201 CONN_02X04, J301 Conn_01x01, J302 Conn_01x01, J303 Conn_01x01, J304 Conn_01x01, J401 CONN_01X02, Q501 Q_NPN_BEC, U1 at25ex321D-UUN, U2 AK09940A, U3 LIS2DU12TR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

Commit message: checkpoint
Connections:
- U2 pad A4: /AK_MISO -> /AK_MOSI
- U2 pad B4: /AK_MOSI -> /AK_MISO
Routing:
- net /AK_MOSI: track 2.60 -> 3.96 mm, vias 0 -> 2
- net /USART2_CK: track 2.25 -> 3.54 mm
- net /AK_CK: track 3.05 -> 4.25 mm

Commit message: checkpoint
Connections:
- U2 pad A1: unconnected-(U2-DRDY/TRG-PadA1) -> /AK_DRDY
- U302 pad 20: unconnected-(U302-PA10-Pad20) -> /AK_DRDY
Routing:
- net /AK_DRDY: track 0.00 -> 11.9 mm
Other:
- board text added: "CpTag V1"
- board text added: "X"
- board text added: "Y"
- board text removed: "BTNG V2"
Changed lines of the file:
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@@
 	(net 26 "unconnected-(U302-PA12-Pad22)")
 	(net 27 "unconnected-(U302-PA11-Pad21)")
-	(net 28 "unconnected-(U302-PA10-Pad20)")
+	(net 28 "/AK_DRDY")
 	(net 29 "/USART2_RX")
 	(net 30 "/WKUP1")
@@
 	(net 37 "/AK_RSTN")
 	(net 38 "/AK_MOSI")
-	(net 39 "unconnected-(U2-DRDY{slash}TRG-PadA1)")
-	(net 40 "/AK_CS")
+	(net 39 "/AK_CS")
 	(footprint "AccelTag:taghole1.1mm"
 		(layer "F.Cu")
@@
 			(pintype "input")
 		)
-		(model "${KIPRJMOD}/LGA-12L_LIS2DU12_STM.step"
-			(offset
-				(xyz 0 0 0)
-			)
-			(scale
-				(xyz 1 1 1)
-			)
-			(rotate
-				(xyz 0 0 0)
-			)
-		)
 	)
 	(footprint "Capacitor_SMD:C_0201_0603Metric"
@@
 			(layers "B.Cu" "B.Paste" "B.Mask")
 			(roundrect_rratio 0.25)
-			(net 40 "/AK_CS")
+			(net 39 "/AK_CS")
 			(pinfunction "PB1")
 			(pintype "bidirectional")
@@
 			(layers "B.Cu" "B.Paste" "B.Mask")
 			(roundrect_rratio 0.25)
-			(net 28 "unconnected-(U302-PA10-Pad20)")
+			(net 28 "/AK_DRDY")
 			(pinfunction "PA10")
-			(pintype "bidirectional+no_connect")
+			(pintype "bidirectional")
 		)
 		(pad "21" smd roundrect
@@
 			(size 0.2286 0.2286)
 			(layers "B.Cu" "B.Paste" "B.Mask")
-			(net 39 "unconnected-(U2-DRDY{slash}TRG-PadA1)")
+			(net 28 "/AK_DRDY")
 			(pinfunction "DRDY/TRG")
-			(pintype "bidirectional+no_connect")
+			(pintype "bidirectional")
 		)
 		(pad "A2" smd circle
@@
 			(size 0.2286 0.2286)
 			(layers "B.Cu" "B.Paste" "B.Mask")
-			(net 40 "/AK_CS")
+			(net 39 "/AK_CS")
 			(pinfunction "CSB")
 			(pintype "input")
@@
 	)
 	(gr_line
+		(start 142.1 111.7)
+		(end 142.3 111.9)
+		(stroke
+			(width 0.15)
+			(type default)
+		)
+		(layer "F.SilkS")
+	)
+	(gr_line
+		(start 143 110.8)
+		(end 142.8 111)
+		(stroke
+			(width 0.15)
+			(type default)
+		)
+		(layer "F.SilkS")
+	)
+	(gr_line
+		(start 143 111.7)
+		(end 142.1 111.7)
+		(stroke
+			(width 0.15)
+			(type default)
+		)
+		(layer "F.SilkS")
+	)
+	(gr_line
+		(start 143 111.7)
+		(end 143 110.8)
+		(stroke
+			(width 0.15)
+			(type default)
+		)
+		(layer "F.SilkS")
+	)
+	(gr_line
+		(start 142.9 111.6)
+		(end 142.6 111.4)
+		(stroke
+			(width 0.15)
+			(type default)
+		)
+		(layer "F.SilkS")
+	)
+	(gr_line
 		(start 111.37 127.95)
 		(end 111.37 127.95)
@@
 		(layer "Edge.Cuts")
 	)
-	(gr_text "BTNG  V2"
+	(gr_text "CpTag V1"
 		(at 157.3 108.4 90)
 		(layer "B.SilkS")
@@
 		)
 	)
+	(gr_text "X"
+		(at 142.7 112.9 0)
+		(layer "F.SilkS")
+		(effects
+			(font
+				(size 0.75 0.75)
+				(thickness 0.15)
+			)
+			(justify left bottom mirror)
+		)
+	)
+	(gr_text "Y"
+		(at 143.85 111.7 0)
+		(layer "F.SilkS")
+		(effects
+			(font
+				(size 0.75 0.75)
+				(thickness 0.15)
+			)
+			(justify left bottom mirror)
+		)
+	)
 	(segment
 		(start 146.905501 108.876358)
@@
 	)
 	(segment
-		(start 141.7 108.7)
-		(end 141.7684 108.7684)
-		(width 0.1016)
-		(layer "B.Cu")
-		(net 1)
-	)
-	(segment
 		(start 149.8875 110.216458)
 		(end 149.8875 109.716458)
@@
 	)
 	(segment
+		(start 141.25 107.2)
+		(end 140.8682 107.5818)
+		(width 0.1016)
+		(layer "B.Cu")
+		(net 28)
+	)
+	(segment
+		(start 143.4 104.95)
+		(end 142.05 106.3)
+		(width 0.1016)
+		(layer "B.Cu")
+		(net 28)
+	)
+	(segment
+		(start 147.2 105.55)
+		(end 146.6 104.95)
+		(width 0.1016)
+		(layer "B.Cu")
+		(net 28)
+	)
+	(segment
+		(start 141.0184 109.9684)
+		(end 141.7684 109.9684)
+		(width 0.1016)
+		(layer "B.Cu")
+		(net 28)
+	)
+	(segment
+		(start 142.05 106.3)
+		(end 141.25 106.3)
+		(width 0.1016)
+		(layer "B.Cu")
+		(net 28)
+	)
+	(segment
+		(start 141.25 106.3)
+		(end 141.25 107.2)
+		(width 0.1016)
+		(layer "B.Cu")
+		(net 28)
+	)
+	(segment
+		(start 146.6 104.95)
+		(end 143.4 104.95)
+		(width 0.1016)
+		(layer "B.Cu")
+		(net 28)
+	)
+	(segment
+		(start 140.8682 109.8182)
+		(end 141.0184 109.9684)
+		(width 0.1016)
+		(layer "B.Cu")
+		(net 28)
+	)
+	(segment
+		(start 147.2 106.028958)
+		(end 147.2 105.55)
+		(width 0.1016)
+		(layer "B.Cu")
+		(net 28)
+	)
+	(segment
+		(start 140.8682 107.5818)
+		(end 140.8682 109.8182)
+		(width 0.1016)
+		(layer "B.Cu")
+		(net 28)
+	)
+	(segment
 		(start 146.4055 110.489258)
 		(end 146.4055 110.476558)
@@
 		(width 0.1016)
 		(layer "B.Cu")
-		(net 40)
+		(net 39)
 	)
 	(segment
@@
 		(width 0.1016)
 		(layer "B.Cu")
-		(net 40)
+		(net 39)
 	)
 	(segment
@@
 		(width 0.1016)
 		(layer "B.Cu")
-		(net 40)
+		(net 39)
 	)
 	(segment
@@
 		(width 0.1016)
 		(layer "B.Cu")
-		(net 40)
+		(net 39)
 	)
 	(segment
@@
 		(width 0.1016)
 		(layer "B.Cu")
-		(net 40)
+		(net 39)
 	)
 	(segment
@@
 		(width 0.1016)
 		(layer "B.Cu")
-		(net 40)
+		(net 39)
 	)
 )

Commit message: tweak compasstag
Parts:
- C501: moved to F.Cu
- D401: moved to B.Cu
- moved J301 0.92 mm to (155.2, 111.7)
- moved J302 0.92 mm to (155.2, 105.2)
- moved D401 0.55 mm to (152.0, 111.3), turned to 0 degrees
- moved U3 0.38 mm to (145.9, 109.9)
Routing:
- net VBAT: track 7.73 -> 8.37 mm, vias 1 -> 2
- net /USART2_TX: track 5.70 -> 5.14 mm
- net VIN: track 39.4 -> 38.9 mm
Other:
- board text removed: "X"
- board text removed: "Y"

Commit message: tweek compass tag
Connections:
- C5 pad 1: /AK_PWR -> VIN
- U2 pad C4: /AK_PWR -> VIN
Routing:
- net VIN: track 38.9 -> 42.8 mm, vias 5 -> 6
- net /AK_PWR: track 9.54 -> 6.03 mm, vias 2 -> 1
Other:
- board text added: "1"
Changed lines of the file:
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@@
 			(pintype "input")
 		)
-		(model "$KIPRJMOD/../kicad_libraries/3d_models/LIS2DW12.STEP"
+		(model "${KIPRJMOD}/LGA-12L_LIS2DU12_STM.step"
 			(offset
 				(xyz 0 0 0)
@@
 			)
 			(rotate
-				(xyz -90 0 180)
+				(xyz 0 0 0)
 			)
 		)
@@
 		(tags "diode")
 		(property "Reference" "D401"
-			(at 0 1.17 360)
+			(at 0 1.17 0)
 			(layer "B.SilkS")
 			(hide yes)
@@
 		)
 		(property "Value" "D"
-			(at 0 -1.17 360)
+			(at 0 -1.17 0)
 			(layer "B.Fab")
 			(hide yes)
@@
 		)
 		(property "Footprint" "Diode_SMD:D_0402_1005Metric"
-			(at 0 0 360)
+			(at 0 0 0)
 			(layer "B.Fab")
 			(hide yes)
@@
 		)
 		(property "Datasheet" ""
-			(at 0 0 360)
+			(at 0 0 0)
 			(layer "B.Fab")
 			(hide yes)
@@
 		)
 		(property "Description" ""
-			(at 0 0 360)
+			(at 0 0 0)
 			(layer "B.Fab")
 			(hide yes)
@@
 		)
 		(property "DISTPN" "641-1519-1-ND"
-			(at 0 0 360)
+			(at 0 0 0)
 			(layer "B.Fab")
 			(hide yes)
@@
 		)
 		(property "LCSC" "C2886012"
-			(at 0 0 360)
+			(at 0 0 0)
 			(layer "B.Fab")
 			(hide yes)
@@
 		)
 		(property "MFN" "COMCHIP"
-			(at 0 0 360)
+			(at 0 0 0)
 			(layer "B.Fab")
 			(hide yes)
@@
 		)
 		(property "MPN" "CDBQC0130L-HF"
-			(at 0 0 360)
+			(at 0 0 0)
 			(layer "B.Fab")
 			(hide yes)
@@
 		)
 		(fp_text user "${REFERENCE}"
-			(at 0 0 360)
+			(at 0 0 0)
 			(layer "B.Fab")
 			(hide yes)
@@
 			(layers "B.Cu" "B.Mask")
 			(roundrect_rratio 0.25)
-			(net 33 "/AK_PWR")
+			(net 10 "VIN")
 			(pintype "passive")
 		)
@@
 			(size 0.2286 0.2286)
 			(layers "B.Cu" "B.Paste" "B.Mask")
-			(net 33 "/AK_PWR")
+			(net 10 "VIN")
 			(pinfunction "VOD")
 			(pintype "power_in")
@@
 	)
 	(gr_line
-		(start 142.4 112.15)
-		(end 142.6 112.35)
+		(start 151.2 111.7)
+		(end 151 111.7)
 		(stroke
 			(width 0.15)
 			(type default)
 		)
-		(layer "F.SilkS")
+		(layer "B.SilkS")
 	)
 	(gr_line
-		(start 143.3 111.25)
-		(end 143.1 111.45)
+		(start 141.2 110.2)
+		(end 141.2 110.5)
 		(stroke
 			(width 0.15)
 			(type default)
 		)
-		(layer "F.SilkS")
+		(layer "B.SilkS")
 	)
 	(gr_line
-		(start 143.3 112.15)
-		(end 142.4 112.15)
+		(start 151 111.1)
+		(end 151 110.9)
 		(stroke
 			(width 0.15)
 			(type default)
 		)
-		(layer "F.SilkS")
+		(layer "B.SilkS")
 	)
 	(gr_line
-		(start 143.3 112.15)
-		(end 143.3 111.25)
+		(start 141.6 110.5)
+		(end 141.2 110.5)
 		(stroke
 			(width 0.15)
 			(type default)
 		)
-		(layer "F.SilkS")
+		(layer "B.SilkS")
 	)
 	(gr_line
-		(start 143.2 112.05)
-		(end 142.9 111.85)
+		(start 151 110.9)
+		(end 151.2 110.9)
 		(stroke
 			(width 0.15)
 			(type default)
 		)
-		(layer "F.SilkS")
+		(layer "B.SilkS")
+	)
+	(gr_line
+		(start 151 111.5)
+		(end 151 111.7)
+		(stroke
+			(width 0.15)
+			(type default)
+		)
+		(layer "B.SilkS")
 	)
 	(gr_line
@@
 		)
 	)
+	(gr_text "1"
+		(at 141.2 111 0)
+		(layer "B.SilkS")
+		(effects
+			(font
+				(size 0.8 0.8)
+				(thickness 0.15)
+			)
+			(justify left bottom mirror)
+		)
+	)
+	(gr_text "1"
+		(at 143.6 112.2 0)
+		(layer "F.SilkS")
+		(effects
+			(font
+				(size 0.8 0.8)
+				(thickness 0.15)
+			)
+			(justify left bottom)
+		)
+	)
 	(segment
 		(start 146.100001 109.0998)
@@
 	)
 	(segment
+		(start 145.52 107.8)
+		(end 144.92 108.4)
+		(width 0.1016)
+		(layer "F.Cu")
+		(net 10)
+	)
+	(segment
 		(start 147.2 111.2)
 		(end 147.5134 111.5134)
@@
 	)
 	(segment
+		(start 144.92 108.4)
+		(end 143.7 108.4)
+		(width 0.1016)
+		(layer "F.Cu")
+		(net 10)
+	)
+	(segment
 		(start 149.996516 106.276458)
 		(end 150.216974 106.056)
@@
 	)
 	(via
+		(at 143.7 108.4)
+		(size 0.4572)
+		(drill 0.254)
+		(layers "F.Cu" "B.Cu")
+		(net 10)
+	)
+	(via
 		(at 143.2 106.1)
 		(size 0.4572)
@@
 	)
 	(segment
+		(start 143.7 108.4368)
+		(end 142.9684 109.1684)
+		(width 0.1016)
+		(layer "B.Cu")
+		(net 10)
+	)
+	(segment
 		(start 142.795 106.675)
 		(end 142.795 106.505)
@@
 	)
 	(segment
+		(start 143.7 108.4)
+		(end 143.7 108.4368)
+		(width 0.1016)
+		(layer "B.Cu")
+		(net 10)
+	)
+	(segment
 		(start 151.68 109.571)
 		(end 152.935 109.571)
@@
 	)
 	(segment
+		(start 142.845 106.725)
+		(end 142.795 106.675)
+		(width 0.1016)
+		(layer "B.Cu")
+		(net 10)
+	)
+	(segment
 		(start 149.2326 110.936558)
 		(end 149.2 110.903958)
@@
 	)
 	(segment
+		(start 142.845 107.475)
+		(end 142.845 106.725)
+		(width 0.1016)
+		(layer "B.Cu")
+		(net 10)
+	)
+	(segment
 		(start 142.795 106.505)
 		(end 143.2 106.1)
@@
 		(net 33)
 	)
-	(segment
-		(start 142.939643 107.425)
-		(end 143.634089 108.119446)
-		(width 0.1016)
-		(layer "F.Cu")
-		(net 33)
-	)
-	(segment
-		(start 143.634089 108.119446)
-		(end 143.634089 108.390149)
-		(width 0.1016)
-		(layer "F.Cu")
-		(net 33)
-	)
 	(via
 		(at 143.915094 107.161489)
@@
 		(net 33)
 	)
-	(via
-		(at 143.634089 108.390149)
-		(size 0.4572)
-		(drill 0.254)
-		(layers "F.Cu" "B.Cu")
-		(net 33)
-	)
 	(segment
 		(start 146.376741 105.2682)
@@
 	)
 	(segment
-		(start 142.9684 109.1684)
-		(end 143.634089 108.502711)
-		(width 0.1016)
-		(layer "B.Cu")
-		(net 33)
-	)
-	(segment
-		(start 143.634089 108.502711)
-		(end 143.634089 108.390149)
-		(width 0.1016)
-		(layer "B.Cu")
-		(net 33)
-	)
-	(segment
-		(start 143.158511 107.161489)
-		(end 143.915094 107.161489)
-		(width 0.1016)
-		(layer "B.Cu")
-		(net 33)
-	)
-	(segment
 		(start 144.6 105.2682)
 		(end 143.8 106.0682)
 		(width 0.1016)
 		(layer "B.Cu")
-		(net 33)
-	)
-	(segment
-		(start 142.845 107.475)
-		(end 143.158511 107.161489)
-		(width 0.1016)
-		(layer "B.Cu")

Commit message: update compasstag hardware
Other:
- board text added: "CTag V1"
- board text removed: "CpTag V1"
Changed lines of the file:
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@@
 		(sheetname "Root")
 		(sheetfile "CompassTag.kicad_sch")
-		(attr through_hole exclude_from_bom)
+		(attr through_hole exclude_from_bom dnp)
 		(pad "" np_thru_hole circle
 			(at 0 0)
 			(size 1.1 1.1)
 			(drill 1.1)
-			(layers "*.Cu" "*.Mask" "In1.Cu" "In2.Cu" "In3.Cu" "In4.Cu" "In5.Cu" "In6.Cu"
-				"In7.Cu" "In8.Cu" "In9.Cu" "In10.Cu" "In11.Cu" "In12.Cu" "In13.Cu" "In14.Cu"
-				"In15.Cu" "In16.Cu" "In17.Cu" "In18.Cu" "In19.Cu" "In20.Cu" "In21.Cu"
-				"In22.Cu" "In23.Cu" "In24.Cu" "In25.Cu" "In26.Cu" "In27.Cu" "In28.Cu"
-				"In29.Cu" "In30.Cu"
-			)
+			(layers "*.Cu" "*.Mask")
 		)
 	)
@@
 		(sheetname "Root")
 		(sheetfile "CompassTag.kicad_sch")
-		(attr smd exclude_from_bom)
+		(attr smd exclude_from_bom dnp)
 		(fp_text user "+"
 			(at 0.3 -2 180)
@@
 			)
 		)
+		(model "${KIPRJMOD}/../kicad_libraries/3d_models/BatteryHolder_Seiko_MS621F.step"
+			(hide yes)
+			(offset
+				(xyz 0 0 0)
+			)
+			(scale
+				(xyz 1 1 1)
+			)
+			(rotate
+				(xyz 0 0 0)
+			)
+		)
 	)
 	(footprint "AccelTag:RV-8803-C7"
@@
 		)
 		(model "${KIPRJMOD}/packages3D/RV-3028-C7.wrl"
+			(hide yes)
 			(offset
 				(xyz 0 0 0)
@@
 			(pintype "passive")
 		)
-		(model "${KIPRJMOD}/packages3D/R_0201_0603Metric.wrl"
+		(model "${KIPRJMOD}/packages3D/R_0201_0603Metric.step"
 			(offset
 				(xyz 0 0 0)
@@
 			)
 		)
-		(property "DISTPN" "490-10403-1-ND"
+		(property "DISTPN" "81-GRM033R60J105ME2D"
 			(at 258.6628 -37.766 0)
 			(layer "F.Fab")
@@
 			)
 		)
-		(property "MPN" "C181047"
+		(property "MPN" "GRM033R60J105MEA2D"
 			(at 258.6628 -37.766 0)
 			(layer "F.Fab")
@@
 			(pintype "passive")
 		)
-		(model "${KIPRJMOD}/packages3D/C_0201_0603Metric.wrl"
+		(model "${KIPRJMOD}/packages3D/C_0201_0603Metric.step"
 			(offset
 				(xyz 0 0 0)
@@
 			)
 		)
-		(property "DISTPN" "490-10403-1-ND"
+		(property "DISTPN" "81-GRM033R60J105ME2D"
 			(at 0 0 90)
 			(layer "F.Fab")
@@
 			)
 		)
-		(property "MPN" "C181047"
+		(property "MPN" "GRM033R60J105MEA2D"
 			(at 0 0 90)
 			(layer "F.Fab")
@@
 			(pintype "passive")
 		)
-		(model "${KIPRJMOD}/packages3D/C_0201_0603Metric.wrl"
+		(model "${KIPRJMOD}/packages3D/C_0201_0603Metric.step"
 			(offset
 				(xyz 0 0 0)
@@
 			)
 		)
-		(property "DISTPN" "490-10403-1-ND"
+		(property "DISTPN" "81-GRM033R60J105ME2D"
 			(at 0 0 0)
 			(layer "F.Fab")
@@
 			)
 		)
-		(property "MPN" "C181047"
+		(property "MPN" "GRM033R60J105MEA2D"
 			(at 0 0 0)
 			(layer "F.Fab")
@@
 			(pintype "passive")
 		)
-		(model "${KIPRJMOD}/packages3D/C_0201_0603Metric.wrl"
+		(model "${KIPRJMOD}/packages3D/C_0201_0603Metric.step"
 			(offset
 				(xyz 0 0 0)
@@
 		(sheetname "Root")
 		(sheetfile "CompassTag.kicad_sch")
-		(attr through_hole exclude_from_bom)
+		(attr through_hole exclude_from_bom dnp)
 		(pad "" np_thru_hole circle
 			(at 0 0)
 			(size 1.1 1.1)
 			(drill 1.1)
-			(layers "*.Cu" "*.Mask" "In1.Cu" "In2.Cu" "In3.Cu" "In4.Cu" "In5.Cu" "In6.Cu"
-				"In7.Cu" "In8.Cu" "In9.Cu" "In10.Cu" "In11.Cu" "In12.Cu" "In13.Cu" "In14.Cu"
-				"In15.Cu" "In16.Cu" "In17.Cu" "In18.Cu" "In19.Cu" "In20.Cu" "In21.Cu"
-				"In22.Cu" "In23.Cu" "In24.Cu" "In25.Cu" "In26.Cu" "In27.Cu" "In28.Cu"
-				"In29.Cu" "In30.Cu"
-			)
+			(layers "*.Cu" "*.Mask")
 		)
 	)
@@
 		(sheetname "Root")
 		(sheetfile "CompassTag.kicad_sch")
-		(attr through_hole exclude_from_bom)
+		(attr through_hole exclude_from_bom dnp)
 		(pad "" np_thru_hole circle
 			(at 0 0)
 			(size 1.1 1.1)
 			(drill 1.1)
-			(layers "*.Cu" "*.Mask" "In1.Cu" "In2.Cu" "In3.Cu" "In4.Cu" "In5.Cu" "In6.Cu"
-				"In7.Cu" "In8.Cu" "In9.Cu" "In10.Cu" "In11.Cu" "In12.Cu" "In13.Cu" "In14.Cu"
-				"In15.Cu" "In16.Cu" "In17.Cu" "In18.Cu" "In19.Cu" "In20.Cu" "In21.Cu"
-				"In22.Cu" "In23.Cu" "In24.Cu" "In25.Cu" "In26.Cu" "In27.Cu" "In28.Cu"
-				"In29.Cu" "In30.Cu"
-			)
+			(layers "*.Cu" "*.Mask")
 		)
 	)
@@
 		(sheetname "Root")
 		(sheetfile "CompassTag.kicad_sch")
-		(attr through_hole exclude_from_bom)
+		(attr through_hole exclude_from_bom dnp)
 		(pad "" np_thru_hole circle
 			(at 0 0)
 			(size 1.1 1.1)
 			(drill 1.1)
-			(layers "*.Cu" "*.Mask" "In1.Cu" "In2.Cu" "In3.Cu" "In4.Cu" "In5.Cu" "In6.Cu"
-				"In7.Cu" "In8.Cu" "In9.Cu" "In10.Cu" "In11.Cu" "In12.Cu" "In13.Cu" "In14.Cu"
-				"In15.Cu" "In16.Cu" "In17.Cu" "In18.Cu" "In19.Cu" "In20.Cu" "In21.Cu"
-				"In22.Cu" "In23.Cu" "In24.Cu" "In25.Cu" "In26.Cu" "In27.Cu" "In28.Cu"
-				"In29.Cu" "In30.Cu"
-			)
+			(layers "*.Cu" "*.Mask")
 		)
 	)
@@
 			(pintype "passive")
 		)
-		(model "${KICAD6_3DMODEL_DIR}/Package_TO_SOT_SMD.3dshapes/SOT-883.wrl"
-			(offset
-				(xyz 0 0 0)
-			)
-			(scale
-				(xyz 1 1 1)
-			)
-			(rotate
-				(xyz 0 0 0)
-			)
-		)
 		(model "${KIPRJMOD}/packages3D/Diodes_DFN1006-3.step"
 			(offset
@@
 			)
 		)
-		(property "DISTPN" "490-10403-1-ND"
+		(property "DISTPN" "81-GRM033R60J105ME2D"
 			(at 0 0 0)
 			(layer "F.Fab")
@@
 			)
 		)
-		(property "MPN" "C181047"
+		(property "MPN" "GRM033R60J105MEA2D"
 			(at 0 0 0)
 			(layer "F.Fab")
@@
 			(pintype "passive")
 		)
-		(model "${KIPRJMOD}/packages3D/C_0201_0603Metric.wrl"
+		(model "${KIPRJMOD}/packages3D/C_0201_0603Metric.step"
 			(offset
 				(xyz 0 0 0)
@@
 			)
 		)
-		(property "DISTPN" "490-7229-2-ND"
+		(property "DISTPN" "81-GRM033R60J105ME2D"
 			(at 284.34 218.142 0)
 			(layer "F.Fab")
@@
 			)
 		)
-		(property "MFN" "murata"
+		(property "MFN" "Murata"
 			(at 284.34 218.142 0)
 			(layer "F.Fab")
@@
 			(pintype "passive")
 		)
-		(model "${KIPRJMOD}/packages3D/C_0201_0603Metric.wrl"
+		(model "${KIPRJMOD}/packages3D/C_0201_0603Metric.step"
 			(offset
 				(xyz 0 0 0)
@@
 			)
 		)
+		(property "DISTPN" "497-LIS2DU12TRCT-ND"
+			(at 0 0 90)
+			(unlocked yes)
+			(layer "F.Fab")
+			(hide yes)
+			(effects
+				(font
+					(size 1 1)
+					(thickness 0.15)
+				)
+			)
+		)
+		(property "MFN" "STMicroelectroincs"
+			(at 0 0 90)
+			(unlocked yes)
+			(layer "F.Fab")
+			(hide yes)
+			(effects
+				(font
+					(size 1 1)
+					(thickness 0.15)
+				)
+			)
+		)
+		(property "MPN" "LIS2DU12TR"
+			(at 0 0 90)
+			(unlocked yes)
+			(layer "F.Fab")
+			(hide yes)
+			(effects
+				(font
+					(size 1 1)
+					(thickness 0.15)
+				)
+			)
+		)
 		(property ki_fp_filters "LGA-12L_LIS2DU12_STM LGA-12L_LIS2DU12_STM-M LGA-12L_LIS2DU12_STM-L")
 		(sheetname "Root")
@@
 			)
 		)
-		(property "DISTPN" "490-10403-1-ND"
+		(property "DISTPN" "81-GRM033R60J105ME2D"
 			(at 0 0 180)
 			(unlocked yes)
@@
 			)
 		)
-		(property "MPN" "C181047"
+		(property "MPN" "GRM033R60J105MEA2D"
 			(at 0 0 180)
 			(unlocked yes)
@@
 			(pintype "passive")
 		)
-		(model "${KICAD8_3DMODEL_DIR}/Capacitor_SMD.3dshapes/C_0201_0603Metric.wrl"
+		(model "${KICAD8_3DMODEL_DIR}/Capacitor_SMD.3dshapes/C_0201_0603Metric.step"
 			(offset
 				(xyz 0 0 0)
@@
 			(pintype "passive")
 		)
-		(model "${KICAD8_3DMODEL_DIR}/Capacitor_SMD.3dshapes/C_0201_0603Metric.wrl"
+		(model "${KICAD8_3DMODEL_DIR}/Capacitor_SMD.3dshapes/C_0201_0603Metric.step"
 			(offset
 				(xyz 0 0 0)
@@
 			)
 		)
-		(property "MPN" "GRM033C81E104KE14D"
+		(property "MPN" "GRM033R60J105MEA2D"
 			(at 0 0 0)
 			(unlocked yes)
@@
 			)
 		)
-		(property "DISTPN" "490-10403-1-ND"
+		(property "DISTPN" "81-GRM033R60J105ME2D"
 			(at 0 0 0)
 			(unlocked yes)
@@
 			(pintype "passive")
 		)
-		(model "${KICAD8_3DMODEL_DIR}/Capacitor_SMD.3dshapes/C_0201_0603Metric.wrl"
+		(model "${KICAD8_3DMODEL_DIR}/Capacitor_SMD.3dshapes/C_0201_0603Metric.step"
 			(offset
 				(xyz 0 0 0)
@@
 			(pintype "passive")
 		)
-		(model "${KICAD6_3DMODEL_DIR}/Capacitor_SMD.3dshapes/C_0402_1005Metric.wrl"
-			(hide yes)
-			(offset
-				(xyz 0 0 0)
-			)
-			(scale
-				(xyz 1 1 1)
-			)
-			(rotate
-				(xyz 0 0 0)
-			)
-		)
-		(model ":PROJ3d:C_0402_1005Metric.step"
-			(offset
-				(xyz 0 0 0)
-			)
-			(scale
-				(xyz 1 1 1)
-			)
-			(rotate
-				(xyz 0 0 0)
-			)
-		)
 		(model "${KIPRJMOD}/packages3D/C_0402_1005Metric.step"
 			(offset
@@
 		(sheetname "Root")
 		(sheetfile "CompassTag.kicad_sch")
-		(attr smd exclude_from_bom)
+		(attr smd exclude_from_bom dnp)
 		(fp_line
 			(start 1.905 -1.27)
@@
 			(zone_connect 2)
 		)
-		(model "${KICAD8_3DMODEL_DIR}/Package_DFN_QFN.3dshapes/QFN-32-1EP_5x5mm_P0.5mm_EP3.45x3.45mm.wrl"
+		(model "${KICAD8_3DMODEL_DIR}/Package_DFN_QFN.3dshapes/QFN-32-1EP_5x5mm_P0.5mm_EP3.45x3.45mm.step"
 			(offset
 				(xyz 0 0 0)
@@
 			)
 		)
-		(property "MPN" "GRM033C81E104KE14D"
+		(property "MPN" "GRM033R60J105MEA2D"
 			(at 0 0 0)
 			(unlocked yes)
@@
 			)
 		)
-		(property "DISTPN" "490-10403-1-ND"
+		(property "DISTPN" "81-GRM033R60J105ME2D"
 			(at 0 0 0)
 			(unlocked yes)
@@
 			(pintype "passive")
 		)
-		(model "${KICAD8_3DMODEL_DIR}/Capacitor_SMD.3dshapes/C_0201_0603Metric.wrl"
+		(model "${KICAD8_3DMODEL_DIR}/Capacitor_SMD.3dshapes/C_0201_0603Metric.step"
 			(offset
 				(xyz 0 0 0)
@@
 			(pintype "passive")
 		)
-		(model "${KICAD8_3DMODEL_DIR}/Capacitor_SMD.3dshapes/C_0201_0603Metric.wrl"
+		(model "${KICAD8_3DMODEL_DIR}/Capacitor_SMD.3dshapes/C_0201_0603Metric.step"
 			(offset
 				(xyz 0 0 0)
@@
 			(pintype "passive")
 		)
-		(model "${KICAD6_3DMODEL_DIR}/Capacitor_SMD.3dshapes/C_0603_1608Metric.wrl"
+		(model "${KICAD6_3DMODEL_DIR}/Capacitor_SMD.3dshapes/C_0603_1608Metric.step"
 			(offset
 				(xyz 0 0 0)
@@
 		(layer "B.SilkS")
 	)
+	(gr_circle
+		(center 147.45 105.55)
+		(end 147.5 105.55)
+		(stroke
+			(width 0.15)
+			(type default)
+		)
+		(fill none)
+		(layer "F.SilkS")
+	)
+	(gr_line
+		(start 144.4 111)
+		(end 144.4 111.35)
+		(stroke
+			(width 0.15)
+			(type default)
+		)
+		(layer "F.SilkS")
+	)
+	(gr_line
+		(start 144.4 111.35)
+		(end 144.8 111.35)
+		(stroke
+			(width 0.15)
+			(type default)
+		)
+		(layer "F.SilkS")
+	)
 	(gr_line
 		(start 111.37 127.95)
@@
 		(layer "Edge.Cuts")
 	)
-	(gr_text "CpTag V1"
+	(gr_text "CTag V1"
 		(at 157.3 108.4 90)
 		(layer "B.SilkS")
