File: hardware/CompassTag/CompassTag.kicad_sch (KiCad schematic)
At the start: 28 parts, among them J201 CONN_02X04, J301 Conn_01x01, J302 Conn_01x01, J303 Conn_01x01, J304 Conn_01x01, J401 CONN_01X02, Q501 Q_NPN_BEC, U1 at25ex321D-UUN, U2 AK09940A, U3 LIS2DU12TR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

Commit message: checkpoint
Connections:
- net AK_MISO: now also U2.B4 (SO); no longer U2.A4 (SDA/SI)
- net AK_MOSI: now also U2.A4 (SDA/SI); no longer U2.B4 (SO)
Other:
- moved on the sheet: C2

Commit message: checkpoint
Connections:
- net AK_DRDY: now reaches U302.20 (PA10)
- net AK_DRDY: now also U2.A1 (DRDY/TRG)
- no-connect marks 9 -> 7
Changed lines of the file:
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@@
-	)
-	(no_connect
-		(at 31.115 119.38)
 	)
 	(no_connect
@@
 	(no_connect
 		(at 87.63 81.28)
-	)
-	(no_connect
-		(at 153.67 88.9)
 	)
 	(no_connect
@@
 		)
 	)
+	(label "AK_DRDY"
+		(at 153.67 88.9 0)
+		(effects
+			(font
+				(size 1.524 1.524)
+			)
+			(justify left bottom)
+		)
+	)
 	(label "AK_CK"
 		(at 115.57 119.38 270)
@@
 		(effects
 			(font
+				(size 1.524 1.524)
+			)
+			(justify right bottom)
+		)
+	)
+	(label "AK_DRDY"
+		(at 31.115 119.38 180)
+		(effects
+			(font

Commit message: tweek compass tag
Connections:
- net +2V5: now also C5.1, U2.C4 (VOD)
- net AK_PWR: no longer C5.1, U2.C4 (VOD)
Changed lines of the file:
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@@
 	)
 	(junction
-		(at 94.615 127)
+		(at 101.6 127)
 		(diameter 0)
 		(color 0 0 0 0)
@@
 	(wire
 		(pts
-			(xy 81.915 127) (xy 94.615 127)
-		)
-		(stroke
-			(width 0)
-			(type default)
-		)
-	)
-	(wire
-		(pts
 			(xy 227.33 33.02) (xy 227.33 41.91)
 		)
@@
 	(wire
 		(pts
-			(xy 94.615 127) (xy 101.6 127)
+			(xy 81.915 127) (xy 101.6 127)
 		)
 		(stroke
@@
 		)
 	)
-	(label "AK_PWR"
-		(at 97.155 127 0)
-		(effects
-			(font
-				(size 1.524 1.524)
-			)
-			(justify left bottom)
-		)
-	)
 	(label "AT25_SCK"
 		(at 128.27 53.34 90)
@@
 	)
 	(symbol
-		(lib_id "power:PWR_FLAG")
-		(at 94.615 127 0)
+		(lib_id "power:+2V5")
+		(at 101.6 127 0)
 		(unit 1)
 		(exclude_from_sim no)
@@
 		(on_board yes)
 		(dnp no)
-		(fields_autoplaced yes)
-		(property "Reference" "#FLG1"
-			(at 94.615 125.095 0)
+		(property "Reference" "#PWR11"
+			(at 101.6 130.81 0)
 			(effects
 				(font
@@
 			)
 		)
-		(property "Value" "PWR_FLAG"
-			(at 94.615 121.92 0)
+		(property "Value" "+2V5"
+			(at 101.981 122.6058 0)
 			(effects
 				(font
@@
 		)
 		(property "Footprint" ""
-			(at 94.615 127 0)
+			(at 101.6 127 0)
 			(effects
 				(font
@@
 			)
 		)
-		(property "Datasheet" "~"
-			(at 94.615 127 0)
+		(property "Datasheet" ""
+			(at 101.6 127 0)
 			(effects
 				(font
@@
 			)
 		)
-		(property "Description" "Special symbol for telling ERC where power comes from"
-			(at 94.615 127 0)
+		(property "Description" "Power symbol creates a global label with name \"+2V5\""
+			(at 101.6 127 0)
 			(effects
 				(font
@@
 		)
 		(instances
-			(project ""
+			(project "CompassTag"
 				(path "/e44ca67a-43be-444b-8652-f54825a2eb6f"
-					(reference "#FLG1")
+					(reference "#PWR11")
 					(unit 1)
 				)

Commit message: update compasstag hardware
Parts:
- C1, C3, C501, C502, C503: DISTPN 490-10403-1-ND -> 81-GRM033R60J105ME2D; MPN C181047 -> GRM033R60J105MEA2D
- C2: DISTPN 490-7229-2-ND -> 81-GRM033R60J105ME2D; MFN murata -> Murata
- C5, C9: DISTPN 490-10403-1-ND -> 81-GRM033R60J105ME2D; MPN GRM033C81E104KE14D -> GRM033R60J105MEA2D
- J201, J301, J302, J303, J304, J401: now not fitted
- U3: DISTPN (none) -> 497-LIS2DU12TRCT-ND; MFN (none) -> STMicroelectroincs; MPN (none) -> LIS2DU12TR

Commit message: update parts
Parts:
- C1, C3, C501, C502, C503: DISTPN 81-GRM033R60J105ME2D -> 490-7229-1-ND
- C2: DISTPN 81-GRM033R60J105ME2D -> 490-7229-1-ND; LCSC C76929 -> C181047
- C5, C9: DISTPN 81-GRM033R60J105ME2D -> 490-7229-1-ND; LCSC (none) -> C181047
- U1: DISTPN 724-AT25FF321A-UUN-T -> 1265-AT25XE321D-UUN-TCT-ND; MPN AT25FF321A-UUN-T -> AT25XE321D-UUN-T
- U2: footprint AccelTag:AK09940a -> LGA11_1p6x1p6x0p58_AKM
Other:
- moved on the sheet: C5, C7, C8, C9, U2, U4

Commit message: update flash for imu tag
Parts:
- C7, C8: DISTPN 490-7229-1-ND -> 490-16305-1-ND; MPN GRM033R60J105MEA2D -> GRT033R60J105ME13D
Changed lines of the file:
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@@
 	(label "USART2_CK"
 		(at 113.03 119.38 270)
-		(fields_autoplaced yes)
 		(effects
 			(font
@@
 	(label "SDA"
 		(at 120.65 53.34 90)
-		(fields_autoplaced yes)
 		(effects
 			(font
@@
 	(label "SDA"
 		(at 213.36 130.81 180)
-		(fields_autoplaced yes)
 		(effects
 			(font
@@
 	(label "AT25_SCK"
 		(at 72.39 38.1 0)
-		(fields_autoplaced yes)
 		(effects
 			(font
@@
 	(label "AK_RSTN"
 		(at 123.19 119.38 270)
-		(fields_autoplaced yes)
 		(effects
 			(font
@@
 	(label "AK_PWR"
 		(at 232.41 83.82 180)
-		(fields_autoplaced yes)
 		(effects
 			(font
@@
 	(label "clkout"
 		(at 213.36 123.19 180)
-		(fields_autoplaced yes)
 		(effects
 			(font
@@
 	(label "WKUP1"
 		(at 87.63 88.9 180)
-		(fields_autoplaced yes)
 		(effects
 			(font
@@
 	(label "AK_PWR"
 		(at 153.67 91.44 0)
-		(fields_autoplaced yes)
 		(effects
 			(font
@@
 	(label "AK_MISO"
 		(at 118.11 119.38 270)
-		(fields_autoplaced yes)
 		(effects
 			(font
@@
 	(label "USART2_RX"
 		(at 58.42 160.02 180)
-		(fields_autoplaced yes)
 		(effects
 			(font
@@
 	(label "AK_CS"
 		(at 31.75 121.92 180)
-		(fields_autoplaced yes)
 		(effects
 			(font
@@
 	(label "clkout"
 		(at 80.01 78.74 180)
-		(fields_autoplaced yes)
 		(effects
 			(font
@@
 	(label "ACCEL_CS"
 		(at 87.63 91.44 180)
-		(fields_autoplaced yes)
 		(effects
 			(font
@@
 	(label "WKUP1"
 		(at 119.38 154.94 0)
-		(fields_autoplaced yes)
 		(effects
 			(font
@@
 	(label "WKUP1"
 		(at 58.42 165.1 180)
-		(fields_autoplaced yes)
 		(effects
 			(font
@@
 	(label "AT25_MOSI"
 		(at 123.19 53.34 90)
-		(fields_autoplaced yes)
 		(effects
 			(font
@@
 	(label "AT25_nCS"
 		(at 35.56 30.48 180)
-		(fields_autoplaced yes)
 		(effects
 			(font
@@
 	(label "AT25_MOSI"
 		(at 72.39 41.91 0)
-		(fields_autoplaced yes)
 		(effects
 			(font
@@
 	(label "AT25_nCS"
 		(at 130.81 53.34 90)
-		(fields_autoplaced yes)
 		(effects
 			(font
@@
 	(label "USART2_CK"
 		(at 58.42 154.94 180)
-		(fields_autoplaced yes)
 		(effects
 			(font
@@
 	(label "USART2_TX"
 		(at 83.82 93.98 180)
-		(fields_autoplaced yes)
 		(effects
 			(font
@@
 	(label "AK_DRDY"
 		(at 153.67 88.9 0)
-		(fields_autoplaced yes)
 		(effects
 			(font
@@
 	(label "AK_CK"
 		(at 115.57 119.38 270)
-		(fields_autoplaced yes)
 		(effects
 			(font
@@
 	(label "AK_CS"
 		(at 125.73 119.38 270)
-		(fields_autoplaced yes)
 		(effects
 			(font
@@
 	(label "AT25_MISO"
 		(at 125.73 53.34 90)
-		(fields_autoplaced yes)
 		(effects
 			(font
@@
 	(label "AK_CK"
 		(at 31.75 124.46 180)
-		(fields_autoplaced yes)
 		(effects
 			(font
@@
 	(label "ACCEL_CS"
 		(at 58.42 157.48 180)
-		(fields_autoplaced yes)
 		(effects
 			(font
@@
 	(label "SCL"
 		(at 118.11 53.34 90)
-		(fields_autoplaced yes)
 		(effects
 			(font
@@
 	(label "AT25_SCK"
 		(at 128.27 53.34 90)
-		(fields_autoplaced yes)
 		(effects
 			(font
@@
 	(label "AT25_MISO"
 		(at 44.45 34.29 180)
-		(fields_autoplaced yes)
 		(effects
 			(font
@@
 	(label "AK_RSTN"
 		(at 82.55 119.38 0)
-		(fields_autoplaced yes)
 		(effects
 			(font
@@
 	(label "AK_MOSI"
 		(at 31.75 127 180)
-		(fields_autoplaced yes)
 		(effects
 			(font
@@
 	(label "SCL"
 		(at 213.36 128.27 180)
-		(fields_autoplaced yes)
 		(effects
 			(font
@@
 	(label "USART2_RX"
 		(at 110.49 119.38 270)
-		(fields_autoplaced yes)
 		(effects
 			(font
@@
 	(label "AK_MOSI"
 		(at 120.65 119.38 270)
-		(fields_autoplaced yes)
 		(effects
 			(font
@@
 	(label "AK_DRDY"
 		(at 31.75 119.38 180)
-		(fields_autoplaced yes)
 		(effects
 			(font
@@
 	(label "AK_MISO"
 		(at 87.63 132.08 0)
-		(fields_autoplaced yes)
 		(effects
 			(font
@@
 	(label "USART2_TX"
 		(at 58.42 162.56 180)
-		(fields_autoplaced yes)
 		(effects
 			(font
@@
 			)
 		)
-		(property "MPN" "GRM033R60J105MEA2D"
+		(property "MPN" "GRT033R60J105ME13D"
 			(at 251.46 86.36 0)
 			(effects
@@
 			)
 		)
-		(property "DISTPN" "490-7229-1-ND"
+		(property "DISTPN" "490-16305-1-ND"
 			(at 182.88 184.15 0)
 			(effects
@@
 			)
 		)
-		(property "MPN" "GRM033R60J105MEA2D"
+		(property "MPN" "GRT033R60J105ME13D"
 			(at 218.44 86.36 0)
 			(effects
@@
 			)
 		)
-		(property "DISTPN" "490-7229-1-ND"
+		(property "DISTPN" "490-16305-1-ND"
 			(at 149.86 184.15 0)
 			(effects

Commit message: checkpoint
Other:
- title: BitTag with External Memory and LI2DW12 -> compass tag
Changed lines of the file:
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@@
 (kicad_sch
-	(version 20231120)
+	(version 20250114)
 	(generator "eeschema")
-	(generator_version "8.0")
+	(generator_version "9.0")
 	(paper "USLetter")
 	(title_block
-		(title "BitTag with External Memory and LI2DW12")
-		(date "2025-02-19")
+		(title "compass tag")
+		(date "2026-04-16")
 		(company "IUCS")
 		(comment 1 "Geoffrey Brown")
 	)
+	(text "Note: PA15 and PB4 pulled up on reset !"
+		(exclude_from_sim no)
+		(at 96.52 34.29 0)
+		(effects
+			(font
+				(size 1.524 1.524)
+			)
+			(justify left bottom)
+		)
+	)
+	(text "Tag Holes"
+		(exclude_from_sim no)
+		(at 24.13 194.31 0)
+		(effects
+			(font
+				(size 1.524 1.524)
+			)
+			(justify left bottom)
+		)
+	)
+	(text "Test Points"
+		(exclude_from_sim no)
+		(at 172.72 36.83 0)
+		(effects
+			(font
+				(size 1.524 1.524)
+			)
+			(justify left bottom)
+		)
+	)
+	(text "Battery"
+		(exclude_from_sim no)
+		(at 213.36 49.53 0)
+		(effects
+			(font
+				(size 1.524 1.524)
+			)
+			(justify left bottom)
+		)
+	)
 	(junction
 		(at 138.43 184.15)
@@
 		)
 	)
-	(text "Note: PA15 and PB4 pulled up on reset !"
-		(exclude_from_sim no)
-		(at 96.52 34.29 0)
-		(effects
-			(font
-				(size 1.524 1.524)
-			)
-			(justify left bottom)
-		)
-	)
-	(text "Tag Holes"
-		(exclude_from_sim no)
-		(at 24.13 194.31 0)
-		(effects
-			(font
-				(size 1.524 1.524)
-			)
-			(justify left bottom)
-		)
-	)
-	(text "Test Points"
-		(exclude_from_sim no)
-		(at 172.72 36.83 0)
-		(effects
-			(font
-				(size 1.524 1.524)
-			)
-			(justify left bottom)
-		)
-	)
-	(text "Battery"
-		(exclude_from_sim no)
-		(at 213.36 49.53 0)
-		(effects
-			(font
-				(size 1.524 1.524)
-			)
-			(justify left bottom)
-		)
-	)
 	(label "USART2_CK"
 		(at 113.03 119.38 270)
@@
 		)
 	)
+	(embedded_fonts no)
 )
