File: hardware/nucleoshield-c071-base-test/nucleoshield-c071-base-test.kicad_pcb (KiCad board)
At the start: 2 copper layers, 50 x 53.4 mm, 13 parts, among them J1 Power, J2 Digital/PWM, J3 Analog, J4 Digital/PWM, J5 Conn_02x03_Odd_Even

Commit message: added nucleoshield template
Connections:
- J1 pad 5: +5V -> unconnected-(J1-Pin_5-Pad5)
- J1 pad 8: VCC -> unconnected-(J1-Pin_8-Pad8)
