File: hardware/tagbase-lipo-v1/tagbase-lipo-v1.kicad_sch (KiCad schematic)
At the start: 40 parts, among them J1 Conn_01x04_Female, J101 Conn_02x03_Odd_Even, J102 Conn_02x05_Odd_Even, J104 USB_B_Mini, J2 Conn_01x06, J5 Conn_01x02, SW1 SW_DIP_x04, U1 XC6206, U105 Tactile Switch, U2 TS5A3159ADBVR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

Commit message: checkpoint
Parts:
- removed D1, D3: DIODE, Diode_SMD:D_SOD-123, symbol Device:D_Schottky
- removed R106, R6: 100, Resistor_SMD:R_0603_1608Metric, symbol Device:R
- removed R108: 620, Resistor_SMD:R_0603_1608Metric, symbol Device:R
- removed R5: 33, Resistor_SMD:R_0603_1608Metric, symbol Device:R
- removed SW1: SW_DIP_x04, Button_Switch_SMD:SW_DIP_SPSTx06_Slide_KingTek_DSHP06TS_W7.62mm_P1.27mm, symbol Switch:SW_DIP_x06
- removed U2, U3, U4, U5: TS5A3159ADBVR, Package_TO_SOT_SMD:SOT-23-6, symbol Analog_Switch:TS5A3159ADBVR
- removed U6: STM32F042G6Ux, Package_DFN_QFN:QFN-28_4x4mm_P0.5mm, symbol MCU_ST_STM32F0:STM32F042G6Ux
- added C4, C5: 1uF, Capacitor_SMD:C_0603_1608Metric, symbol Device:C
- added D1: D_Schottky_Small, Diode_SMD:D_SOD-323, symbol Device:D_Schottky_Small
- added R1: 30K, Resistor_SMD:R_0603_1608Metric, symbol Device:R
- added SW1, SW2: SW_SPDT, tagbase:CJS-1200B_NDC, symbol Switch:SW_SPDT
- added U2: XC6808ANC28R-G, tagbase:xc6808, symbol xc6808:XC6808ANC28R-G
- added U3: XC6206P182MR, Package_TO_SOT_SMD:SOT-23-3, symbol Regulator_Linear:XC6206PxxxMR
- added U4: STM32C071GBU6N, UFQFPN-28_STM, symbol STM32C071GBU6N:STM32C071GBU6N
- D101: footprint LED_SMD:LED_0603_1608Metric -> Diode_SMD:D_0805_2012Metric; LCSC C2286 -> C84256; MFN Hubei KENTO Elec -> Foshan NationStar Optoelectronics; MPN KT-0603R -> NCD0805R1
- D102, D105: footprint LED_SMD:LED_0603_1608Metric -> Diode_SMD:D_0805_2012Metric; LCSC C72043 -> C2297; MFN Everlight Elec -> Hubei KENTO Elec; MPN 19-217/GHC-YR1S2/3T -> KT-0805G
- H1, H2, H3, H4, J1, J102, J2, J5: now not fitted
- J101: footprint tagbase:6pin_tagpoints_new_offset -> tagbase:6pin_tagpoints_double_screws; now not fitted
- R101, R102, R107: value 620 -> 680; LCSC C23220 -> C23228; MPN 0603WAF6200T5E -> 0603WAF6800T5E
- R2: value 1.5K -> 10K; LCSC C22843 -> C25804; MFN Uniroyal Elec -> Uniroyal Elec.; MPN 0603WAF1501T5E -> 0603WAF1002T5E
- R3: value 2K -> 10K; LCSC C22975 -> C25804; MFN Uniroyal Elec -> Uniroyal Elec.; MPN 0603WAF2001T5E -> 0603WAF1002T5E
- U1: value XC6206 -> XC6206P332MR
Connections:
- net VIN is gone; now on net VUSB: C1.1, U1.3 (VI)
- net +3V3: now also SW1.3 (C), U4.17 (VDDIO2); no longer C2.1
- net GND: now also R2.2, C4.2, C5.2, R1.2, U2.2 (VSS), U2.7 (EPAD), U3.1 (GND), U4.4 (VSS/VSSA)
- net NRST: now also U4.5 (PF2-NRST)
- net SWDIO: now also U4.20 (PA13)
- net TAG_3V3: now also D1.1 (K)
- net TAG_3V3_IN: now also SW1.1 (A)
- net TAG_VBAT: now also SW2.2 (B)
- net USB_DM: now also U4.18 (PA11[PA9])
- net USB_DP: now also U4.19 (PA12[PA10])
- net VUSB: now also C4.1, U2.6 (VIN), U3.3 (VI)
- net boot0: now also U4.21 (PA14-BOOT0)
- net at R2.1: now also U2.5 (THIN/NF); no longer R3.1
- net CSO: now reaches R3.2
- net CSO: now also U2.3 (CSO)
- new net: D1.2 (A), SW1.2 (B)
- new net: R1.1, U2.4 (ISET)
- new net +1V8: C2.1, C5.1, R3.1, U3.2 (VO), U4.3 (VDD/VDDA)
- new net BAT: SW2.1 (A), U2.1 (BAT)
- no-connect marks 11 -> 4
Other:
- note added: "Rset = 351K * Icharge(mA)^-1.1 e.g Rset(10mA) = 351/(12.6) = 27.9K Rset(9.35mA) = 30K"
- note added: "VDDIO2 3.3V"
- note added: "boot0 = swclk"
- moved on the sheet: C101, C107, C2, C3, D101, D102, D105, R101, R102, R104, R105, R107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

Commit message: checkpoint
Parts:
- removed R105: 10K, Resistor_SMD:R_0603_1608Metric, symbol Device:R
- added C6, C7: 4.7uf, Capacitor_SMD:C_0402_1005Metric, symbol Device:C
- C1, C104, C4, C5: footprint Capacitor_SMD:C_0603_1608Metric -> Capacitor_SMD:C_0402_1005Metric; LCSC C15849 -> C52923; MPN CL10A105KB8NNNC -> CL05A105KA5NQNC
- C101, C107, C2, C3: footprint Capacitor_SMD:C_0603_1608Metric -> Capacitor_SMD:C_0402_1005Metric; LCSC C14663 -> C1525; MFN YAGEO -> Samsung Electro-Mechanics; MPN CC0603KRX7R9BB104 -> CL05B104KO5NNNC
- R1: value 30K -> 33K; footprint Resistor_SMD:R_0603_1608Metric -> Resistor_SMD:R_0402_1005Metric; LCSC C22984 -> C25779; MPN 0603WAF3002T5E -> 0402WGF3302TCE
- R101: value 680 -> 220; LCSC C23228 -> C22775; MPN 0603WAF6800T5E -> 0603WAF1000T5E
- R102: value 680 -> 100; LCSC C23228 -> C22775; MPN 0603WAF6800T5E -> 0603WAF1000T5E
- R104: footprint Resistor_SMD:R_0603_1608Metric -> Resistor_SMD:R_0402_1005Metric; LCSC C4190 -> C25879; MPN 0603WAF1002T5E -> 0402WGF2201TCE
- R107: value 680 -> 300; LCSC C23228 -> C23025; MPN 0603WAF6800T5E -> 0603WAF3000T5E
- R2, R3: footprint Resistor_SMD:R_0603_1608Metric -> Resistor_SMD:R_0402_1005Metric; LCSC C25804 -> C25744; MPN 0603WAF1002T5E -> 0402WGF1002TCE
- U3: value XC6206P182MR -> XC6206P202MR; LCSC C21659 -> C2891260; MPN XC6206P182MR -> XC6206P202MR-G
Connections:
- net +3V3: now also R3.1, C7.1
- net GND: now also C6.2, C7.2
- net LED_GREEN: now also U4.16 (PA8)
- net LED_RED: now also U4.22 (PA15)
- net SCLK: no longer J102.4 (Pin_4)
- net +1V8 renamed +2V
- net +2V: now also C6.1; no longer R3.1
- net boot0 renamed SWCLK
- net SWCLK: now also J102.4 (Pin_4)
- no-connect marks 4 -> 6
Other:
- note added: "DFU - pullup, weak pulldown on pin"
- note added: "No need for pulldown on PA14 -- weak internal pull-down activated on reset"
- note added: "Red 2Vf, 6mA, 216 ohm (3.3v) Green 2.7Vf, 6mA, 100 ohm (3.3V) Green 2.7Vf, 6mA, 300 ohm (4.5V)"
- note added: "Rset = 351K * Icharge(mA)^-1.1 e.g Rset(10mA) = 351/(12.6) = 27.9K Rset(9.35mA) = 30K Rset(8.58mA) = 33K"
- note removed: "Rset = 351K * Icharge(mA)^-1.1 e.g Rset(10mA) = 351/(12.6) = 27.9K Rset(9.35mA) = 30K"
- note removed: "VDDIO2 3.3V"
- note removed: "boot0 = swclk"
- moved on the sheet: C101, C2

Commit message: restructure data logging
Parts:
- removed C3: 0.1uF, Capacitor_SMD:C_0402_1005Metric, symbol Device:C
- removed R107: 300, Resistor_SMD:R_0603_1608Metric, symbol Device:R
- added R4: 1K, Resistor_SMD:R_0402_1005Metric, symbol Device:R
- added R5: 100, Resistor_SMD:R_0603_1608Metric, symbol Device:R
- U2: footprint tagbase:xc6808 -> USP-6B_TOR
- U4: LCSC (none) -> C42240018; MFN (none) -> STMicroelectronics; MPN (none) -> STM32C071GBU6N
Connections:
- net +2V: now also R3.1
- net +3V3: now also D105.2 (A); no longer R3.1
- net CSO: now also U4.11 (PA5), U4.12 (PA6)
- net GND: now also R5.2
- net TAG_SCK: now also U4.6 (PA0), U4.7 (PA1)
- net TAG_SWDIO: now also U4.10 (PA4), R4.2
- net UART_TX: now also U4.26 (PB6)
- net VUSB: no longer D105.2 (A)
- net at R104.2: now also U4.27 (PB7)
- net at D105.1 (K): now also R5.1
- net at U4.8 (PA2): now also R4.1
- net EXT_PWR: no longer names the net of J1.3 (Pin_3)
- net TAG_MIRROR: no longer names the net of J1.1 (Pin_1)
- no-connect marks 6 -> 16
Other:
- moved on the sheet: C107, C7, D105, R1, R104, R2, R3, U2
