File: hardware/tag-breakout-template/tag-breakout-template.kicad_pcb (KiCad board)
At the start: 2 copper layers, 48.3 x 48.3 mm, 17 parts, among them J3 Conn_01x17, J4 Conn_01x17, U1 TPS7A2018PDQN, U2 MX25L12835G, U3 AK09940A, U4 LSM6DSV, U5 LPS22DF

Commit message: checkpoint
Parts:
- C1, C10, C2, C3, C4, C5, C6, C7, C8, C9: footprint Capacitor_SMD:C_0201_0603Metric -> Capacitor_SMD:C_0603_1608Metric
- U4: value LSM6DSV -> LSM6DSV16XTR; footprint taglibrary:LGA14-L_2P59X3P1X0P5_STM -> Package_LGA:LGA-14_3x2.5mm_P0.5mm_LayoutBorder3x4y
- U5: value LPS22DF -> LPS22HH
- moved C2 3.90 mm to (124.9, 88.0), turned to 90 degrees
- moved C3 2.79 mm to (132.9, 92.0), turned to 90 degrees
- moved C5 1.42 mm to (133.7, 98.0)
- moved C6 1.09 mm to (126.0, 96.0), turned to 180 degrees
- moved C9 1.05 mm to (128.2, 103.5), turned to -90 degrees
- moved C1 1.00 mm to (130.0, 103.5), turned to -90 degrees
- moved C4 0.84 mm to (133.7, 96.5)
- moved C7 0.68 mm to (126.6, 88.0)
- moved C10 0.63 mm to (122.7, 81.8)
- moved C8 0.31 mm to (131.0, 96.3)
Routing:
- net +3.3V: track 115.3 -> 124.1 mm
- net GND: track 18.9 -> 27.6 mm, vias 10 -> 12
- net +1V8: track 5.12 -> 7.20 mm
- net /LSM_CS: track 37.3 -> 38.9 mm
Other:
- board text added: "LPS22HH because LPS22DV not available"
