File: hardware/tag-breakout-template/tag-breakout-template.kicad_sch (KiCad schematic)
At the start: 17 parts, among them J3 Conn_01x17, J4 Conn_01x17, U1 TPS7A2018PDQN, U2 MX25L12835G, U3 AK09940A, U4 LSM6DSV, U5 LPS22DF

Commit message: checkpoint
Parts:
- C1, C10, C2, C7, C8, C9: footprint Capacitor_SMD:C_0201_0603Metric -> Capacitor_SMD:C_0603_1608Metric; LCSC C181047 -> C14663; MFN Murata -> YAGEO; MPN C181047 -> CC0603KRX7R9BB104
- C3, C4: footprint Capacitor_SMD:C_0201_0603Metric -> Capacitor_SMD:C_0603_1608Metric; LCSC C76930 -> C15849; MFN Murata -> Samsung Electro-Mechanics; MPN GRM033R60J105MEA2D -> CL10A105KB8NNNC
- C5, C6: footprint Capacitor_SMD:C_0201_0603Metric -> Capacitor_SMD:C_0603_1608Metric; LCSC C181047 -> C14663; MFN Murata -> YAGEO; MPN GRM033C81E104KE14D -> CC0603KRX7R9BB104
- J3, J4: now left out of the parts list
- U4: value LSM6DSV -> LSM6DSV16XTR; footprint LGA14-L_2P59X3P1X0P5_STM -> Package_LGA:LGA-14_3x2.5mm_P0.5mm_LayoutBorder3x4y; LCSC C41785564 -> C5267406
- U5: value LPS22DF -> LPS22HH; LCSC C3253714 -> C2827824; MPN LPS22DF -> LPS22HH
Other:
- note added: "Should be lps22df but jlcpcb only has lps22hh which is an inferior part with different registers"
Changed lines of the file:
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@@
 		)
 	)
+	(text "Should be lps22df but jlcpcb only has lps22hh which \nis an inferior part with different registers"
+		(exclude_from_sim no)
+		(at 79.502 198.12 0)
+		(effects
+			(font
+				(size 1.27 1.27)
+			)
+		)
+	)
 	(text "PA3"
 		(exclude_from_sim no)
@@
 		(unit 1)
 		(exclude_from_sim no)
-		(in_bom yes)
+		(in_bom no)
 		(on_board yes)
 		(dnp yes)
@@
 		(unit 1)
 		(exclude_from_sim no)
-		(in_bom yes)
+		(in_bom no)
 		(on_board yes)
 		(dnp yes)
@@
 			)
 		)
-		(property "Footprint" "Capacitor_SMD:C_0201_0603Metric"
+		(property "Footprint" "Capacitor_SMD:C_0603_1608Metric"
 			(at 123.4948 143.51 0)
 			(effects
@@
 			)
 		)
-		(property "MFN" "Murata"
+		(property "MFN" "YAGEO"
 			(at 124.46 139.7 0)
 			(effects
@@
 			)
 		)
-		(property "MPN" "C181047"
+		(property "MPN" "CC0603KRX7R9BB104"
 			(at 302.26 242.57 0)
 			(effects
@@
 			)
 		)
-		(property "LCSC" "C181047"
+		(property "LCSC" "C14663"
 			(at 124.46 139.7 0)
 			(effects
@@
 			)
 		)
-		(property "Footprint" "Capacitor_SMD:C_0201_0603Metric"
+		(property "Footprint" "Capacitor_SMD:C_0603_1608Metric"
 			(at 220.0148 85.09 0)
 			(effects
@@
 			)
 		)
-		(property "MFN" "Murata"
+		(property "MFN" "YAGEO"
 			(at 220.98 81.28 0)
 			(effects
@@
 			)
 		)
-		(property "MPN" "C181047"
+		(property "MPN" "CC0603KRX7R9BB104"
 			(at 398.78 184.15 0)
 			(effects
@@
 			)
 		)
-		(property "LCSC" "C181047"
+		(property "LCSC" "C14663"
 			(at 220.98 81.28 0)
 			(effects
@@
 			)
 		)
-		(property "Footprint" "Capacitor_SMD:C_0201_0603Metric"
+		(property "Footprint" "Capacitor_SMD:C_0603_1608Metric"
 			(at 254.9652 33.02 0)
 			(effects
@@
 			)
 		)
-		(property "MFN" "Murata"
+		(property "MFN" "YAGEO"
 			(at 254 29.21 0)
 			(effects
@@
 			)
 		)
-		(property "MPN" "GRM033C81E104KE14D"
+		(property "MPN" "CC0603KRX7R9BB104"
 			(at 254 29.21 0)
 			(effects
@@
 			)
 		)
-		(property "LCSC" "C181047"
+		(property "LCSC" "C14663"
 			(at 254 29.21 0)
 			(effects
@@
 			)
 		)
-		(property "Value" "LSM6DSV"
+		(property "Value" "LSM6DSV16XTR"
 			(at 81.28 110.49 0)
 			(effects
@@
 			)
 		)
-		(property "Footprint" "LGA14-L_2P59X3P1X0P5_STM"
+		(property "Footprint" "Package_LGA:LGA-14_3x2.5mm_P0.5mm_LayoutBorder3x4y"
 			(at 55.88 118.11 0)
 			(effects
@@
 			)
 		)
-		(property "LCSC" "C41785564"
+		(property "LCSC" "C5267406"
 			(at 55.88 118.11 0)
 			(effects
@@
 			)
 		)
-		(property "Value" "LPS22DF"
+		(property "Value" "LPS22HH"
 			(at 69.85 176.5299 0)
 			(effects
@@
 			)
 		)
-		(property "LCSC" "C3253714"
+		(property "LCSC" "C2827824"
 			(at 81.28 176.53 0)
 			(effects
@@
 			)
 		)
-		(property "MPN" "LPS22DF"
+		(property "MPN" "LPS22HH"
 			(at 81.28 176.53 0)
 			(effects
@@
 			)
 		)
-		(property "Footprint" "Capacitor_SMD:C_0201_0603Metric"
+		(property "Footprint" "Capacitor_SMD:C_0603_1608Metric"
 			(at 246.0752 133.35 0)
 			(effects
@@
 			)
 		)
-		(property "MFN" "Murata"
+		(property "MFN" "YAGEO"
 			(at 245.11 129.54 0)
 			(effects
@@
 			)
 		)
-		(property "MPN" "GRM033C81E104KE14D"
+		(property "MPN" "CC0603KRX7R9BB104"
 			(at 245.11 129.54 0)
 			(effects
@@
 			)
 		)
-		(property "LCSC" "C181047"
+		(property "LCSC" "C14663"
 			(at 245.11 129.54 0)
 			(effects
@@
 			)
 		)
-		(property "Footprint" "Capacitor_SMD:C_0201_0603Metric"
+		(property "Footprint" "Capacitor_SMD:C_0603_1608Metric"
 			(at 157.7848 137.16 0)
 			(effects
@@
 			)
 		)
-		(property "MFN" "Murata"
+		(property "MFN" "YAGEO"
 			(at 158.75 133.35 0)
 			(effects
@@
 			)
 		)
-		(property "MPN" "C181047"
+		(property "MPN" "CC0603KRX7R9BB104"
 			(at 336.55 236.22 0)
 			(effects
@@
 			)
 		)
-		(property "LCSC" "C181047"
+		(property "LCSC" "C14663"
 			(at 158.75 133.35 0)
 			(effects
@@
 			)
 		)
-		(property "Footprint" "Capacitor_SMD:C_0201_0603Metric"
+		(property "Footprint" "Capacitor_SMD:C_0603_1608Metric"
 			(at 40.9448 180.34 0)
 			(effects
@@
 			)
 		)
-		(property "MFN" "Murata"
+		(property "MFN" "YAGEO"
 			(at 41.91 176.53 0)
 			(effects
@@
 			)
 		)
-		(property "MPN" "C181047"
+		(property "MPN" "CC0603KRX7R9BB104"
 			(at 219.71 279.4 0)
 			(effects
@@
 			)
 		)
-		(property "LCSC" "C181047"
+		(property "LCSC" "C14663"
 			(at 41.91 176.53 0)
 			(effects
@@
 			)
 		)
-		(property "Footprint" "Capacitor_SMD:C_0201_0603Metric"
+		(property "Footprint" "Capacitor_SMD:C_0603_1608Metric"
 			(at 28.2448 137.16 0)
 			(effects
@@
 			)
 		)
-		(property "MFN" "Murata"
+		(property "MFN" "YAGEO"
 			(at 29.21 133.35 0)
 			(effects
@@
 			)
 		)
-		(property "MPN" "C181047"
+		(property "MPN" "CC0603KRX7R9BB104"
 			(at 207.01 236.22 0)
 			(effects
@@
 			)
 		)
-		(property "LCSC" "C181047"
+		(property "LCSC" "C14663"
 			(at 29.21 133.35 0)
 			(effects
@@
 			)
 		)
-		(property "Footprint" "Capacitor_SMD:C_0201_0603Metric"
+		(property "Footprint" "Capacitor_SMD:C_0603_1608Metric"
 			(at 215.5952 33.02 0)
 			(effects
@@
 			)
 		)
-		(property "MFN" "Murata"
+		(property "MFN" "Samsung Electro-Mechanics"
 			(at 214.63 29.21 0)
 			(effects
@@
 			)
 		)
-		(property "MPN" "GRM033R60J105MEA2D"
+		(property "MPN" "CL10A105KB8NNNC"
 			(at 214.63 29.21 0)
 			(effects
@@
 			)
 		)
-		(property "LCSC" "C76930"
+		(property "LCSC" "C15849"
 			(at 214.63 29.21 0)
 			(effects
@@
 			)
 		)
-		(property "Footprint" "Capacitor_SMD:C_0201_0603Metric"
+		(property "Footprint" "Capacitor_SMD:C_0603_1608Metric"
 			(at 53.6448 180.34 0)
 			(effects
@@
 			)
 		)
-		(property "MFN" "Murata"
+		(property "MFN" "YAGEO"
 			(at 54.61 176.53 0)
 			(effects
@@
 			)
 		)
-		(property "MPN" "C181047"
+		(property "MPN" "CC0603KRX7R9BB104"
 			(at 232.41 279.4 0)
 			(effects
@@
 			)
 		)
-		(property "LCSC" "C181047"
+		(property "LCSC" "C14663"
 			(at 54.61 176.53 0)
 			(effects
@@
 			)
 		)
-		(property "Footprint" "Capacitor_SMD:C_0201_0603Metric"
+		(property "Footprint" "Capacitor_SMD:C_0603_1608Metric"
 			(at 248.6152 33.02 0)
 			(effects
@@
 			)
 		)
-		(property "MFN" "Murata"
+		(property "MFN" "Samsung Electro-Mechanics"
 			(at 247.65 29.21 0)
 			(effects
@@
 			)
 		)
-		(property "MPN" "GRM033R60J105MEA2D"
+		(property "MPN" "CL10A105KB8NNNC"
 			(at 247.65 29.21 0)
 			(effects
@@
 			)
 		)
-		(property "LCSC" "C76930"
+		(property "LCSC" "C15849"
 			(at 247.65 29.21 0)
 			(effects

Commit message: checkpoint
Other:
- note removed: "Check capacitor requirements for LSM"
- note removed: "Need capacitors for Flash"
Changed lines of the file:
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@@
-		)
-	)
-	(text "Need capacitors for\nFlash"
-		(exclude_from_sim no)
-		(at 200.406 97.536 0)
-		(effects
-			(font
-				(size 1.27 1.27)
-			)
 		)
 	)
@@
 		(effects
 			(font
-				(size 1.27 1.27)
-			)
-		)
-	)
-	(text "Check capacitor requirements for LSM"
-		(exclude_from_sim no)
-		(at 83.312 144.272 0)
-		(effects
-			(font
