File: hardware/imutag/imutag.kicad_pcb (KiCad board)
At the start: 2 copper layers, 18 x 9 mm, 26 parts, among them J201 CONN_02X04, J301 Conn_01x01, J302 Conn_01x01, J303 Conn_01x01, J304 Conn_01x01, J401 CONN_01X02, Q501 Q_NPN_BEC, U2 AK09940A, U3 LPS22DF, U302 stm32l431kc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

Commit message: checkpoint
Parts:
- added C4: 4.7uf, Capacitor_SMD:C_0201_0603Metric, F.Cu at (151.1, 110.9)
- moved C501 0.66 mm to (151.1, 110.9)
- turned U3 to 90 degrees
Connections:
- U302 pad 31: GND -> Net-(U302-BOOT0)
Routing:
- net GND: track 60.5 -> 54.5 mm
- net Net-(U302-BOOT0): track 0.00 -> 1.70 mm, vias 0 -> 1
- net /SDA: track 3.94 -> 2.30 mm
- net /LPS_MOSI: track 5.69 -> 4.55 mm
- net +1V8: track 53.1 -> 52.4 mm
- net /SCL: track 4.20 -> 3.49 mm
- net RST: track 11.0 -> 10.3 mm
- net /LSM_CK: track 6.03 -> 6.55 mm
