File: hardware/IMUTagBreakout/IMUTagBreakout.kicad_pcb (KiCad board)
At the start: 2 copper layers, 48.3 x 48.3 mm, 21 parts, among them J3 Conn_01x17, J4 Conn_01x17, U1 TPS7A0218PDQNR, U2 MX25L12835G, U3 AK09940A, U4 LSM6DSV16XTR, U5 LPS22HH

Commit message: checkpoint
Other:
- board text added: "LPS_RDY PA9"
- board text added: "PA5 LMS_CK"
- board text removed: "LMS_RDY PA9"
- board text removed: "PA5 LPS_CK"
Changed lines of the file:
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@@
 		)
 	)
-	(gr_text "LMS_RDY PA9"
+	(gr_text "LPS_RDY PA9"
 		(at 147.32 91.44 0)
 		(layer "F.SilkS")
@@
 		)
 	)
-	(gr_text "PA5 LPS_CK"
+	(gr_text "PA5 LMS_CK"
 		(at 109.22 106.68 0)
 		(layer "F.SilkS")
@@
 		)
 	)
-	(gr_text "PA5 LPS_CK"
+	(gr_text "PA5 LMS_CK"
 		(at 118.237 106.68 0)
 		(layer "B.SilkS")
@@
 		)
 	)
-	(gr_text "LMS_RDY PA9"
+	(gr_text "LPS_RDY PA9"
 		(at 137.541 91.44 0)
 		(layer "B.SilkS")
